File: V1/ESP-relay-16ch-V1.kicad_sch (KiCad schematic)
At the start: 48 parts, among them J1 +24VDC, J2 INPUTS, J3 ETHERNET, J4 OUTPUTS, J5 USB_B_Micro, Q1 UMH3N, U1 SY8089A1AAC, U2 TX4138, U3 LAN8710A, U4 CH340C, U5 ESP32-WROOM-32E-8MB, U6 PCF8574T, U7 PCF8574T

Commit message: Dev updates
Parts:
- added C27: 10uF/16V/1206, Tales:C_1206_3216Metric, symbol Device:C_Polarized_Small_US
- added R100, R101, R102, R103, R104, R95, R96, R97, R98: 2.2k/0,125W/0805, Tales:R_0805_2012Metric, symbol Device:R_US
- added R99: 10k/625mW/0402, Tales:R_0402_1005Metric, symbol Device:R_US
- added U24: PCF8574T, Tales:SO-16_7.5x10.3mm_P1.27mm, symbol Interface_Expansion:PCF8574
- R10: value 470R/0,125W/0805 -> 470R/625mW/0402; footprint Tales:R_0805_2012Metric -> Tales:R_0402_1005Metric; LCSC Part # C17710 -> C25117; Mfr PN 0805W8F4700T5E -> 0402WGF4700TCE; Vendor PN C17710 -> C25117
- R11, R12: value 10k/0,125W/0805 -> 10k/625mW/0402; footprint Tales:R_0805_2012Metric -> Tales:R_0402_1005Metric; Case 0805/2012 -> 0402/1005; LCSC Part # C17414 -> C25890; Mfr PN 0805W8F3301T5E -> 0402WGF3301TCE; Vendor PN C26010 -> C25890
- R13, R14: value 10k/0,125W/0805 -> 2.2k/0,125W/0805; LCSC Part # C17414 -> C17520; Mfr PN 0805W8F3301T5E -> 0805W8F2201T5E; Vendor PN C26010 -> C17520
- R7: value 5k6/0,125W/0805 -> 10k/625mW/0402; footprint Tales:R_0805_2012Metric -> Tales:R_0402_1005Metric; Case 0805/2012 -> 0402/1005; LCSC Part # C4382 -> C25890; Mfr PN 0805W8F5601T5E -> 0402WGF3301TCE; Vendor PN C4382 -> C25890
- R8: value 820R/0,125W/0805 -> 1.5k/625mW/0402; footprint Tales:R_0805_2012Metric -> Tales:R_0402_1005Metric; Case 0805/2012 -> 0402/1005; LCSC Part # C17837 -> C25867; Mfr PN 0805W8F8200T5E -> 0402WGF1501TCE; Vendor PN C17837 -> C25867
- R9: value 330R/0,125W/0805 -> 680R/625mW/0402; footprint Tales:R_0805_2012Metric -> Tales:R_0402_1005Metric; Case 0805/2012 -> 0402/1005; LCSC Part # C17630 -> C25130; Mfr PN 0805W8F3300T5E -> 0402WGF6800TCE; Vendor PN C17630 -> C25130
Connections:
- net +3.3V: now also R100.1, R103.1, R104.1, R95.1, R96.1, R97.1, R99.1, U24.16 (VDD), U24.2 (A1); no longer R13.1, R14.1
- net GNDREF: now also R14.2, U3.33 (VSS), C27.2, R101.2, R102.2, R98.2, U24.1 (A0), U24.3 (A2), U24.8 (VSS)
- net IN1: now also U5.24 (IO2); no longer U5.16 (IO13)
- net IN10: now also U6.5 (P1); no longer U5.12 (IO27)
- net IN11: now also U6.6 (P2); no longer U5.8 (IO32)
- net IN12: now also U6.7 (P3); no longer U5.9 (IO33)
- net IN13: now also U6.9 (P4); no longer U5.6 (IO34)
- net IN14: now also U6.10 (P5); no longer U5.7 (IO35)
- net IN15: now also U6.11 (P6); no longer U5.4 (SENSOR_VP)
- net IN16: now also U6.12 (P7); no longer U5.5 (SENSOR_VN)
- net IN2: now also U5.26 (IO4); no longer U5.13 (IO14)
- net IN3: now also U5.29 (IO5); no longer U5.23 (IO15)
- net IN4: now also U5.16 (IO13); no longer U5.27 (IO16)
- net IN5: now also U5.13 (IO14); no longer U5.30 (IO18)
- net IN6: now also U5.23 (IO15); no longer U5.31 (IO19)
- net IN7: now also U5.27 (IO16); no longer U5.37 (IO23)
- net IN8: now also U5.6 (IO34); no longer U5.10 (IO25)
- net IN9: now also U6.4 (P0); no longer U5.11 (IO26)
- net OUT1: now also U7.4 (P0); no longer U6.4 (P0)
- net OUT10: now also U24.5 (P1); no longer U7.5 (P1)
- net OUT11: now also U24.6 (P2); no longer U7.6 (P2)
- net OUT12: now also U24.7 (P3); no longer U7.7 (P3)
- net OUT13: now also U24.9 (P4); no longer U7.9 (P4)
- net OUT14: now also U24.10 (P5); no longer U7.10 (P5)
- net OUT15: now also U24.11 (P6); no longer U7.11 (P6)
- net OUT16: now also U24.12 (P7); no longer U7.12 (P7)
- net OUT2: now also U7.5 (P1); no longer U6.5 (P1)
- net OUT3: now also U7.6 (P2); no longer U6.6 (P2)
- net OUT4: now also U7.7 (P3); no longer U6.7 (P3)
- net OUT5: now also U7.9 (P4); no longer U6.9 (P4)
- net OUT6: now also U7.10 (P5); no longer U6.10 (P5)
- net OUT7: now also U7.11 (P6); no longer U6.11 (P6)
- net OUT8: now also U7.12 (P7); no longer U6.12 (P7)
- net OUT9: now also U24.4 (P0); no longer U7.4 (P0)
- net EMAC_RXD1: now reaches U3.10 (RXD1/~{MODE1})
- net EMAC_RXD1: now also U5.11 (IO26), R96.2
- net EMAC_RXD0: now reaches U3.11 (RXD0/~{MODE0})
- net EMAC_RXD0: now also U5.10 (IO25), R97.2
- net at U3.13 (RXER/RXD4/~{PHYAD0}): now also R102.1
- net EMAC_RX: now reaches U3.15 (COL/CRS_DV/~{MODE2})
- net EMAC_RX: now also U5.12 (IO27), R100.2
- net EMAC_MDIO: now reaches U3.16 (MDIO)
- net EMAC_MDIO: now also U5.30 (IO18)
- net EMAC_MDC: now reaches U3.17 (MDC)
- net EMAC_MDC: now also U5.37 (IO23)
- net at U3.19 (~{RST}): now also C27.1, R99.2
- net LED_G_K: now reaches U3.2 (LED2/~{INTSEL})
- net LED_G_K: now also J3.10
- net EMAC_TXEN: now reaches U3.21 (TXEN)
- net EMAC_TXEN: now also U5.33 (IO21)
- net EMAC_TXD0: now reaches U3.22 (TXD0)
- net EMAC_TXD0: now also U5.31 (IO19)
- net EMAC_TXD1: now reaches U3.23 (TXD1)
- net EMAC_TXD1: now also U5.36 (IO22)
- net LED_Y_A: now reaches U3.3 (LED1/~{REGOFF})
- net LED_Y_A: now also J3.12
- net at U3.7 (RXCLK/~{PHYAD1}): now also R101.1
- net at U3.8 (RXD3/~{PHYAD2}): now also R98.1
- net at U3.9 (RXD2/~{RMIISEL}): now also R95.2
- net I2C_SCL: now reaches U6.14 (SCL), U7.14 (SCL)
- net I2C_SCL: now also U5.8 (IO32), R104.2, U24.14 (SCL); no longer R14.2, U5.36 (IO22)
- net I2C_SDA: now reaches U6.15 (SDA), U7.15 (SDA)
- net I2C_SDA: now also U5.9 (IO33), R103.2, U24.15 (SDA); no longer R13.2, U5.33 (IO21)
- net at J3.11: now also R14.1
- net at J3.9: now also R13.2
- net PHY_CLK renamed EMAC_CLK
- new net ADC1: U5.7 (IO35)
- new net ADC2: U5.4 (SENSOR_VP)
- new net ADC3: U5.5 (SENSOR_VN)
- no-connect marks 21 -> 22
Other:
- note added: "ADDRESS 0x22"
- moved on the sheet: J3, U3, U6, U7

Commit message: Development updates
Parts:
- removed C5, C9: 10uF/16V/1206, Tales:C_1206_3216Metric, symbol Device:C_Polarized_Small_US
- removed D5, D7: BLUE/0603, Tales:LED_0603_1608Metric, symbol Device:LED_Small
- removed R8: 1.5k/625mW/0402, Tales:R_0402_1005Metric, symbol Device:R_US
- removed R9: 680R/625mW/0402, Tales:R_0402_1005Metric, symbol Device:R_US
- added C28: 22uF/6,3V/0603, Tales:C_0805_2012Metric, symbol Device:C_Small
- added C29: 1uF/6,3V/0402, Tales:C_0402_1005Metric, symbol Device:C_Small
- added C30: 470pF/16V/0402, Tales:C_0402_1005Metric, symbol Device:C_Small
- added C5, C9: 10uF/6,3V/0603, Tales:C_0603_1608Metric, symbol Device:C_Small
- added C?: 1uF/10V/0603, Tales:C_0603_1608Metric, symbol Device:C_Small
- added J2: ADC, Tales:TerminalBlock_Phoenix_MKDS-3-4-5.08_1x04_P5.08mm_Horizontal, symbol Connector_Generic:Conn_01x04
- added L3: 2A 600R, Inductor_SMD:L_0805_2012Metric, symbol Device:L_Ferrite_Small
- added Q18: WPM2015-3/TR, Tales:SOT-23, symbol Device:Q_PMOS_GSD
- added Q19: LMUN2211LT1G, Tales:SOT-23, symbol Device:Q_NPN_BEC_BRT
- added R105, R106, R107, R94: 49,9R/62,5mW/0402, Tales:R_0402_1005Metric, symbol Device:R_US
- added R93: 1k/62,5mW/0402, Tales:R_0402_1005Metric, symbol Device:R_US
- C27: value 10uF/16V/1206 -> 10uF/6,3V/0603; footprint Tales:C_1206_3216Metric -> Tales:C_0603_1608Metric; Case 1206/3216 -> 0603/1608; LCSC Part # C1849 -> C1691; Mfr PN CL31A106KOHNNNE -> CL10A106MQ8NNNC; Vendor PN C1849 -> C1691
- J1: value +24VDC -> VIN
- J4: renamed from J5; value USB_B_Micro -> USB
- L1: Case 12x12 -> 3x3
- LOGO1: JLCPCB BOM (none) -> 1
- R10: value 470R/625mW/0402 -> 10k/62,5mW/0402; Case 0805/2012 -> 0402/1005; LCSC Part # C25117 -> C25890; Mfr PN 0402WGF4700TCE -> 0402WGF1002TCE; Vendor PN C25117 -> C25890
- R100, R101, R102, R103, R104, R95, R96, R97, R98: value 2.2k/0,125W/0805 -> 3k3/62,5mW/0402; footprint Tales:R_0805_2012Metric -> Tales:R_0402_1005Metric; Case 0805/2012 -> 0402/1005; LCSC Part # C17520 -> C25890; Mfr PN 0805W8F2201T5E -> 0402WGF3301TCE; Vendor PN C17520 -> C25890
- R11, R12, R99: value 10k/625mW/0402 -> 10k/62,5mW/0402; Mfr PN 0402WGF3301TCE -> 0402WGF1002TCE
- R13, R14: value 2.2k/0,125W/0805 -> 270R/62,5mW/0402; footprint Tales:R_0805_2012Metric -> Tales:R_0402_1005Metric; Case 0805/2012 -> 0402/1005; LCSC Part # C17520 -> C25099; Mfr PN 0805W8F2201T5E -> 0402WGF2700TCE; Vendor PN C17520 -> C25099
- R7: value 10k/625mW/0402 -> 5,6k/0,100W/0603; footprint Tales:R_0402_1005Metric -> Tales:R_0603_1608Metric; Case 0402/1005 -> 0603/1608; LCSC Part # C25890 -> C23189; Mfr PN 0402WGF3301TCE -> 0603WAF5601T5E; Vendor PN C25890 -> C23189
- U5: Case (none) -> ESP32-WROOM
- renumbered J2 to J5, J4 to J6
Connections:
- net +3.3V: now also R10.1, C28.1, C5.1, C9.1, Q18.2 (S)
- net ADC1: now also J2.1 (Pin_1)
- net ADC2: now also J2.2 (Pin_2)
- net ADC3: now also J2.3 (Pin_3)
- net I2C_SCL: now also R103.2; no longer R104.2
- net I2C_SDA: now also R104.2; no longer R103.2
- net PHY_PWR: now also Q19.1 (B)
- net +3.3VA: now reaches U3.1 (VDD2A)
- net +3.3VA: now also U3.27 (VDD1A), L3.2, R105.1, R106.1, R107.1, R94.1
- net +3.3VLAN: now reaches U3.12 (VDDIO)
- net +3.3VLAN: now also L3.1, Q18.3 (D)
- net at U3.28 (TXN): now also R105.2
- net at U3.29 (TXP): now also R94.2
- net at U3.30 (RXN): now also R107.2
- net at U3.31 (RXP): now also R106.2
- net at U3.6 (VDDCR): now also C29.1, C30.1
- net at U4.3 (RXD): now also U5.35 (TXD0/IO1); no longer R10.2
- net USB_D+: now reaches J4.3 (D+), U4.5 (UD+)
- net USB_D-: now reaches J4.2 (D-), U4.6 (UD-)
- net at Q1.6 (C1), R11.2, U5.3 (EN): now also C?.1
- net GNDREF renamed GND
- net GND: now also C29.2, C30.2, C5.2, C9.2, C?.2, J2.4 (Pin_4), Q19.2 (E)
- new net: C28.2, Q18.1 (G), R10.2, R93.1
- new net: Q19.3 (C), R93.2
Other:
- title: ESP 8x 24VDC Input 8x Relay Output Module -> ESP 16x 24VDC Input 16x External Relay Output Module
- moved on the sheet: C1, C10, C2, C27, C3, C4, C6, C7, C8, D1, D2, D3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

Commit message: Update ESP-relay-16ch-V1.kicad_sch
Parts:
- added C? (x2): 100nF/16V/0402, Tales:C_0402_1005Metric, symbol Device:C_Small
- added R?: 12,1k/62,5mW/0402, Tales:R_0402_1005Metric, symbol Device:R_US
Connections:
- net +3.3VA: now also J3.4, J3.5, R13.1, C?.1, C?.1
- net GND: now also C?.2, C?.2, R?.2
- net TD-: now reaches R105.2, U3.28 (TXN)
- net TD-: now also J3.2 (TD-)
- net TD+: now reaches R94.2, U3.29 (TXP)
- net TD+: now also J3.1 (TD+)
- net RD-: now reaches R107.2, U3.30 (RXN)
- net RD-: now also J3.6 (RD-)
- net RD+: now reaches R106.2, U3.31 (RXP)
- net RD+: now also J3.3 (RD+)
- net at U3.32 (RBIAS): now also R?.1
Other:
- moved on the sheet: C27, C29, C30, J3, R100, R101, R102, R105, R106, R107, R13, R14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

Commit message: Development updates
Parts:
- removed C1: 10uF/16V/1206, Tales:C_1206_3216Metric, symbol Device:C_Polarized_Small_US
- removed C10, C4, C6: 0,1uF/50V/0805, Tales:C_0805_2012Metric, symbol Device:C_Small
- removed C2: 22pF/50V/0603, Tales:C_0603_1608Metric, symbol Device:C_Small
- removed C27: 10uF/6,3V/0603, Tales:C_0603_1608Metric, symbol Device:C_Polarized_Small_US
- removed C28: 22uF/6,3V/0603, Tales:C_0805_2012Metric, symbol Device:C_Small
- removed C29: 1uF/6,3V/0402, Tales:C_0402_1005Metric, symbol Device:C_Small
- removed C3: 47uF/35V/6,3x5,4, Tales:CP_Elec_6.3x5.4, symbol Device:C_Polarized_Small_US
- removed C30: 470pF/16V/0402, Tales:C_0402_1005Metric, symbol Device:C_Small
- removed C5, C9: 10uF/6,3V/0603, Tales:C_0603_1608Metric, symbol Device:C_Small
- removed C7: 12pF/50V/0603, Tales:C_0603_1608Metric, symbol Device:C_Small
- removed C8: 470uF/16V/10x10, Tales:CP_Elec_10x10, symbol Device:C_Polarized_Small_US
- removed C?: 1uF/10V/0603, Tales:C_0603_1608Metric, symbol Device:C_Small
- removed C? (x2): 100nF/16V/0402, Tales:C_0402_1005Metric, symbol Device:C_Small
- removed D1: SM4007PL/SOD-123, Tales:D_SOD-123, symbol Device:D_Small
- removed D2: SS510, Tales:D_SMA, symbol Device:D_Schottky_Small
- removed D3: BLUE/0603, Tales:LED_0603_1608Metric, symbol Device:LED_Small
- removed D4: SS34, Tales:D_SMA, symbol Device:D_Schottky_Small
- removed D6: B5819W, Tales:D_SOD-123, symbol Device:D_Schottky_Small
- removed F1: 500mA, Tales:Fuse_0402_1005Metric, symbol Device:Fuse_Small
- removed J2: ADC, Tales:TerminalBlock_Phoenix_MKDS-3-4-5.08_1x04_P5.08mm_Horizontal, symbol Connector_Generic:Conn_01x04
- removed J3: ETHERNET, Tales:RJ45_HanRun_HR911105A, symbol Tales:HanRun_HR911105A
- removed J4: USB, Connector_USB:USB_Micro-B_Amphenol_10118194_Horizontal, symbol Connector:USB_B_Micro
- removed J5: INPUTS, Tales:TerminalBlock_Phoenix_MKDS-3-16-5.08_1x16_P5.08mm_Horizontal, symbol Connector_Generic:Conn_01x16
- removed J6: OUTPUTS, Tales:TerminalBlock_Phoenix_MKDS-3-18-5.08_1x18_P5.08mm_Horizontal, symbol Connector_Generic:Conn_01x18
- removed L1: 2,2uH 1,5A, Tales:L_3x3_H1.5, symbol Device:L
- removed L2: 33uH 2,1A, Tales:L_12x12mm_H6mm, symbol Device:L
- removed L3: 2A 600R, Inductor_SMD:L_0805_2012Metric, symbol Device:L_Ferrite_Small
- removed LOGO1: Logo_Open_Hardware_Large, Symbol:OSHW-Logo2_14.6x12mm_SilkScreen, symbol Graphic:Logo_Open_Hardware_Large
- removed Q1: UMH3N, Package_TO_SOT_SMD:SOT-363_SC-70-6, symbol Transistor_BJT:UMH3N
- removed Q18: WPM2015-3/TR, Tales:SOT-23, symbol Device:Q_PMOS_GSD
- removed Q19: LMUN2211LT1G, Tales:SOT-23, symbol Device:Q_NPN_BEC_BRT
- removed R1: 100k/0,125W/0805, Tales:R_0805_2012Metric, symbol Device:R_US
- removed R10, R11, R12, R99: 10k/62,5mW/0402, Tales:R_0402_1005Metric, symbol Device:R_US
- removed R100, R101, R102, R103, R104, R95, R96, R97, R98: 3k3/62,5mW/0402, Tales:R_0402_1005Metric, symbol Device:R_US
- removed R105, R106, R107, R94: 49,9R/62,5mW/0402, Tales:R_0402_1005Metric, symbol Device:R_US
- removed R13, R14: 270R/62,5mW/0402, Tales:R_0402_1005Metric, symbol Device:R_US
- removed R2: 22,1k/0,125W/0805, Tales:R_0805_2012Metric, symbol Device:R_US
- removed R3: 30mR/0,250W/0805, Tales:R_0805_2012Metric, symbol Device:R_US
- removed R4: 5R1/0,125W/0805, Tales:R_0805_2012Metric, symbol Device:R_US
- removed R5: 300k/0,125W/0805, Tales:R_0805_2012Metric, symbol Device:R_US
- removed R6: 52,3k/0,125W/0805, Tales:R_0805_2012Metric, symbol Device:R_US
- removed R7: 5,6k/0,100W/0603, Tales:R_0603_1608Metric, symbol Device:R_US
- removed R93: 1k/62,5mW/0402, Tales:R_0402_1005Metric, symbol Device:R_US
- removed R?: 12,1k/62,5mW/0402, Tales:R_0402_1005Metric, symbol Device:R_US
- removed U1: SY8089A1AAC, Tales:TSOT-23-5, symbol Tales:SY8089AAAC
- removed U2: TX4138, Tales:SOIC-8-1EP_3.9x4.9mm_P1.27mm_EP2.29x3mm_ThermalVias, symbol Tales:TX4138
- removed U24, U6, U7: PCF8574T, Tales:SO-16_7.5x10.3mm_P1.27mm, symbol Interface_Expansion:PCF8574
- removed U3: LAN8710A, Package_DFN_QFN:QFN-32-1EP_5x5mm_P0.5mm_EP3.3x3.3mm_ThermalVias, symbol Interface_Ethernet:LAN8710A
- removed U4: CH340C, Package_SO:SOIC-16_3.9x9.9mm_P1.27mm, symbol Interface_USB:CH340C
- removed U5: ESP32-WROOM-32E-8MB, RF_Module:ESP32-WROOM-32, symbol RF_Module:ESP32-WROOM-32
- added J10, J3, J4, J5, J6, J7, J8, J9: DIG IN, TerminalBlock_Phoenix:TerminalBlock_Phoenix_PT-1,5-2-3.5-H_1x02_P3.50mm_Horizontal, symbol Connector_Generic:Conn_01x02
- added J11, J12, J13, J14, J15, J16: DIG OUT, TerminalBlock_Phoenix:TerminalBlock_Phoenix_PT-1,5-3-3.5-H_1x03_P3.50mm_Horizontal, symbol Connector_Generic:Conn_01x03
- added J2: ANA IN, TerminalBlock_Phoenix:TerminalBlock_Phoenix_PT-1,5-2-3.5-H_1x02_P3.50mm_Horizontal, symbol Connector_Generic:Conn_01x02
- J1: value VIN -> ANA IN; footprint Tales:TerminalBlock_Phoenix_MKDS-3-2-5.08_1x02_P5.08mm_Horizontal -> TerminalBlock_Phoenix:TerminalBlock_Phoenix_PT-1,5-2-3.5-H_1x02_P3.50mm_Horizontal; Mfr PN 1x LM 5.08/02/90 3.5SN OR BX -> (none); Vendor PN 1x 1716080000 -> (none)
Connections:
- net +24V: now also J11.1 (Pin_1), J16.3 (Pin_3)
- net GND: now also J2.2 (Pin_2); no longer J1.2 (Pin_2)
- net Inputs/J2-IN1: now also J3.1 (Pin_1)
- net Inputs/J2-IN10: now also J7.2 (Pin_2)
- net Inputs/J2-IN11: now also J8.1 (Pin_1)
- net Inputs/J2-IN12: now also J8.2 (Pin_2)
- net Inputs/J2-IN13: now also J9.1 (Pin_1)
- net Inputs/J2-IN14: now also J9.2 (Pin_2)
- net Inputs/J2-IN15: now also J10.1 (Pin_1)
- net Inputs/J2-IN16: now also J10.2 (Pin_2)
- net Inputs/J2-IN2: now also J3.2 (Pin_2)
- net Inputs/J2-IN3: now also J4.1 (Pin_1)
- net Inputs/J2-IN4: now also J4.2 (Pin_2)
- net Inputs/J2-IN5: now also J5.1 (Pin_1)
- net Inputs/J2-IN6: now also J5.2 (Pin_2)
- net Inputs/J2-IN7: now also J6.1 (Pin_1)
- net Inputs/J2-IN8: now also J6.2 (Pin_2)
- net Inputs/J2-IN9: now also J7.1 (Pin_1)
- net Outputs/J5-OUT1: now also J11.2 (Pin_2)
- net Outputs/J5-OUT10: now also J14.2 (Pin_2)
- net Outputs/J5-OUT11: now also J14.3 (Pin_3)
- net Outputs/J5-OUT12: now also J15.1 (Pin_1)
- net Outputs/J5-OUT13: now also J15.2 (Pin_2)
- net Outputs/J5-OUT14: now also J15.3 (Pin_3)
- net Outputs/J5-OUT15: now also J16.1 (Pin_1)
- net Outputs/J5-OUT16: now also J16.2 (Pin_2)
- net Outputs/J5-OUT2: now also J11.3 (Pin_3)
- net Outputs/J5-OUT3: now also J12.1 (Pin_1)
- net Outputs/J5-OUT4: now also J12.2 (Pin_2)
- net Outputs/J5-OUT5: now also J12.3 (Pin_3)
- net Outputs/J5-OUT6: now also J13.1 (Pin_1)
- net Outputs/J5-OUT7: now also J13.2 (Pin_2)
- net Outputs/J5-OUT8: now also J13.3 (Pin_3)
- net Outputs/J5-OUT9: now also J14.1 (Pin_1)
- net MCU/ADC1: now reaches J1.1 (Pin_1)
- new net MCU/ADC2: J1.2 (Pin_2)
- new net MCU/ADC3: J2.1 (Pin_1)
- no-connect marks 22 -> 0
Other:
- added sheet Ethernet (ESP-relay-16ch-V1-ethernet.kicad_sch)
- added sheet MCU (ESP-relay-16ch-V1-mcu.kicad_sch)
- added sheet Power (ESP-relay-16ch-V1-power.kicad_sch)
- note removed: "5V MAIN"
- note removed: "5V USB"
- note removed: "ADDRESS 0x20"
- note removed: "ADDRESS 0x21"
- note removed: "ADDRESS 0x22"
- note removed: "OPEN HARDWARE"
