File: V1/ESP-relay-16ch-V1-ethernet.kicad_sch (KiCad schematic)
At the start: 27 parts, among them J17 ETHERNET, U17 LAN8710A

Commit message: Dev updates
Connections:
- no-connect marks 5 -> 6
Changed lines of the file:
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@@
   (junction (at 184.15 30.48) (diameter 0) (color 0 0 0 0)
   )
+  (no_connect (at 63.5 158.75))
   (no_connect (at 156.21 92.71))
   (no_connect (at 156.21 80.01))
@@
       (effects (font (size 1.27 1.27)) (justify left top) hide)
     )
-    (property "Case" "~" (id 4) (at 48.26 148.59 0)
-      (effects (font (size 1.27 1.27)) hide)
-    )
-    (property "JLCPCB BOM" "1" (id 5) (at 48.26 148.59 0)
+    (property "Case" "~" (id 4) (at 48.26 144.78 0)
+      (effects (font (size 1.27 1.27)) hide)
+    )
+    (property "JLCPCB BOM" "1" (id 5) (at 48.26 153.035 0)
       (effects (font (size 1.27 1.27)) hide)
     )
     (property "LCSC Part #" "C12074" (id 6) (at 29.21 153.67 0))
-    (property "Mfr" "HanRun" (id 7) (at 48.26 148.59 0)
-      (effects (font (size 1.27 1.27)) hide)
-    )
-    (property "Mfr PN" "HR911105A" (id 8) (at 48.26 148.59 0)
+    (property "Mfr" "HanRun" (id 7) (at 48.26 146.685 0)
+      (effects (font (size 1.27 1.27)) hide)
+    )
+    (property "Mfr PN" "HR911105A" (id 8) (at 48.26 143.51 0)
       (effects (font (size 1.27 1.27)) hide)
     )
@@
       (effects (font (size 1.27 1.27)) hide)
     )
-    (property "Vendor" "JLCPCB" (id 10) (at 48.26 148.59 0)
-      (effects (font (size 1.27 1.27)) hide)
-    )
-    (property "Vendor PN" "C12074" (id 11) (at 48.26 148.59 0)
+    (property "Vendor" "JLCPCB" (id 10) (at 48.26 151.13 0)
+      (effects (font (size 1.27 1.27)) hide)
+    )
+    (property "Vendor PN" "C12074" (id 11) (at 48.26 154.94 0)
       (effects (font (size 1.27 1.27)) hide)
     )
@@
     (pin "5")
     (pin "6")
+    (pin "7")
     (pin "8")
     (pin "9")

Commit message: Dev updates
Parts:
- renumbered J17 to J6
Other:
- moved on the sheet: J6
Changed lines of the file:
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@@
   (junction (at 184.15 30.48) (diameter 0) (color 0 0 0 0)
   )
-  (no_connect (at 63.5 158.75))
+  (no_connect (at 63.5 160.02))
   (no_connect (at 156.21 92.71))
   (no_connect (at 156.21 80.01))
@@
     (stroke (width 0) (type default) (color 0 0 0 0))
   )
-  (wire (pts (xy 63.5 163.83) (xy 63.5 161.29))
+  (wire (pts (xy 64.77 163.83) (xy 64.77 162.56))
     (stroke (width 0) (type default) (color 0 0 0 0))
   )
@@
     (stroke (width 0) (type default) (color 0 0 0 0))
   )
+  (wire (pts (xy 64.77 162.56) (xy 63.5 162.56))
+    (stroke (width 0) (type default) (color 0 0 0 0))
+  )
   (wire (pts (xy 147.32 97.79) (xy 156.21 97.79))
     (stroke (width 0) (type default) (color 0 0 0 0))
@@
     (stroke (width 0) (type default) (color 0 0 0 0))
   )
-  (wire (pts (xy 48.26 173.99) (xy 48.26 176.53))
+  (wire (pts (xy 48.26 173.99) (xy 48.26 175.26))
     (stroke (width 0) (type default) (color 0 0 0 0))
   )
@@
     (stroke (width 0) (type default) (color 0 0 0 0))
   )
-  (wire (pts (xy 48.26 166.37) (xy 48.26 168.91))
+  (wire (pts (xy 48.26 167.64) (xy 48.26 168.91))
     (stroke (width 0) (type default) (color 0 0 0 0))
   )
@@
     (stroke (width 0) (type default) (color 0 0 0 0))
   )
-  (wire (pts (xy 63.5 163.83) (xy 73.66 163.83))
+  (wire (pts (xy 64.77 163.83) (xy 73.66 163.83))
     (stroke (width 0) (type default) (color 0 0 0 0))
   )
@@
   (symbol (lib_id "Tales:HanRun_HR911105A") (at 48.26 148.59 0) (unit 1)
     (in_bom yes) (on_board yes)
-    (property "Reference" "J17" (id 0) (at 33.655 148.5899 0)
+    (property "Reference" "J6" (id 0) (at 33.655 148.5899 0)
       (effects (font (size 1.27 1.27)) (justify right))
     )
@@
     (pin "1")
   )
-  (symbol (lib_id "power:GND") (at 48.26 176.53 0) (unit 1)
-    (in_bom yes) (on_board yes)
-    (property "Reference" "#PWR0101" (id 0) (at 48.26 182.88 0)
-      (effects (font (size 1.27 1.27)) hide)
-    )
-    (property "Value" "GNDREF" (id 1) (at 48.387 180.9242 0)
-      (effects (font (size 1.27 1.27)) hide)
-    )
-    (property "Footprint" "" (id 2) (at 48.26 176.53 0)
-      (effects (font (size 1.27 1.27)) hide)
-    )
-    (property "Datasheet" "" (id 3) (at 48.26 176.53 0)
-      (effects (font (size 1.27 1.27)) hide)
-    )
+  (symbol (lib_id "power:GND") (at 48.26 175.26 0) (unit 1)
+    (in_bom yes) (on_board yes)
+    (property "Reference" "#PWR0101" (id 0) (at 48.26 181.61 0)
+      (effects (font (size 1.27 1.27)) hide)
+    )
+    (property "Value" "GNDREF" (id 1) (at 48.387 179.6542 0)
+      (effects (font (size 1.27 1.27)) hide)
+    )
+    (property "Footprint" "" (id 2) (at 48.26 175.26 0)
+      (effects (font (size 1.27 1.27)) hide)
+    )
+    (property "Datasheet" "" (id 3) (at 48.26 175.26 0)
+      (effects (font (size 1.27 1.27)) hide)
+    )
