File: V1/ESP-relay-16ch-V1-outputs.kicad_sch (KiCad schematic)
At the start: 40 parts

Commit message: Dev updates
Parts:
- added D32, D33, D34, D35, D36, D37, D38, D39: BLUE/0603, Tales:LED_0603_1608Metric, symbol Device:LED_Small
- added Q10, Q11, Q12, Q13, Q14, Q15, Q16, Q17: MMBT2222A/SOT-23-3, Tales:SOT-23, symbol Device:Q_NPN_BEC
- added R71, R72, R73, R74, R83, R84, R85, R86: 10k/0,125W/0805, Tales:R_0805_2012Metric, symbol Device:R_US
- added R75, R76, R77, R78, R87, R88, R89, R90: 1k/0,125W/0805, Tales:R_0805_2012Metric, symbol Device:R_US
- added R79, R80, R81, R82, R91, R92, R93, R94: 4k7/0,125W/0805, Tales:R_0805_2012Metric, symbol Device:R_US
- gave numbers to parts that had none: 40
Connections:
- net +24V: now also R79.1, R80.1, R81.1, R82.1, R91.1, R92.1, R93.1, R94.1
- net GNDREF: now also Q10.2 (E), Q11.2 (E), Q12.2 (E), Q13.2 (E), Q14.2 (E), Q15.2 (E), Q16.2 (E), Q17.2 (E), R71.2, R72.2, R73.2, R74.2, R83.2, R84.2, R85.2, R86.2
- new net: D37.2 (A), R92.2
- new net: Q10.1 (B), R75.1
- new net: Q17.1 (B), R90.1
- new net: D39.2 (A), R94.2
- new net: Q15.1 (B), R88.1
- new net: Q12.1 (B), R77.1
- new net: D35.2 (A), R82.2
- new net: Q14.1 (B), R87.1
- new net: D33.2 (A), R80.2
- new net: D34.2 (A), R81.2
- new net: D38.2 (A), R93.2
- new net: Q11.1 (B), R76.1
- new net: D36.2 (A), R91.2
- new net: Q13.1 (B), R78.1
- new net: Q16.1 (B), R89.1
- new net: D32.2 (A), R79.2
- new net J5-OUT10: D33.1 (K), Q11.3 (C)
- new net J5-OUT11: D34.1 (K), Q12.3 (C)
- new net J5-OUT12: D35.1 (K), Q13.3 (C)
- new net J5-OUT13: D36.1 (K), Q14.3 (C)
- new net J5-OUT14: D37.1 (K), Q15.3 (C)
- new net J5-OUT15: D38.1 (K), Q16.3 (C)
- new net J5-OUT16: D39.1 (K), Q17.3 (C)
- new net J5-OUT9: D32.1 (K), Q10.3 (C)
- new net OUT10: R72.1, R76.2
- new net OUT11: R73.1, R77.2
- new net OUT12: R74.1, R78.2
- new net OUT13: R83.1, R87.2
- new net OUT14: R84.1, R88.2
- new net OUT15: R85.1, R89.2
- new net OUT16: R86.1, R90.2
- new net OUT9: R71.1, R75.2
Other:
- moved on the sheet: D24, D25, D26, D27, D28, D29, D30, D31, Q2, Q3, Q4, Q5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

Commit message: Dev updates
Parts:
- R47, R48, R49, R50, R59, R60, R61, R62, R71, R72, R73, R74, R83, R84, R85, R86: value 10k/0,125W/0805 -> 10k/625mW/0402; footprint Tales:R_0805_2012Metric -> Tales:R_0402_1005Metric; Case 0805/2012 -> 0402/1005; LCSC Part # C17414 -> C25890; Mfr PN 0805W8F3301T5E -> 0402WGF3301TCE; Vendor PN C26010 -> C25890
- R51, R52, R53, R54, R63, R64, R65, R66, R75, R76, R77, R78, R87, R88, R89, R90: value 1k/0,125W/0805 -> 1k/625mW/0402; footprint Tales:R_0805_2012Metric -> Tales:R_0402_1005Metric; Case 0805/2012 -> 0402/1005; LCSC Part # C17513 -> C11702; Mfr PN 0805W8F1001T5E -> 0402WGF1001TCE; Vendor PN C17513 -> C11702
- R55, R56, R57, R58, R67, R68, R69, R70, R79, R80, R81, R82, R91, R92, R93, R94: value 4k7/0,125W/0805 -> 10k/625mW/0402; footprint Tales:R_0805_2012Metric -> Tales:R_0402_1005Metric; Case 0805/2012 -> 0402/1005; LCSC Part # C17673 -> C25890; Mfr PN 0805W8F4701T5E -> 0402WGF3301TCE; Vendor PN C17673 -> C25890

Commit message: Development updates
Parts:
- removed R93, R94: 10k/625mW/0402, Tales:R_0402_1005Metric, symbol Device:R_US
- added R8, R9: 5,6k/0,100W/0603, Tales:R_0603_1608Metric, symbol Device:R_US
- R47, R48, R49, R50, R59, R60, R61, R62, R71, R72, R73, R74, R83, R84, R85, R86: value 10k/625mW/0402 -> 10k/62,5mW/0402; Mfr PN 0402WGF3301TCE -> 0402WGF1002TCE
- R51, R52, R53, R54, R63, R64, R65, R66, R75, R76, R77, R78, R87, R88, R89, R90: value 1k/625mW/0402 -> 1k/62,5mW/0402
- R55, R56, R57, R58, R67, R68, R69, R70, R79, R80, R81, R82, R91, R92: value 10k/625mW/0402 -> 5,6k/0,100W/0603; footprint Tales:R_0402_1005Metric -> Tales:R_0603_1608Metric; Case 0402/1005 -> 0603/1608; LCSC Part # C25890 -> C23189; Mfr PN 0402WGF3301TCE -> 0603WAF5601T5E; Vendor PN C25890 -> C23189
Connections:
- net +24V: now also R8.1, R9.1
- net at R58.2: now also D29.2 (A); no longer D27.2 (A)
- net at D37.2 (A): now also R82.2; no longer R92.2
- net at D26.2 (A): now also R55.2; no longer R57.2
- net at R70.2: now also D33.2 (A); no longer D31.2 (A)
- net at D39.2 (A): now also R92.2
- net at D24.2 (A): now also R8.2; no longer R55.2
- net at D35.2 (A): now also R80.2; no longer R82.2
- net at R68.2: now also D31.2 (A); no longer D29.2 (A)
- net at R56.2: now also D27.2 (A); no longer D25.2 (A)
- net at D30.2 (A): now also R67.2; no longer R69.2
- net at R81.2: now also D36.2 (A); no longer D34.2 (A)
- net at D38.2 (A): now also R91.2
- net at D28.2 (A): now also R57.2; no longer R67.2
- net at D32.2 (A): now also R69.2; no longer R79.2
- net GNDREF renamed GND
- new net: D25.2 (A), R9.2
- new net: D34.2 (A), R79.2
Other:
- title: (none) -> ESP 16x 24VDC Input 16x External Relay Output Module

Commit message: Development updates
Parts:
- renumbered D24 to D17, D25 to D18, D26 to D19, D27 to D20, D28 to D21, D29 to D22, D30 to D23, D31 to D24, D32 to D25, D33 to D26, D34 to D27, D35 to D28, D36 to D29, D37 to D30, D38 to D31, D39 to D32, Q2 to Q1, Q11 to Q10, Q12 to Q11, Q13 to Q12, Q14 to Q13, Q15 to Q14, Q16 to Q15, Q17 to Q16, Q3 to Q2, Q4 to Q3, Q5 to Q4, Q6 to Q5, Q7 to Q6, Q8 to Q7, Q9 to Q8, Q10 to Q9, R47 to R33, R48 to R34, R49 to R35, R50 to R36, R51 to R37, R52 to R38, R53 to R39, R54 to R40, R8 to R41, R9 to R42, R55 to R43, R56 to R44, R59 to R45, R60 to R46, R61 to R47, R62 to R48, R63 to R49, R64 to R50, R65 to R51, R66 to R52, R57 to R53, R58 to R54, R67 to R55, R68 to R56, R71 to R57, R72 to R58, R73 to R59, R74 to R60, R75 to R61, R76 to R62, R77 to R63, R78 to R64, R69 to R65, R70 to R66, R79 to R67, R80 to R68, R83 to R69, R84 to R70, R85 to R71, R86 to R72, R87 to R73, R88 to R74, R89 to R75, R90 to R76, R81 to R77, R82 to R78, R91 to R79, R92 to R80
Other:
- moved on the sheet: D18, D19, D20, D22, D23, D24, D26, D27, D28, D30, D31, D32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

Commit message: Dev updates
Parts:
- R102: renamed from R56; value 5,6k/0,100W/0603 -> 5,6k/0,1W/0603
- R105: renamed from R65; value 5,6k/0,100W/0603 -> 5,6k/0,1W/0603
- R108: renamed from R66; value 5,6k/0,100W/0603 -> 5,6k/0,1W/0603
- R111: renamed from R67; value 5,6k/0,100W/0603 -> 5,6k/0,1W/0603
- R114: renamed from R68; value 5,6k/0,100W/0603 -> 5,6k/0,1W/0603
- R117: renamed from R77; value 5,6k/0,100W/0603 -> 5,6k/0,1W/0603
- R120: renamed from R78; value 5,6k/0,100W/0603 -> 5,6k/0,1W/0603
- R123: renamed from R79; value 5,6k/0,100W/0603 -> 5,6k/0,1W/0603
- R126: renamed from R80; value 5,6k/0,100W/0603 -> 5,6k/0,1W/0603
- R81: renamed from R41; value 5,6k/0,100W/0603 -> 5,6k/0,1W/0603
- R84: renamed from R42; value 5,6k/0,100W/0603 -> 5,6k/0,1W/0603
- R87: renamed from R43; value 5,6k/0,100W/0603 -> 5,6k/0,1W/0603
- R90: renamed from R44; value 5,6k/0,100W/0603 -> 5,6k/0,1W/0603
- R93: renamed from R53; value 5,6k/0,100W/0603 -> 5,6k/0,1W/0603
- R96: renamed from R54; value 5,6k/0,100W/0603 -> 5,6k/0,1W/0603
- R99: renamed from R55; value 5,6k/0,100W/0603 -> 5,6k/0,1W/0603
- renumbered D17 to D39, D18 to D40, D19 to D41, D20 to D42, D21 to D43, D22 to D44, D23 to D45, D24 to D46, D25 to D47, D26 to D48, D27 to D49, D28 to D50, D29 to D51, D30 to D52, D31 to D53, D32 to D54, Q7 to Q10, Q8 to Q11, Q9 to Q12, Q10 to Q13, Q11 to Q14, Q12 to Q15, Q13 to Q16, Q14 to Q17, Q15 to Q18, Q16 to Q19, Q1 to Q4, Q2 to Q5, Q3 to Q6, Q4 to Q7, Q5 to Q8, Q6 to Q9, R48 to R100, R52 to R101, R57 to R103, R61 to R104, R58 to R106, R62 to R107, R59 to R109, R63 to R110, R60 to R112, R64 to R113, R69 to R115, R73 to R116, R70 to R118, R74 to R119, R71 to R121, R75 to R122, R72 to R124, R76 to R125, R33 to R79, R37 to R80, R34 to R82, R38 to R83, R35 to R85, R39 to R86, R36 to R88, R40 to R89, R45 to R91, R49 to R92, R46 to R94, R50 to R95, R47 to R97, R51 to R98
