File: V1/ESP-relay-16ch-V1-power.kicad_sch (KiCad schematic)
At the start: 34 parts, among them J18 VIN, J19 USB, Q17 WPM2015-3/TR, Q18 LMUN2211LT1G, U18 SY8089A1AAC, U19 TX4138

Commit message: Dev updates
Parts:
- removed C29: 10uF/6,3V/0603, Tales:C_0603_1608Metric, symbol Device:C_Small
- added C29: 10uF/16V/1206, Tales:C_1206_3216Metric, symbol Device:C_Polarized_Small_US
Connections:
- net +3.3V: now also C29.1
- net GND: now also C29.2
Changed lines of the file:
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@@
-    (pin "2")
-  )
-  (symbol (lib_id "Device:C_Small") (at 115.57 130.81 0) (unit 1)
-    (in_bom yes) (on_board yes)
-    (property "Reference" "C29" (id 0) (at 118.11 127 0)
-      (effects (font (size 1.27 1.27)) (justify left))
-    )
-    (property "Value" "10uF/6,3V/0603" (id 1) (at 118.11 129.54 0)
-      (effects (font (size 1.27 1.27)) (justify left))
-    )
-    (property "Footprint" "Tales:C_0603_1608Metric" (id 2) (at 115.57 130.81 0)
-      (effects (font (size 1.27 1.27)) hide)
-    )
-    (property "Datasheet" "~" (id 3) (at 115.57 130.81 0)
-      (effects (font (size 1.27 1.27)) hide)
-    )
-    (property "Technology" "Ceramic X5R" (id 4) (at 118.11 132.08 0)
-      (effects (font (size 1.27 1.27)) (justify left))
-    )
-    (property "Case" "0603/1608" (id 5) (at 115.57 130.81 0)
-      (effects (font (size 1.27 1.27)) hide)
-    )
-    (property "Mfr" "Samsung" (id 6) (at 115.57 130.81 0)
-      (effects (font (size 1.27 1.27)) hide)
-    )
-    (property "Mfr PN" "CL10A106MQ8NNNC" (id 7) (at 115.57 130.81 0)
-      (effects (font (size 1.27 1.27)) hide)
-    )
-    (property "Vendor" "JLCPCB" (id 8) (at 115.57 130.81 0)
-      (effects (font (size 1.27 1.27)) hide)
-    )
-    (property "Vendor PN" "C1691" (id 9) (at 115.57 130.81 0)
-      (effects (font (size 1.27 1.27)) hide)
-    )
-    (property "LCSC Part #" "C1691" (id 10) (at 118.11 134.62 0)
-      (effects (font (size 1.27 1.27)) (justify left))
-    )
-    (property "JLCPCB BOM" "1" (id 11) (at 115.57 130.81 0)
-      (effects (font (size 1.27 1.27)) hide)
-    )
-    (pin "1")
     (pin "2")
   )
@@
       (effects (font (size 1.27 1.27)) hide)
     )
+    (pin "1")
+    (pin "2")
+  )
+  (symbol (lib_id "Device:C_Polarized_Small_US") (at 115.57 130.81 0) (unit 1)
+    (in_bom yes) (on_board yes)
+    (property "Reference" "C29" (id 0) (at 118.11 128.905 0)
+      (effects (font (size 1.27 1.27)) (justify left))
+    )
+    (property "Value" "10uF/16V/1206" (id 1) (at 118.11 131.445 0)
+      (effects (font (size 1.27 1.27)) (justify left))
+    )
+    (property "Footprint" "Tales:C_1206_3216Metric" (id 2) (at 115.57 130.81 0)
+      (effects (font (size 1.27 1.27)) hide)
+    )
+    (property "Datasheet" "~" (id 3) (at 115.57 130.81 0)
+      (effects (font (size 1.27 1.27)) hide)
+    )
+    (property "Mfr" "Samsung" (id 4) (at 115.57 130.81 0)
+      (effects (font (size 1.27 1.27)) hide)
+    )
+    (property "Mfr PN" "CL31A106KOHNNNE" (id 5) (at 115.57 130.81 0)
+      (effects (font (size 1.27 1.27)) hide)
+    )
+    (property "JLCPCB BOM" "1" (id 6) (at 115.57 130.81 0)
+      (effects (font (size 1.27 1.27)) hide)
+    )
+    (property "LCSC Part #" "C1849" (id 7) (at 118.11 136.525 0)
+      (effects (font (size 1.27 1.27)) (justify left))
+    )
+    (property "Technology" "Ceramic X5R" (id 8) (at 118.11 133.985 0)
+      (effects (font (size 1.27 1.27)) (justify left))
+    )
+    (property "Vendor" "JLCPCB" (id 9) (at 115.57 130.81 0)
+      (effects (font (size 1.27 1.27)) hide)
+    )
+    (property "Vendor PN" "C1849" (id 10) (at 115.57 130.81 0)
+      (effects (font (size 1.27 1.27)) hide)
+    )
+    (property "Case" "1206/3216" (id 11) (at 115.57 130.81 0)
+      (effects (font (size 1.27 1.27)) hide)
+    )

Commit message: Dev updates
Parts:
- renumbered J18 to J4, J19 to J5
Changed lines of the file:
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@@
   (symbol (lib_id "Connector:USB_B_Micro") (at 38.1 91.44 0) (unit 1)
     (in_bom yes) (on_board yes)
-    (property "Reference" "J19" (id 0) (at 38.1 76.2 0))
+    (property "Reference" "J5" (id 0) (at 38.1 76.2 0))
     (property "Value" "USB" (id 1) (at 38.1 78.74 0))
     (property "Footprint" "Connector_USB:USB_Micro-B_Amphenol_10118194_Horizontal" (id 2) (at 41.91 92.71 0)
@@
   (symbol (lib_id "Connector_Generic:Conn_01x02") (at 34.29 36.83 0) (mirror y) (unit 1)
     (in_bom yes) (on_board yes) (fields_autoplaced)
-    (property "Reference" "J18" (id 0) (at 34.29 30.48 0))
+    (property "Reference" "J4" (id 0) (at 34.29 30.48 0))
     (property "Value" "VIN" (id 1) (at 34.29 33.02 0))
     (property "Footprint" "Tales:TerminalBlock_Phoenix_MKDS-3-2-5.08_1x02_P5.08mm_Horizontal" (id 2) (at 34.29 36.83 0)

Commit message: Dev updates
Parts:
- removed C30, C33: 22uF/6,3V/0603, Tales:C_0805_2012Metric, symbol Device:C_Small
- added C10, C9: 10uF/6,3V/0603, Tales:C_0603_1608Metric, symbol Device:C_Small
- C6: renamed from C25; symbol Device:C_Polarized_Small_US -> Device:C_Small
- C8: renamed from C29; symbol Device:C_Polarized_Small_US -> Device:C_Small
- R1: renamed from R97; value 5,6k/0,100W/0603 -> 5,6k/0,1W/0603
- renumbered C26 to C1, C28 to C2, C31 to C3, C32 to C4, C34 to C5, C27 to C7, D34 to D1, D35 to D2, D37 to D3, D38 to D4, D36 to D5, J4 to J1, J5 to J2, L2 to L1, L1 to L2, Q17 to Q1, Q18 to Q2, R100 to R2, R101 to R3, R104 to R4, R105 to R5, R98 to R6, R99 to R7, R102 to R8, R103 to R9, U19 to U1, U18 to U2
Connections:
- net +3.3V: now also C9.1
- net +3.3VLAN: now also C10.1
- net GND: now also C10.2
- net at Q1.1 (G), R8.2, R9.2: now also C9.2
Other:
- moved on the sheet: R6, R7

Commit message: Dev updates
Parts:
- J1: footprint Tales:TerminalBlock_Phoenix_MKDS-3-2-5.08_1x02_P5.08mm_Horizontal -> Tales:TerminalBlock_Phoenix_PT-1,5-2-3.5-H_1x02_P3.50mm_Horizontal
Changed lines of the file:
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@@
     (property "Reference" "J1" (id 0) (at 34.29 30.48 0))
     (property "Value" "VIN" (id 1) (at 34.29 33.02 0))
-    (property "Footprint" "Tales:TerminalBlock_Phoenix_MKDS-3-2-5.08_1x02_P5.08mm_Horizontal" (id 2) (at 34.29 36.83 0)
+    (property "Footprint" "Tales:TerminalBlock_Phoenix_PT-1,5-2-3.5-H_1x02_P3.50mm_Horizontal" (id 2) (at 34.29 36.83 0)
       (effects (font (size 1.27 1.27)) hide)
     )
