File: V1/ESP-relay-16ch-V1.kicad_pcb (KiCad board)
At the start: 2 copper layers, 198 x 67.8 mm, 272 parts, among them J1 VIN, J2 USB, J3 ANA IN, J4 DIG IN, J5 ETHERNET, J6 DIG OUT, Q1 WPM2015-3/TR, Q10 MMBT2222A/SOT-23-3, Q11 MMBT2222A/SOT-23-3, Q12 MMBT2222A/SOT-23-3, Q13 MMBT2222A/SOT-23-3, Q14 MMBT2222A/SOT-23-3, Q15 MMBT2222A/SOT-23-3, Q16 MMBT2222A/SOT-23-3, Q17 MMBT2222A/SOT-23-3, Q18 MMBT2222A/SOT-23-3, Q19 MMBT2222A/SOT-23-3, Q2 LMUN2211LT1G, Q3 UMH3N, Q4 MMBT2222A/SOT-23-3, Q5 MMBT2222A/SOT-23-3, Q6 MMBT2222A/SOT-23-3, Q7 MMBT2222A/SOT-23-3, Q8 MMBT2222A/SOT-23-3, Q9 MMBT2222A/SOT-23-3, SW1 RESET, U1 TX4138, U10 LTV-817S, U11 LTV-817S, U12 LTV-817S, U13 LTV-817S, U14 LTV-817S, U15 LTV-817S, U16 LTV-817S, U17 LTV-817S, U18 LTV-817S, U19 CH340C, U2 SY8089A1AAC, U20 ESP32-WROOM-32E-8MB, U21 PCF8574TS, U22 PCF8574TS, U23 PCF8574TS, U24 LAN8710A, U3 LTV-817S, U4 LTV-817S, U5 LTV-817S, U6 LTV-817S, U7 LTV-817S, U8 LTV-817S, U9 LTV-817S

Commit message: Update ESP-relay-16ch-V1.kicad_pcb
Parts:
- moved C12 183.0 mm to (103.5, 147.3)
- moved R15 181.4 mm to (105.3, 143.5)
- moved C13 174.6 mm to (129.1, 168.0)
- moved C14 174.6 mm to (124.6, 174.0)
- moved C15 174.6 mm to (120.2, 167.9)
- moved C16 174.6 mm to (152.1, 144.7)
- moved C17 174.6 mm to (138.9, 158.0)
- moved C18 174.6 mm to (132.1, 164.6)
- moved C19 174.6 mm to (140.1, 154.6)
- moved C20 174.6 mm to (124.6, 168.0)
- moved C21 174.6 mm to (112.2, 184.4)
- moved C22 174.6 mm to (145.7, 148.0)
- moved C23 174.6 mm to (132.6, 161.3)
- moved C24 174.6 mm to (118.2, 177.8)
- moved C25 174.6 mm to (113.3, 174.6)
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
Commit message: Dev updates
Parts:
- removed J3: ANA IN, TerminalBlock_Phoenix:TerminalBlock_Phoenix_PT-1,5-4-3.5-H_1x04_P3.50mm_Horizontal
- moved R54 107.5 mm to (148.0, 78.0), turned to -90 degrees
- moved D17 106.7 mm to (97.8, 71.3), turned to 90 degrees
- moved C21 105.4 mm to (113.7, 79.1), turned to -90 degrees
- moved D25 103.3 mm to (116.3, 85.2), turned to 90 degrees
- moved U24 102.7 mm to (176.5, 80.5)
- moved D35 100.1 mm to (134.6, 78.3), turned to 90 degrees
- moved C26 99.2 mm to (132.1, 72.1), turned to -90 degrees
- moved C25 97.4 mm to (132.1, 79.1), turned to -90 degrees
- moved D13 96.0 mm to (97.8, 85.2), turned to 90 degrees
- moved D15 93.3 mm to (97.8, 78.3), turned to 90 degrees
- moved C24 92.8 mm to (132.1, 86.0), turned to -90 degrees
- moved C14 92.7 mm to (95.2, 86.0), turned to -90 degrees
- moved D11 92.6 mm to (97.8, 92.2), turned to 90 degrees
- moved C15 92.3 mm to (95.2, 79.1), turned to -90 degrees
- moved C16 92.2 mm to (95.2, 72.1), turned to -90 degrees
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Connections:
- U20 pad 4: /MCU/ADC2 -> /Inputs/IN10
- U20 pad 5: /MCU/ADC3 -> /Inputs/IN11
- U20 pad 7: /MCU/ADC1 -> /Inputs/IN9
- U21 pad 10: /Inputs/IN9 -> /Inputs/IN12
- U21 pad 11: /Inputs/IN10 -> /Inputs/IN13
- U21 pad 12: /Inputs/IN11 -> /Inputs/IN14
- U21 pad 14: /Inputs/IN12 -> /Inputs/IN15
- U21 pad 16: /Inputs/IN13 -> /Inputs/IN16
- U21 pad 17: /Inputs/IN14 -> unconnected-(U21-Pad17)
- U21 pad 19: /Inputs/IN15 -> unconnected-(U21-Pad19)
- U21 pad 20: /Inputs/IN16 -> unconnected-(U21-Pad20)
Routing:
- net GND: track 80.4 -> 90.6 mm
- net Net-(D1-Pad2): track 10.2 -> 0.00 mm

Commit message: Dev updates
Parts:
- J1: footprint Tales:TerminalBlock_Phoenix_MKDS-3-2-5.08_1x02_P5.08mm_Horizontal -> Tales:TerminalBlock_Phoenix_PT-1,5-2-3.5-H_1x02_P3.50mm_Horizontal
- J3: renamed from J4; footprint TerminalBlock_Phoenix:TerminalBlock_Phoenix_PT-1,5-16-3.5-H_1x16_P3.50mm_Horizontal -> Tales:TerminalBlock_Phoenix_PT-1,5-16-3.5-H_1x16_P3.50mm_Horizontal
- moved D2 181.9 mm to (71.8, 114.5), turned to 90 degrees
- moved R1 180.5 mm to (69.8, 114.5), turned to 90 degrees
- moved D1 170.8 mm to (70.9, 121.9)
- moved R85 152.2 mm to (180.3, 113.8), turned to -90 degrees
- moved Q4 150.8 mm to (173.4, 117.1), turned to -90 degrees
- moved R97 148.2 mm to (195.6, 113.8), turned to -90 degrees
- moved R84 147.9 mm to (177.0, 109.9), turned to 180 degrees
- moved R101 147.5 mm to (200.7, 113.8), turned to 90 degrees
- moved R79 147.0 mm to (172.7, 113.8), turned to -90 degrees
- moved Q19 146.1 mm to (230.5, 117.1), turned to -90 degrees
- moved D41 145.7 mm to (180.8, 111.8), turned to 180 degrees
- moved R80 145.3 mm to (174.0, 113.8), turned to 90 degrees
- moved Q18 144.8 mm to (226.7, 117.1), turned to -90 degrees
- moved Q7 144.5 mm to (184.8, 117.1), turned to -90 degrees
- moved R96 144.1 mm to (192.2, 109.9), turned to 180 degrees
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- renumbered J5 to J4, J6 to J5
Routing:
- net GND: track 90.6 -> 483.8 mm, vias 40 -> 45
- net /Inputs/J2-IN16: track 0.00 -> 6.96 mm
- net /Inputs/J2-IN7: track 0.00 -> 6.89 mm
- net /Inputs/J2-IN1: track 0.00 -> 6.88 mm
- net /Inputs/J2-IN15: track 0.00 -> 6.83 mm
- net /Inputs/J2-IN8: track 0.00 -> 6.77 mm
- net /Inputs/J2-IN2: track 0.00 -> 6.75 mm
- net /Inputs/J2-IN14: track 0.00 -> 6.70 mm
- net /Inputs/J2-IN9: track 0.00 -> 6.64 mm
- net /Inputs/J2-IN3: track 0.00 -> 6.62 mm
- net /Inputs/J2-IN13: track 0.00 -> 6.58 mm
- net /Inputs/J2-IN10: track 0.00 -> 6.51 mm
- net /Inputs/J2-IN4: track 0.00 -> 6.49 mm
- net /Inputs/J2-IN6: track 0.00 -> 6.47 mm
- net /Inputs/J2-IN12: track 0.00 -> 6.45 mm
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Other:
- board size 198 x 67.8 mm -> 173 x 67.8 mm
- board text added: "SUPORTES PCI METALTEX SP7 1x pé macho 9 mm 1x pé fêmea 9 mm 3x espaçadores 45 mm 1x espaçador 20 mm Comprimento total 173 mm Largura da placa 67,8 mm"
- board text removed: "SUPORTES PCI METALTEX SP7 1x pé macho 9 mm 1x pé fêmea 9 mm 4x espaçadores 45 mm Comprimento total 198 mm Largura da placa 67,8 mm"

Commit message: Update ESP-relay-16ch-V1.kicad_pcb
Parts:
- moved U21 3.86 mm to (145.4, 101.0)
- moved R50 2.54 mm to (138.4, 117.3)
- moved R53 2.54 mm to (142.2, 117.3)
- moved R56 2.54 mm to (146.1, 117.3)
- moved R11 2.54 mm to (88.9, 117.3)
- moved R23 2.54 mm to (104.1, 117.3)
- moved R26 2.54 mm to (108.0, 117.3)
- moved R29 2.54 mm to (111.8, 117.3)
- moved R41 2.54 mm to (127.0, 117.3)
- moved R14 2.54 mm to (92.7, 117.3)
- moved R17 2.54 mm to (96.5, 117.3)
- moved R20 2.54 mm to (100.3, 117.3)
- moved R32 2.54 mm to (115.6, 117.3)
- moved R35 2.54 mm to (119.4, 117.3)
- moved R38 2.54 mm to (123.2, 117.3)
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Routing:
- net GND: track 483.8 -> 381.8 mm, vias 45 -> 48
- net Net-(C22-Pad1): track 2.54 -> 56.7 mm
- net Net-(C16-Pad1): track 2.54 -> 52.9 mm
- net Net-(C26-Pad1): track 2.54 -> 51.8 mm
- net Net-(C21-Pad1): track 2.54 -> 46.3 mm
- net Net-(C15-Pad1): track 2.54 -> 44.0 mm
- net Net-(C25-Pad1): track 2.54 -> 42.8 mm
- net Net-(C14-Pad1): track 2.54 -> 37.7 mm
- net Net-(C20-Pad1): track 2.54 -> 36.6 mm
- net Net-(C24-Pad1): track 2.54 -> 35.0 mm
- net Net-(C13-Pad1): track 2.54 -> 32.8 mm
- net Net-(C19-Pad1): track 2.54 -> 29.8 mm
- net Net-(C12-Pad1): track 2.55 -> 28.0 mm
- net Net-(C18-Pad1): track 2.54 -> 25.3 mm
- net Net-(C23-Pad1): track 2.54 -> 24.9 mm
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
Commit message: Update ESP-relay-16ch-V1.kicad_pcb
Parts:
- moved R63 108.9 mm to (222.2, 46.5), turned to 90 degrees
- moved R64 106.7 mm to (221.0, 46.5), turned to 90 degrees
- moved J4 105.0 mm to (217.2, 33.7), turned to 0 degrees
- moved C31 97.6 mm to (207.0, 32.2), turned to 90 degrees
- moved C30 82.8 mm to (217.8, 46.4), turned to -90 degrees
- moved Q3 66.7 mm to (137.8, 37.9), turned to 90 degrees
- moved J2 65.9 mm to (126.3, 36.9)
- moved U19 62.4 mm to (132.1, 45.3), turned to 90 degrees
- moved C10 60.9 mm to (182.2, 35.7)
- moved C32 60.9 mm to (174.0, 44.0)
- moved C33 60.9 mm to (175.3, 43.7)
- moved C35 60.9 mm to (176.5, 35.1)
- moved C36 60.9 mm to (168.3, 40.5)
- moved C37 60.9 mm to (169.5, 40.5)
- moved C38 60.9 mm to (178.4, 40.8)
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Routing:
- net GND: track 381.8 -> 568.4 mm, vias 48 -> 78
- net /MCU/OUT1: track 1.27 -> 55.6 mm
- net /MCU/OUT2: track 1.27 -> 48.2 mm
- net /MCU/OUT3: track 1.27 -> 45.4 mm
- net /MCU/OUT4: track 1.27 -> 42.9 mm
- net /Inputs/IN16: track 1.79 -> 42.8 mm
- net /MCU/OUT5: track 1.27 -> 40.3 mm
- net /Inputs/IN15: track 1.79 -> 38.5 mm
- net /MCU/OUT9: track 1.27 -> 37.7 mm
- net /MCU/OUT6: track 1.27 -> 37.2 mm
- net /Inputs/IN13: track 1.79 -> 35.9 mm
- net /MCU/OUT7: track 1.27 -> 34.3 mm
- net /Inputs/IN14: track 1.79 -> 34.7 mm
- net /MCU/OUT8: track 1.27 -> 31.5 mm
- net /MCU/OUT10: track 1.27 -> 29.3 mm
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Other:
- board size 173 x 67.8 mm -> 148 x 67.8 mm
- board text added: "SUPORTES PCI METALTEX SP7 1x pé macho 9 mm 1x pé fêmea 9 mm 2x espaçadores 45 mm 2x espaçador 20 mm Comprimento total 148 mm Largura da placa 67,8 mm"
- board text removed: "SUPORTES PCI METALTEX SP7 1x pé macho 9 mm 1x pé fêmea 9 mm 3x espaçadores 45 mm 1x espaçador 20 mm Comprimento total 173 mm Largura da placa 67,8 mm"

Commit message: Dev updates
Parts:
- moved R60 44.6 mm to (188.1, 82.5), turned to 180 degrees
- moved D38 13.9 mm to (173.7, 30.0)
- moved R9 9.16 mm to (192.4, 30.4)
- moved Q2 9.16 mm to (194.7, 27.3)
- moved C10 9.16 mm to (187.3, 28.1)
- moved C9 9.16 mm to (189.2, 30.6)
- moved R8 9.16 mm to (191.1, 30.4)
- moved L3 9.16 mm to (184.6, 27.3)
- moved Q1 9.16 mm to (190.2, 27.3)
- moved C36 1.91 mm to (166.4, 40.5)
- moved C37 1.91 mm to (167.6, 40.5)
- moved C38 1.27 mm to (179.7, 40.8)
- moved R73 1.27 mm to (178.4, 40.5)
- moved C32 1.27 mm to (174.0, 45.2)
- moved C33 1.27 mm to (175.3, 44.9)
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Routing:
- net Net-(R71-Pad1): track 0.00 -> 5.87 mm
- net /LAN/EMAC_RX: track 0.00 -> 5.80 mm
- net /LAN/EMAC_MDIO: track 0.00 -> 5.67 mm
- net Net-(R72-Pad1): track 0.00 -> 5.09 mm
- net Net-(R70-Pad1): track 0.00 -> 4.69 mm
- net Net-(R65-Pad2): track 0.00 -> 3.67 mm
- net +3.3VLAN: track 0.00 -> 3.21 mm
- net Net-(C36-Pad1): track 0.00 -> 3.19 mm
- net /LAN/EMAC_RXD1: track 0.00 -> 3.03 mm
- net /LAN/EMAC_RXD0: track 0.00 -> 2.89 mm

Commit message: Dev updates
Parts:
- moved C35 61.4 mm to (201.9, 89.7)
- moved C36 61.4 mm to (191.8, 96.4)
- moved C37 61.4 mm to (193.0, 96.4)
- moved R73 61.4 mm to (203.8, 96.4)
- moved R74 61.4 mm to (195.6, 89.7)
- moved R76 61.4 mm to (200.7, 89.7)
- moved R77 61.4 mm to (196.8, 89.7)
- moved R78 61.4 mm to (198.1, 89.7)
- moved U24 61.4 mm to (198.7, 95.1)
- moved C33 61.4 mm to (200.7, 100.8)
- moved C34 61.4 mm to (193.7, 93.8)
- moved R65 61.4 mm to (195.6, 100.8)
- moved R66 61.4 mm to (196.8, 100.8)
- moved R67 61.4 mm to (198.1, 100.8)
- moved R68 61.4 mm to (204.5, 100.8)
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Routing:
- net +24V: track 37.5 -> 230.3 mm, vias 0 -> 16
- net +3.3V: track 36.7 -> 213.9 mm, vias 2 -> 19
- net /Inputs/IN1: track 1.80 -> 85.7 mm
- net /Inputs/IN2: track 1.80 -> 77.4 mm
- net /Inputs/IN3: track 1.80 -> 69.2 mm
- net GND: track 568.4 -> 631.3 mm
- net /Inputs/IN7: track 1.80 -> 64.3 mm
- net /Inputs/IN4: track 1.80 -> 60.9 mm
- net /Inputs/IN8: track 1.80 -> 56.0 mm
- net /Inputs/IN5: track 1.80 -> 52.6 mm
- net /Inputs/IN12: track 1.80 -> 49.0 mm
- net /Inputs/IN9: track 1.80 -> 47.8 mm
- net /Inputs/IN6: track 1.80 -> 43.6 mm
- net /Inputs/IN10: track 1.80 -> 39.5 mm
- net /Inputs/IN11: track 1.80 -> 31.3 mm
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Other:
- board text added: "O1"
- board text added: "O10"
- board text added: "O11"
- board text added: "O12"
- board text added: "O13"
- board text added: "O14"
- board text added: "O15"
- board text added: "O16"
- board text added: "O17"
- board text added: "O2"
- board text added: "O3"
- board text added: "O4"
- board text added: "O5"
- board text added: "O6"
- board text added: "O7"
- board text added: "O8"
- board text added: "O9"

Commit message: Dev updates
Parts:
- moved F1 59.8 mm to (90.7, 76.8), turned to 180 degrees
- moved D38 57.0 mm to (187.5, 92.4), turned to 180 degrees
- moved C27 47.2 mm to (163.2, 81.4), turned to 90 degrees
- moved C28 43.1 mm to (163.2, 77.8)
- moved D5 37.3 mm to (164.5, 72.8), turned to 90 degrees
- moved U19 34.6 mm to (158.2, 76.2), turned to 180 degrees
- moved Q3 27.5 mm to (154.3, 68.3)
- moved C31 20.3 mm to (184.8, 74.1)
- moved R64 9.65 mm to (168.8, 88.9), turned to 180 degrees
- moved R74 2.12 mm to (193.8, 90.8), turned to 180 degrees
- moved R78 1.94 mm to (196.3, 88.9), turned to 180 degrees
- moved R63 1.40 mm to (181.1, 88.9), turned to 180 degrees
- moved J2 1.40 mm to (160.6, 67.1)
- moved R76 1.37 mm to (199.9, 90.8), turned to 0 degrees
- moved U21 1.27 mm to (155.8, 100.1)
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Routing:
- net GND: track 631.3 -> 695.9 mm
- net Net-(U19-Pad3): track 0.00 -> 58.4 mm
- net Net-(U19-Pad2): track 0.00 -> 55.6 mm
- net /LAN/EMAC_MDC: track 0.00 -> 45.8 mm
- net /LAN/RD+: track 0.00 -> 40.8 mm
- net /LAN/EMAC_TXD1: track 0.00 -> 37.9 mm, vias 0 -> 2
- net /LAN/TD+: track 0.00 -> 33.3 mm
- net /LAN/EMAC_TXEN: track 0.00 -> 32.2 mm
- net /LAN/RD-: track 0.00 -> 31.5 mm
- net /LAN/TD-: track 0.00 -> 31.1 mm
- net /LAN/EMAC_TXD0: track 0.00 -> 28.9 mm
- net +3.3V: track 213.9 -> 234.3 mm
- net Net-(C31-Pad1): track 0.00 -> 19.2 mm
- net /LAN/EMAC_MDIO: track 0.00 -> 18.8 mm
- net Net-(Q3-Pad1): track 0.00 -> 13.2 mm
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