File: V2/ESP-24v-16ch-V2-power.kicad_sch (KiCad schematic)
At the start: 34 parts, among them J10 USB, J9 VIN, Q1 WPM2015-3/TR, Q2 LMUN2211LT1G, U1 SY8089A1AAC, U2 TX4138

Commit message: Add interrupt pins
Parts:
- removed J10: USB, Tales:USB_Micro-B_Amphenol_10104110_Horizontal, symbol Connector:USB_B_Micro
- removed J9: VIN, Tales:TerminalBlock_Phoenix_MKDS-3-2-5.08_1x02_P5.08mm_Horizontal, symbol Connector_Generic:Conn_01x02
Connections:
- net USB_VBUS: now reaches D3.2 (A)
- net VIN: now reaches D1.2 (A)
- no-connect marks 3 -> 2
Changed lines of the file:
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@@
   (junction (at 78.74 124.46) (diameter 0) (color 0 0 0 0)
-  )
-  (junction (at 38.1 102.87) (diameter 0) (color 0 0 0 0)
   )
   (junction (at 100.33 137.16) (diameter 0) (color 0 0 0 0)
@@
   (no_connect (at 153.67 46.99))
   (no_connect (at 153.67 44.45))
-  (no_connect (at 45.72 96.52))
   (wire (pts (xy 227.33 46.99) (xy 252.73 46.99))
     (stroke (width 0) (type default))
@@
     (stroke (width 0) (type default))
   )
-  (wire (pts (xy 45.72 91.44) (xy 63.5 91.44))
-    (stroke (width 0) (type default))
-  )
   (wire (pts (xy 54.61 36.83) (xy 78.74 36.83))
     (stroke (width 0) (type default))
@@
     (stroke (width 0) (type default))
   )
-  (wire (pts (xy 45.72 86.36) (xy 52.07 86.36))
+  (wire (pts (xy 39.37 86.36) (xy 52.07 86.36))
     (stroke (width 0) (type default))
   )
@@
     (stroke (width 0) (type default))
   )
-  (wire (pts (xy 38.1 101.6) (xy 38.1 102.87))
-    (stroke (width 0) (type default))
-  )
   (wire (pts (xy 173.99 46.99) (xy 175.26 46.99))
     (stroke (width 0) (type default))
@@
     (stroke (width 0) (type default))
   )
-  (wire (pts (xy 38.1 102.87) (xy 38.1 104.14))
-    (stroke (width 0) (type default))
-  )
   (wire (pts (xy 158.75 124.46) (xy 180.34 124.46))
     (stroke (width 0) (type default))
@@
     (stroke (width 0) (type default))
   )
-  (wire (pts (xy 35.56 101.6) (xy 35.56 102.87))
-    (stroke (width 0) (type default))
-  )
   (wire (pts (xy 186.69 36.83) (xy 186.69 39.37))
     (stroke (width 0) (type default))
@@
     (stroke (width 0) (type default))
   )
-  (wire (pts (xy 45.72 93.98) (xy 63.5 93.98))
-    (stroke (width 0) (type default))
-  )
   (wire (pts (xy 63.5 83.82) (xy 63.5 86.36))
     (stroke (width 0) (type default))
@@
   )
   (wire (pts (xy 78.74 124.46) (xy 78.74 128.27))
-    (stroke (width 0) (type default))
-  )
-  (wire (pts (xy 35.56 102.87) (xy 38.1 102.87))
     (stroke (width 0) (type default))
   )
@@
     (effects (font (size 1.5 1.5)) (justify left bottom))
   )
-  (hierarchical_label "USB_D-" (shape output) (at 63.5 93.98 0) (fields_autoplaced)
-    (effects (font (size 1.27 1.27)) (justify left))
+  (hierarchical_label "GND" (shape input) (at 39.37 39.37 180) (fields_autoplaced)
+    (effects (font (size 1.27 1.27)) (justify right))
+  )
+  (hierarchical_label "USB_VBUS" (shape input) (at 39.37 86.36 180) (fields_autoplaced)
+    (effects (font (size 1.27 1.27)) (justify right))
+  )
+  (hierarchical_label "VIN" (shape input) (at 39.37 36.83 180) (fields_autoplaced)
+    (effects (font (size 1.27 1.27)) (justify right))
   )
   (hierarchical_label "PHY_PWR" (shape input) (at 218.44 158.75 0) (fields_autoplaced)
-    (effects (font (size 1.27 1.27)) (justify left))
-  )
-  (hierarchical_label "USB_D+" (shape output) (at 63.5 91.44 0) (fields_autoplaced)
     (effects (font (size 1.27 1.27)) (justify left))
   )
@@
     )
   )
-  (symbol (lib_id "Connector:USB_B_Micro") (at 38.1 91.44 0) (unit 1)
-    (in_bom yes) (on_board yes) (dnp no)
-    (property "Reference" "J10" (at 38.1 76.2 0)
-      (effects (font (size 1.27 1.27)))
-    )
-    (property "Value" "USB" (at 38.1 78.74 0)
-      (effects (font (size 1.27 1.27)))
-    )
-    (property "Footprint" "Tales:USB_Micro-B_Amphenol_10104110_Horizontal" (at 41.91 92.71 0)
-      (effects (font (size 1.27 1.27)) hide)
-    )
-    (property "Datasheet" "~" (at 41.91 92.71 0)
-      (effects (font (size 1.27 1.27)) hide)
-    )
-    (property "Case" "~" (at 38.1 91.44 0)
-      (effects (font (size 1.27 1.27)) hide)
-    )
-    (property "JLCPCB BOM" "1" (at 38.1 91.44 0)
-      (effects (font (size 1.27 1.27)) hide)
-    )
-    (property "LCSC Part #" "C132563" (at 38.1 81.28 0)
-      (effects (font (size 1.27 1.27)))
-    )
-    (property "Mfr" "Amphenol" (at 38.1 91.44 0)
-      (effects (font (size 1.27 1.27)) hide)
-    )
-    (property "Mfr PN" "10118194-0001LF" (at 38.1 91.44 0)
-      (effects (font (size 1.27 1.27)) hide)
-    )
-    (property "Technology" "~" (at 38.1 91.44 0)
-      (effects (font (size 1.27 1.27)) hide)
-    )
-    (property "Vendor" "JLCPCB" (at 38.1 91.44 0)
-      (effects (font (size 1.27 1.27)) hide)
-    )
-    (property "Vendor PN" "C132563" (at 38.1 91.44 0)
-      (effects (font (size 1.27 1.27)) hide)
-    )
-    (pin "1")
-    (pin "2")
-    (pin "3")
-    (pin "4")
-    (pin "5")
-    (pin "6")
-    (instances
-      (project "ESP-24v-16ch-V2"
-        (path "/2bc5a21a-1d79-419d-a592-6852cc07b00a/7b388c9c-6faf-4681-b727-510de2ea001e"
-          (reference "J10") (unit 1)
-        )
-      )
-    )
-  )
   (symbol (lib_id "Device:Fuse_Small") (at 63.5 81.28 90) (unit 1)
     (in_bom yes) (on_board yes) (dnp no)
@@
         (path "/2bc5a21a-1d79-419d-a592-6852cc07b00a/7b388c9c-6faf-4681-b727-510de2ea001e"
           (reference "Q1") (unit 1)
-        )
-      )
-    )
-  )
-  (symbol (lib_id "Connector_Generic:Conn_01x02") (at 34.29 36.83 0) (mirror y) (unit 1)
-    (in_bom yes) (on_board yes) (dnp no) (fields_autoplaced)
-    (property "Reference" "J9" (at 34.29 30.48 0)
-      (effects (font (size 1.27 1.27)))
-    )
-    (property "Value" "VIN" (at 34.29 33.02 0)
-      (effects (font (size 1.27 1.27)))
-    )
-    (property "Footprint" "Tales:TerminalBlock_Phoenix_MKDS-3-2-5.08_1x02_P5.08mm_Horizontal" (at 34.29 36.83 0)
-      (effects (font (size 1.27 1.27)) hide)
-    )
-    (property "Datasheet" "~" (at 34.29 36.83 0)
-      (effects (font (size 1.27 1.27)) hide)
-    )
-    (property "Case" "~" (at 34.29 36.83 0)
-      (effects (font (size 1.27 1.27)) hide)
-    )
-    (property "JLCPCB BOM" "0" (at 34.29 36.83 0)
-      (effects (font (size 1.27 1.27)) hide)
-    )
-    (property "Mfr" "Conexel" (at 34.29 36.83 0)
-      (effects (font (size 1.27 1.27)) hide)
-    )
-    (property "Mfr PN" "1x LM 5.08/02/90 3.5SN OR BX" (at 34.29 36.83 0)
-      (effects (font (size 1.27 1.27)) hide)
-    )
-    (property "Technology" "~" (at 34.29 36.83 0)
-      (effects (font (size 1.27 1.27)) hide)
-    )
-    (property "Vendor" "Conexel" (at 34.29 36.83 0)
-      (effects (font (size 1.27 1.27)) hide)
-    )
-    (property "Vendor PN" "1x 1716080000" (at 34.29 36.83 0)
-      (effects (font (size 1.27 1.27)) hide)
-    )
-    (property "LCSC Part #" "~" (at 34.29 36.83 0)
-      (effects (font (size 1.27 1.27)) hide)
-    )
-    (pin "1")
-    (pin "2")
-    (instances
-      (project "ESP-24v-16ch-V2"
-        (path "/2bc5a21a-1d79-419d-a592-6852cc07b00a/7b388c9c-6faf-4681-b727-510de2ea001e"
-          (reference "J9") (unit 1)
         )
       )
@@
         )
       )
-    )
-  )
-  (symbol (lib_id "power:GND") (at 38.1 104.14 0) (unit 1)
-    (in_bom yes) (on_board yes) (dnp no)
-    (property "Reference" "#PWR0307" (at 38.1 110.49 0)
-      (effects (font (size 1.27 1.27)) hide)
-    )
-    (property "Value" "GNDREF" (at 38.227 108.5342 0)
-      (effects (font (size 1.27 1.27)) hide)
-    )
-    (property "Footprint" "" (at 38.1 104.14 0)
-      (effects (font (size 1.27 1.27)) hide)
-    )
-    (property "Datasheet" "" (at 38.1 104.14 0)
-      (effects (font (size 1.27 1.27)) hide)
-    )
-    (pin "1")
-    (instances
-      (project "ESP-24v-16ch-V2"
-        (path "/2bc5a21a-1d79-419d-a592-6852cc07b00a/7b388c9c-6faf-4681-b727-510de2ea001e"
-          (reference "#PWR0307") (unit 1)
-        )
-      )

Commit message: Adjustments for fabrication.
Parts:
- F1: footprint Tales:Fuse_0402_1005Metric -> Fuse:Fuse_1206_3216Metric; Case 0402 -> 1206; LCSC Part # C136320 -> C140466; Mfr JDT -> Xucheng Elec; Mfr PN JFC0402-0500FS -> 12F.05000063AG12S1B02; Vendor PN C136320 -> C140466
Changed lines of the file:
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@@
       (effects (font (size 1.27 1.27)) (justify right))
     )
-    (property "Footprint" "Tales:Fuse_0402_1005Metric" (at 63.5 81.28 0)
+    (property "Footprint" "Fuse:Fuse_1206_3216Metric" (at 63.5 81.28 0)
       (effects (font (size 1.27 1.27)) hide)
     )
@@
       (effects (font (size 1.27 1.27)) hide)
     )
-    (property "LCSC Part #" "C136320" (at 66.04 81.28 90)
+    (property "LCSC Part #" "C140466" (at 66.04 81.28 90)
       (effects (font (size 1.27 1.27)) (justify right))
     )
-    (property "Mfr" "JDT" (at 63.5 81.28 0)
+    (property "Mfr" "Xucheng Elec" (at 63.5 81.28 0)
       (effects (font (size 1.27 1.27)) hide)
     )
-    (property "Mfr PN" "JFC0402-0500FS" (at 63.5 81.28 0)
+    (property "Mfr PN" "12F.05000063AG12S1B02" (at 63.5 81.28 0)
       (effects (font (size 1.27 1.27)) hide)
     )
@@
       (effects (font (size 1.27 1.27)) hide)
     )
-    (property "Vendor PN" "C136320" (at 63.5 81.28 0)
+    (property "Vendor PN" "C140466" (at 63.5 81.28 0)
       (effects (font (size 1.27 1.27)) hide)
     )
-    (property "Case" "0402" (at 63.5 81.28 0)
+    (property "Case" "1206" (at 63.5 81.28 0)
       (effects (font (size 1.27 1.27)) hide)
     )

Commit message: Upgrade USB-Micro-B to Type-C connector.
Parts:
- added C39: 1uF/50V/0603, Tales:C_0603_1608Metric, symbol Device:C_Small
- added C40: 0,1uF/50V/0402, Tales:C_0402_1005Metric, symbol Device:C_Small
- added J1: VIN, Tales:TerminalBlock_Phoenix_MKDS-3-2-5.08_1x02_P5.08mm_Horizontal, symbol Connector_Generic:Conn_01x02
- added J2: USB_C_Receptacle_USB2.0, Tales:USB_C_Receptacle_JAE_DX07S024WJ1R350, symbol Connector:USB_C_Receptacle_USB2.0
- added R131, R132: 5k1/62,5mW/0402, Tales:R_0402_1005Metric, symbol Device:R_US
Connections:
- net GND: now also C39.2, C40.2, J1.2 (Pin_2), J2.A1 (GND), J2.A12 (GND), J2.B1 (GND), J2.B12 (GND), J2.S1 (SHIELD), R131.2, R132.2
- net USB_VBUS: no longer names the net of D3.2 (A)
- net USB_VBUS: now also C39.1, C40.1, J2.A4 (VBUS), J2.A9 (VBUS), J2.B4 (VBUS), J2.B9 (VBUS)
- net VIN: no longer names the net of D1.2 (A)
- net VIN: now also J1.1 (Pin_1)
- new net: J2.A5 (CC1), R131.1
- new net: J2.B5 (CC2), R132.1
- new net USB_D+: J2.A6 (D+), J2.B6 (D+)
- new net USB_D-: J2.A7 (D-), J2.B7 (D-)
- no-connect marks 2 -> 4
Other:
- moved on the sheet: C1, C3, C5, L1, R2, R3, U1

Commit message: Update documentation in the schematics
Other:
- note added: "24VDC"
Changed lines of the file:
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@@
     (title "ESP 16x 24VDC Input 16x 24VDC Output Module")
     (date "2023-05-05")
-    (rev "V1")
+    (rev "V2")
   )
   (junction (at 180.34 46.99) (diameter 0) (color 0 0 0 0)
@@
     (effects (font (size 1.5 1.5)) (justify left bottom))
   )
+  (text "24VDC" (at 20.32 39.37 0)
+    (effects (font (size 2.5 2.5)) (justify left bottom))
+  )
   (text "R2" (at 223.52 78.74 0)
