File: V2/ESP-24v-16ch-V2-outputs-1.kicad_sch (KiCad schematic)
At the start: 80 parts, among them Q10 MMBT2222A/SOT-23-3, Q11 MMBT2222A/SOT-23-3, Q12 MMBT2222A/SOT-23-3, Q13 MMBT2222A/SOT-23-3, Q14 MMBT2222A/SOT-23-3, Q15 MMBT2222A/SOT-23-3, Q16 MMBT2222A/SOT-23-3, Q17 MMBT2222A/SOT-23-3, Q18 MMBT2222A/SOT-23-3, Q19 MMBT2222A/SOT-23-3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

Commit message: Add interrupt pins
Parts:
- renumbered D71 to D39, D72 to D40, D73 to D41, D74 to D42, D75 to D43, D76 to D44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
