File: V2/esp-24v-16ch-v2-expanders.kicad_sch (KiCad schematic)
At the start: 4 parts, among them U25 MCP23017_SS, U27 MCP23017_SS

Commit message: Update Kicad 8
Parts:
- renumbered U25 to U6, U27 to U7
