File: V2/esp-24v-16ch-v2-power.kicad_sch (KiCad schematic)
At the start: 38 parts, among them Q1 WPM2015-3/TR, Q2 LMUN2211LT1G, U1 SY8089A1AAC, U2 TX4138

Commit message: Adjusted footprint
Parts:
- L1: footprint Tales:L_3x3_h1.5 -> Tales:L_3x3mm_h1.5mm
Changed lines of the file:
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@@
       (effects (font (size 1.27 1.27)))
     )
-    (property "Footprint" "Tales:L_3x3_h1.5" (at 68.58 144.78 0)
+    (property "Footprint" "Tales:L_3x3mm_h1.5mm" (at 68.58 144.78 0)
       (effects (font (size 1.27 1.27)) hide)
     )

Commit message: Update Kicad 8
Parts:
- gave numbers to parts that had none: 2
