File: V3/ESP-24v-16ch-V3-inputs-1.kicad_sch (KiCad schematic)
At the start: 100 parts, among them U10 OR-3H4-4, U11 OR-3H4-4, U8 OR-3H4-4, U9 OR-3H4-4

Commit message: Replaced R16 and R17 for a R-Pack
Parts:
- R33, R34, R35, R36, R45, R46, R47, R48, R57, R58, R59, R60, R69, R70, R71, R72: value 5,6k/0,1W/0603 -> 6,8k/0,1W/0603; LCSC Part # C23189 -> C23212; Mfr PN 0603WAF5601T5E -> 0603WAF6801T5E; Vendor PN C23189 -> C23212
Other:
- note added: "INPUT LEDS Target current: 3mA V_{F} @ 3mA = 2,85V 24V - 2,85V = R * 0,003A R = 7050 ohm If R = 6,8kohm --> I = 3,11mA --> OK Power dissipated at the resistor P = 6800 * 0,00311^{2} = 65,8mW Use 0,1W/0603 resistor"
- note added: "OPTO INPUT LED current 24V - 9,1V -1,2V = 13,7V 13,7V / 1800R = 7,62mA -> OK Power dissipated on series resistor 1800 x 0,00762^{2} = 0,1045 104,5mW - use 125mW resistor"
- note added: "OPTO OUTPUT CTR @ i=8mA and Vce = 0,4V ~= 150% Output current can reach 12mA Maximum current at opto output 3,3V - 0,4V = 2,9V 2,9V / 2200R = 1,32mA -> OK"
- note removed: "ENTRADA OPTO Corrente na entrada 24V - 9,1V -1,2V = 13,7V 13,7V / 1800R = 7,62mA Potência dissipada no resistor série 1800 x SQ(0,00762) = 0,1045 104,5mW - usar resistor 125mW"
- note removed: "SAÍDA OPTO CTR opto com i=8mA e Vce = 0,4V ~= 150% Corrente na saída do opto pode chegar a 12mA Corrente máxima prevista na saída do opto 3,3V - 0,4V = 2,9V 2,9V / 2200R = 1,32mA"
