File: V3/ESP-24v-16ch-V3.kicad_pcb (KiCad board)
At the start: 2 copper layers, 138 x 67.8 mm, 268 parts, among them J1 VIN, J2 USB_C_Receptacle_USB2.0, J3 Conn_01x08, J4 Conn_01x08, J5 Conn_01x08, J6 Conn_01x08, J7 ETHERNET, Q1 WPM2015-3/TR, Q10 MMBT2222A/SOT-23-3, Q11 MMBT2222A/SOT-23-3, Q12 MMBT2222A/SOT-23-3, Q13 MMBT2222A/SOT-23-3, Q14 MMBT2222A/SOT-23-3, Q15 MMBT2222A/SOT-23-3, Q16 MMBT2222A/SOT-23-3, Q17 MMBT2222A/SOT-23-3, Q18 MMBT2222A/SOT-23-3, Q19 MMBT2222A/SOT-23-3, Q2 LMUN2211LT1G, Q3 UMH3N, Q4 MMBT2222A/SOT-23-3, Q5 MMBT2222A/SOT-23-3, Q6 MMBT2222A/SOT-23-3, Q7 MMBT2222A/SOT-23-3, Q8 MMBT2222A/SOT-23-3, Q9 MMBT2222A/SOT-23-3, SW1 RESET, U1 SY8089A1AAC, U10 OR-3H4-4, U11 OR-3H4-4, U2 TX4138, U3 CH340C, U4 ESP32-WROOM-32UE-N16, U5 LAN8710A, U6 MCP23017_SS, U7 MCP23017_SS, U8 OR-3H4-4, U9 OR-3H4-4

Commit message: Connectors rotated 180deg
Routing:
- net Net-(D30-A): track 79.6 -> 76.1 mm
- net Net-(D29-A): track 76.2 -> 72.7 mm
- net Net-(D28-A): track 72.8 -> 69.5 mm
- net Net-(D27-A): track 68.7 -> 65.5 mm
Other:
- board text added: "ESP-24V-16CH-V3"
- board text removed: "ESP-24V-16CH-V2"
