File: V3/esp-24v-16ch-v3-expanders.kicad_sch (KiCad schematic)
At the start: 4 parts, among them U6 MCP23017_SS, U7 MCP23017_SS

Commit message: working on v3
Parts:
- R31, R32: value 1k/62,5mW/0402 -> 1k/62,5mW
Changed lines of the file:
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@@
 		(on_board yes)
 		(dnp no)
-		(fields_autoplaced yes)
 		(property "Reference" "U6"
-			(at 62.9159 74.93 0)
+			(at 63.5 72.39 0)
 			(effects
 				(font
@@
 		)
 		(property "Value" "MCP23017_SS"
-			(at 62.9159 77.47 0)
+			(at 63.5 74.93 0)
 			(effects
 				(font
@@
 		)
 		(property "LCSC Part #" "C558584"
-			(at 60.96 101.6 0)
-			(effects
-				(font
-					(size 1.27 1.27)
-				)
-				(hide yes)
+			(at 63.5 77.47 0)
+			(effects
+				(font
+					(size 1.27 1.27)
+				)
+				(justify left)
 			)
 		)
@@
 			)
 		)
-		(property "Value" "1k/62,5mW/0402"
+		(property "Value" "1k/62,5mW"
 			(at 20.32 106.68 0)
 			(effects
@@
 		)
 		(property "LCSC Part #" "C11702"
-			(at 25.4 97.79 0)
-			(effects
-				(font
-					(size 1.27 1.27)
-				)
-				(hide yes)
+			(at 20.32 109.22 0)
+			(effects
+				(font
+					(size 1.27 1.27)
+				)
+				(justify left)
 			)
 		)
@@
 		(on_board yes)
 		(dnp no)
-		(fields_autoplaced yes)
 		(property "Reference" "U7"
-			(at 182.2959 74.93 0)
+			(at 182.88 72.39 0)
 			(effects
 				(font
@@
 		)
 		(property "Value" "MCP23017_SS"
-			(at 182.2959 77.47 0)
+			(at 182.88 74.93 0)
 			(effects
 				(font
@@
 		)
 		(property "LCSC Part #" "C558584"
-			(at 180.34 101.6 0)
-			(effects
-				(font
-					(size 1.27 1.27)
-				)
-				(hide yes)
+			(at 182.88 77.47 0)
+			(effects
+				(font
+					(size 1.27 1.27)
+				)
+				(justify left)
 			)
 		)
@@
 			)
 		)
-		(property "Value" "1k/62,5mW/0402"
+		(property "Value" "1k/62,5mW"
 			(at 142.24 106.68 0)
 			(effects
@@
 		)
 		(property "LCSC Part #" "C11702"
-			(at 147.32 97.79 0)
-			(effects
-				(font
-					(size 1.27 1.27)
-				)
-				(hide yes)
-			)
-		)
+			(at 142.24 109.22 0)
+			(effects
+				(font
+					(size 1.27 1.27)
+				)
+				(justify left)
+			)
+		)

Commit message: Added temperature sensor
Parts:
- added C41: 100nF/50V, Tales:C_0402_1005Metric, symbol Device:C_Small
- added U12: AHT20, Tales:DFN-6-3x3mm_P1mm, symbol Tales:AHT20
Connections:
- net +3.3V: now also C41.1, U12.2 (VDD)
- net GND: now also C41.2, U12.5 (GND)
- net I2C_SCL: now also U12.3 (SCL)
- net I2C_SDA: now also U12.4 (SDA)
Other:
- note added: "TEMP/HUMID ADDRESS 0x38"
- moved on the sheet: R32, U7

Commit message: Preparations for fabrication
Parts:
- U12: Case (none) -> DFN-6; JLCPCB BOM (none) -> 1; LCSC Part # (none) -> C2757850; Mfr (none) -> Aosong; Mfr PN (none) -> AHT20; Vendor (none) -> JLCPCB; Vendor PN (none) -> C2757850
Changed lines of the file:
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@@
+			)
+		)
+		(property "Case" "DFN-6"
+			(at 231.14 99.06 0)
+			(effects
+				(font
+					(size 1.27 1.27)
+				)
+				(hide yes)
+			)
+		)
+		(property "JLCPCB BOM" "1"
+			(at 231.14 99.06 0)
+			(effects
+				(font
+					(size 1.27 1.27)
+				)
+				(hide yes)
+			)
+		)
+		(property "LCSC Part #" "C2757850"
+			(at 231.14 99.06 0)
+			(effects
+				(font
+					(size 1.27 1.27)
+				)
+				(hide yes)
+			)
+		)
+		(property "Mfr" "Aosong"
+			(at 231.14 99.06 0)
+			(effects
+				(font
+					(size 1.27 1.27)
+				)
+				(hide yes)
+			)
+		)
+		(property "Mfr PN" "AHT20"
+			(at 231.14 99.06 0)
+			(effects
+				(font
+					(size 1.27 1.27)
+				)
+				(hide yes)
+			)
+		)
+		(property "Technology" "~"
+			(at 231.14 99.06 0)
+			(effects
+				(font
+					(size 1.27 1.27)
+				)
+				(hide yes)
+			)
+		)
+		(property "Vendor" "JLCPCB"
+			(at 231.14 99.06 0)
+			(effects
+				(font
+					(size 1.27 1.27)
+				)
+				(hide yes)
+			)
+		)
+		(property "Vendor PN" "C2757850"
+			(at 231.14 99.06 0)
+			(effects
+				(font
+					(size 1.27 1.27)
+				)
+				(hide yes)
 			)
 		)
