File: V3/esp-24v-16ch-v3-power.kicad_sch (KiCad schematic)
At the start: 38 parts, among them J1 VIN, J2 USB_C_Receptacle_USB2.0, Q1 WPM2015-3/TR, Q2 LMUN2211LT1G, U1 SY8089A1AAC, U2 TX4138

Commit message: working on v3
Parts:
- removed F1: 500mA, Tales:Fuse_1206_3216Metric, symbol Device:Fuse_Small
- removed J2: USB_C_Receptacle_USB2.0, Tales:USB_C_Receptacle_JAE_DX07S024WJ1R350, symbol Connector:USB_C_Receptacle_USB2.0
- added F1: 33V/500mA, Tales:R_1206_3216Metric, symbol Device:Polyfuse
- added J2: USB_C_Receptacle_USB2.0, Tales:USB_C_Receptacle_GCT_USB4105-xx-A_16P_TopMnt_Horizontal, symbol Tales:USB_C_Receptacle_USB2.0
- C1: value 10uF/50V/1206 -> 10uF/10V; footprint Tales:C_1206_3216Metric -> Tales:C_0603_1608Metric; Case 1206/3216 -> 0603/1608; LCSC Part # C13585 -> C19702; Mfr PN CL31A106KBHNNNE -> CL10A106KP8NNNC; Package (none) -> 0603/1608; Vendor PN C13585 -> C19702
- C10: value 470uF/16V/10x10 -> 470uF/16V; footprint Tales:CP_Elec_10x10 -> Tales:CP_Elec_8x10.5; Case 10x10 -> 8x10,5; LCSC Part # C249930 -> C96179; Mfr Lelon -> Semtech; Mfr PN VZH471M1CTR-1010 -> CS1C471M-CRF10; Package (none) -> D8xL10.5mm; Vendor PN C249930 -> C96179
- C2: value 47uF/35V/6,3x5,4 -> 47uF/35V
- C3: value 22pF/50V/0603 -> 22pF/50V; footprint Tales:C_0603_1608Metric -> Tales:C_0402_1005Metric; Case 0603/1608 -> 0402/1005; LCSC Part # C1653 -> C1555; Mfr Samsung -> FH; Mfr PN CL10C220JB8NNNC -> 0402CG220J500NT; Package (none) -> 0402/1005; Technology Ceramic -> Ceramic C0G; Vendor PN C1653 -> C1555
- C39: value 1uF/50V/0603 -> 1uF/25V; footprint Tales:C_0603_1608Metric -> Tales:C_0402_1005Metric; Case 0603/1608 -> 0402/1005; LCSC Part # C15849 -> C52923; Mfr PN CL10A105KB8NNNC -> CL05A105KA5NQNC; Package (none) -> 0402/1005; Vendor PN C15849 -> C52923
- C4: value 0,1uF/50V/0805 -> 0,1uF/50V; footprint Tales:C_0805_2012Metric -> Tales:C_0402_1005Metric; Case 0805/2012 -> 0402/1005; LCSC Part # C49678 -> C307331; Mfr Yageo -> Samsung; Mfr PN CC0805KRX7R9BB104 -> CL05B104KB54PNC; Package (none) -> 0402/1005; Technology Ceramic -> Ceramic X7R; Vendor PN C49678 -> C307331
- C40: value 0,1uF/50V/0402 -> 0,1uF/50V; Package (none) -> 0402/1005
- C5: value 10uF/50V/1206 -> 22uF/10V; LCSC Part # C13585 -> C5672; Mfr PN CL31A106KBHNNNE -> CL31A226KPHNNNE; Package (none) -> 1206/3216; Vendor PN C13585 -> C5672
- C6: value 10uF/10V/0603 -> 22uF/10V; footprint Tales:C_0603_1608Metric -> Tales:C_1206_3216Metric; Case 0603/1608 -> 1206/3216; LCSC Part # C19702 -> C5672; Mfr PN CL10A106KP8NNNC -> CL31A226KPHNNNE; Package (none) -> 1206/3216; Vendor PN C19702 -> C5672
- C7: value 0,1uF/50V/0805 -> 100nF/100V; LCSC Part # C49678 -> C28233; Mfr Yageo -> Samsung; Mfr PN CC0805KRX7R9BB104 -> CL21B104KCFNNNE; Package (none) -> 0805/2012; Technology Ceramic -> Ceramix X7R; Vendor PN C49678 -> C28233
- C8: value 12pF/50V/0603 -> 12pF/50V
- C9: value 10uF/10V/0603 -> 10uF/10V
- D1: value SM4007PL/SOD-123 -> SM4007PL
- D2: value GREEN/0603 -> GREEN; Case 0603 -> 0603/1608
- D3: value B5819W -> SS34; footprint Tales:D_SOD-123 -> Tales:D_SMA; Case SOD-123 -> SMA; LCSC Part # C8598 -> C8678; Mfr Jiangsu -> Microdiode; Mfr PN B5819W -> SS34; Vendor PN C8598 -> C8678
- R1: value 5,6k/0,1W/0603 -> 5,6k/0,1W
- R131, R132: value 5k1/62,5mW/0402 -> 5,1k/62,5mW; LCSC Part # C319557 -> C105872; Mfr Viking Tech -> YAGEO; Mfr PN AR02DTD5101 -> RC0402FR-075K1L; Package (none) -> 0402/1005; Technology (none) -> 1%; Vendor PN C319557 -> C105872
- R2: value 100k/0,125W/0805 -> 100k/0,125W
- R3: value 22,1k/0,125W/0805 -> 22,1k/0,125W
- R4: value 30mR/0,250W/0805 -> 30mR/333mW; footprint Tales:R_0805_2012Metric -> Tales:R_1206_3216Metric; Case 0805/2012 -> 1206/3216; LCSC Part # C247605 -> C473665; Mfr Uniroyal -> UNI-ROYAL(Uniroyal Elec); Mfr PN 0805W4F300MT5E -> 1206W3F300MT5E; Package (none) -> 1206/3216; Technology (none) -> 1%; Vendor PN C247605 -> C473665
- R5: value 5R1/0,125W/0805 -> 5,1R/100mW; footprint Tales:R_0805_2012Metric -> Tales:R_0603_1608Metric; Case 0805/2012 -> 0603/1608; LCSC Part # C17724 -> C25197; Mfr Uniroyal -> UNI-ROYAL(Uniroyal Elec); Mfr PN 0805W8F510KT5E -> 0603WAF510KT5E; Package (none) -> 0603/1608; Technology (none) -> 1%; Vendor PN C17724 -> C25197
- R6: value 10k/62,5mW/0402 -> 10k/62,5mW; LCSC Part # C25744 -> C60490; Mfr Uniroyal -> Yageo; Mfr PN 0402WGF1002TCE -> RC0402FR-0710KL; Package (none) -> 0402/1005; Technology (none) -> 1%; Vendor PN C25744 -> C60490
- R7: value 1k/62,5mW/0402 -> 1k/62,5mW
- R8: value 300k/0,125W/0805 -> 300k/100mW; footprint Tales:R_0805_2012Metric -> Tales:R_0603_1608Metric; Case 0805/2012 -> 0603/1608; LCSC Part # C17616 -> C23024; Mfr Uniroyal -> UNI-ROYAL(Uniroyal Elec); Mfr PN 0805W8F3003T5E -> 0603WAF3003T5E; Package (none) -> 0603/1608; Technology (none) -> 1%; Vendor PN C17616 -> C23024
- R9: value 52,3k/0,125W/0805 -> 52,3k/100mW; footprint Tales:R_0805_2012Metric -> Tales:R_0603_1608Metric; Case 0805/2012 -> 0603/1608; LCSC Part # C17740 -> C185323; Mfr Uniroyal -> Yageo; Mfr PN 0805W8F5232T5E -> RC0603FR-0752K3L; Package (none) -> 0603/1608; Technology (none) -> 1%; Vendor PN C17740 -> C185323
Connections:
- net +5V: now also F1.1
- net GND: now also J2.A1 (GND), J2.A12 (GND), J2.B1 (GND), J2.B12 (GND), J2.S1 (SHIELD)
- net USB_D+: now also J2.A6 (D+), J2.B6 (D+)
- net USB_D-: now also J2.A7 (D-), J2.B7 (D-)
- net at C39.1, C40.1, D3.2 (A): now also J2.A4 (VBUS), J2.A9 (VBUS), J2.B4 (VBUS), J2.B9 (VBUS)
- net at D3.1 (K): now also F1.2
- net at R131.1: now also J2.A5 (CC1)
- net at R132.1: now also J2.B5 (CC2)
Other:
- moved on the sheet: C2

Commit message: Update esp-24v-16ch-v3-power.kicad_sch
Parts:
- J1: footprint Tales:TerminalBlock_Phoenix_MKDS-3-2-5.08_1x02_P5.08mm_Horizontal -> Tales:TerminalBlock_Dibo_DB142V-5.08-2P_1x02_P5.08mm_Vertical; JLCPCB BOM 0 -> 1; LCSC Part # (none) -> C2898699; Mfr Conexel -> Dorabo; Mfr PN 1x LM 5.08/02/90 3.5SN OR BX -> DB142V-5.08-2P-GN; Vendor Conexel -> JLCPCB; Vendor PN 1x 1716080000 -> C2898699
Changed lines of the file:
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@@
 			)
 		)
-		(property "Footprint" "Tales:TerminalBlock_Phoenix_MKDS-3-2-5.08_1x02_P5.08mm_Horizontal"
+		(property "Footprint" "Tales:TerminalBlock_Dibo_DB142V-5.08-2P_1x02_P5.08mm_Vertical"
 			(at 34.29 36.83 0)
 			(effects
@@
 			)
 		)
-		(property "JLCPCB BOM" "0"
+		(property "JLCPCB BOM" "1"
 			(at 34.29 36.83 0)
 			(effects
@@
 			)
 		)
-		(property "Mfr" "Conexel"
+		(property "Mfr" "Dorabo"
 			(at 34.29 36.83 0)
 			(effects
@@
 			)
 		)
-		(property "Mfr PN" "1x LM 5.08/02/90 3.5SN OR BX"
+		(property "Mfr PN" "DB142V-5.08-2P-GN"
 			(at 34.29 36.83 0)
 			(effects
@@
 			)
 		)
-		(property "Vendor" "Conexel"
+		(property "Vendor" "JLCPCB"
 			(at 34.29 36.83 0)
 			(effects
@@
 			)
 		)
-		(property "Vendor PN" "1x 1716080000"
+		(property "Vendor PN" "C2898699"
 			(at 34.29 36.83 0)
 			(effects
@@
 			)
 		)
-		(property "LCSC Part #" "~"
+		(property "LCSC Part #" "C2898699"
 			(at 34.29 36.83 0)
 			(effects

Commit message: Update esp-24v-16ch-v3-power.kicad_sch
Parts:
- L2: LCSC Part # C127788 -> C169386; Mfr PN SWRH1205B-330MT -> SWRB1205S-330MT; Vendor PN C127788 -> C169386
- R1: value 5,6k/0,1W -> 560R/0,1W; LCSC Part # C23189 -> C23204; Mfr PN 0603WAF5601T5E -> 0603WAF5600T5E; Vendor PN C23189 -> C23204
Connections:
- net +24V: no longer R1.1
- net +5V: now also R1.1
Other:
- moved on the sheet: C3, C5, L1, R2, R3, U1

Commit message: Update esp-24v-16ch-v3-power.kicad_sch
Parts:
- C2: LCSC Part # C263963 -> C129415; Mfr PN CK1V470MCRE54 -> CK1V470M-CRE54; Vendor PN C263963 -> C129415
- Q2: value LMUN2211LT1G -> MMUN2211LT3G; LCSC Part # C12775 -> C150229; Mfr LRC -> Onsemi; Mfr PN LMUN2211LT1G -> MMUN2211LT3G; Vendor PN C12775 -> C150229
Changed lines of the file:
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@@
 			)
 		)
-		(property "Value" "LMUN2211LT1G"
+		(property "Value" "MMUN2211LT3G"
 			(at 214.63 140.97 90)
 			(effects
@@
 			)
 		)
-		(property "LCSC Part #" "C12775"
+		(property "LCSC Part #" "C150229"
 			(at 214.63 143.51 90)
 			(effects
@@
 			)
 		)
-		(property "Vendor PN" "C12775"
+		(property "Vendor PN" "C150229"
 			(at 214.63 148.59 0)
 			(effects
@@
 			)
 		)
-		(property "Mfr" "LRC"
+		(property "Mfr" "Onsemi"
 			(at 214.63 148.59 0)
 			(effects
@@
 			)
 		)
-		(property "Mfr PN" "LMUN2211LT1G"
+		(property "Mfr PN" "MMUN2211LT3G"
 			(at 214.63 148.59 0)
 			(effects
@@
 			)
 		)
-		(property "Mfr PN" "CK1V470MCRE54"
+		(property "Mfr PN" "CK1V470M-CRE54"
 			(at 74.93 43.18 0)
 			(effects
@@
 			)
 		)
-		(property "Vendor PN" "C263963"
+		(property "Vendor PN" "C129415"
 			(at 74.93 43.18 0)
 			(effects
@@
 			)
 		)
-		(property "LCSC Part #" "C263963"
+		(property "LCSC Part #" "C129415"
 			(at 78.74 49.53 0)
 			(effects

Commit message: Final touches to fabrication
Parts:
- D2: value GREEN -> GREEN/0603
- U1: footprint Tales:TSOT-23-5 -> Tales:SOT-23-5_Shorter_Pins
Changed lines of the file:
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@@
 			)
 		)
-		(property "Footprint" "Tales:TSOT-23-5"
+		(property "Footprint" "Tales:SOT-23-5_Shorter_Pins"
 			(at 67.31 148.59 0)
 			(effects
@@
 			)
 		)
-		(property "Value" "GREEN"
+		(property "Value" "GREEN/0603"
 			(at 49.53 170.18 90)
 			(effects

Commit message: Added temperature sensor
Parts:
- C4, C40: value 0,1uF/50V -> 100nF/50V
- R1: value 560R/0,1W -> 560R/100mW
- R2: value 100k/0,125W -> 100k/125mW
- R3: value 22,1k/0,125W -> 22,1k/125mW
- R4, R5, R8: Mfr UNI-ROYAL(Uniroyal Elec) -> Uniroyal
Changed lines of the file:
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@@
 			)
 		)
-		(property "Value" "560R/0,1W"
+		(property "Value" "560R/100mW"
 			(at 49.53 161.29 0)
 			(effects
@@
 			)
 		)
-		(property "Value" "0,1uF/50V"
+		(property "Value" "100nF/50V"
 			(at 130.81 87.63 0)
 			(effects
@@
 			)
 		)
-		(property "Value" "0,1uF/50V"
+		(property "Value" "100nF/50V"
 			(at 99.06 43.18 0)
 			(effects
@@
 			)
 		)
-		(property "Mfr" "UNI-ROYAL(Uniroyal Elec)"
+		(property "Mfr" "Uniroyal"
 			(at 180.34 36.83 0)
 			(effects
@@
 			)
 		)
-		(property "Mfr" "UNI-ROYAL(Uniroyal Elec)"
+		(property "Mfr" "Uniroyal"
 			(at 127 44.45 0)
 			(effects
@@
 			)
 		)
-		(property "Mfr" "UNI-ROYAL(Uniroyal Elec)"
+		(property "Mfr" "Uniroyal"
 			(at 227.33 57.15 0)
 			(effects
@@
 			)
 		)
-		(property "Value" "22,1k/0,125W"
+		(property "Value" "22,1k/125mW"
 			(at 120.65 165.1 0)
 			(effects
@@
 			)
 		)
-		(property "Value" "100k/0,125W"
+		(property "Value" "100k/125mW"
 			(at 120.65 152.4 0)
 			(effects

Commit message: Updating component part numbers
Parts:
- D2: value GREEN/0603 -> AMBER/0603; LCSC Part # C72043 -> C165983; Mfr Everlight -> BrtLed(Bright LED Elec); Mfr PN 19-217/GHC-YR1S2/3T -> BL-HJC36G-AV-TRB; Vendor PN C72043 -> C165983
Changed lines of the file:
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@@
 			)
 		)
-		(property "Value" "GREEN/0603"
+		(property "Value" "AMBER/0603"
 			(at 49.53 170.18 90)
 			(effects
@@
 			)
 		)
-		(property "Mfr" "Everlight"
+		(property "Mfr" "BrtLed(Bright LED Elec)"
 			(at 46.99 170.18 0)
 			(effects
@@
 			)
 		)
-		(property "Mfr PN" "19-217/GHC-YR1S2/3T"
+		(property "Mfr PN" "BL-HJC36G-AV-TRB"
 			(at 46.99 170.18 0)
 			(effects
@@
 			)
 		)
-		(property "Vendor PN" "C72043"
+		(property "Vendor PN" "C165983"
 			(at 46.99 170.18 0)
 			(effects
@@
 			)
 		)
-		(property "LCSC Part #" "C72043"
+		(property "LCSC Part #" "C165983"
 			(at 49.53 172.72 90)
 			(effects
