File: V3/esp-24v-16ch-v3-outputs-1.kicad_sch (KiCad schematic)
At the start: 80 parts, among them Q10 MMBT2222A/SOT-23-3, Q11 MMBT2222A/SOT-23-3, Q12 MMBT2222A/SOT-23-3, Q13 MMBT2222A/SOT-23-3, Q14 MMBT2222A/SOT-23-3, Q15 MMBT2222A/SOT-23-3, Q16 MMBT2222A/SOT-23-3, Q17 MMBT2222A/SOT-23-3, Q18 MMBT2222A/SOT-23-3, Q19 MMBT2222A/SOT-23-3, Q4 MMBT2222A/SOT-23-3, Q5 MMBT2222A/SOT-23-3, Q6 MMBT2222A/SOT-23-3, Q7 MMBT2222A/SOT-23-3, Q8 MMBT2222A/SOT-23-3, Q9 MMBT2222A/SOT-23-3

Commit message: working on v3
Parts:
- Q10, Q11, Q12, Q13, Q14, Q15, Q16, Q17, Q18, Q19, Q4, Q5, Q6, Q7, Q8, Q9: value MMBT2222A/SOT-23-3 -> MMBT2222A
- R100, R109, R110, R111, R112, R121, R122, R123, R124, R85, R86, R87, R88, R97, R98, R99: value 1k/62,5mW/0402 -> 1k/62,5mW
- R101, R102, R103, R104, R113, R114, R115, R116, R125, R126, R127, R128, R89, R90, R91, R92: value 5,6k/0,1W/0603 -> 5,6k/0,1W
- R105, R106, R107, R108, R117, R118, R119, R120, R81, R82, R83, R84, R93, R94, R95, R96: value 10k/62,5mW/0402 -> 10k/62,5mW; LCSC Part # C25744 -> C60490; Mfr Uniroyal -> Yageo; Mfr PN 0402WGF1002TCE -> RC0402FR-0710KL; Package (none) -> 0402/1005; Technology (none) -> 1%; Vendor PN C25744 -> C60490
Connections:
- net GND: now also R105.1, R106.1, R107.1, R108.1, R117.1, R118.1, R119.1, R120.1, R81.1, R82.1, R83.1, R84.1, R93.1, R94.1, R95.1, R96.1; no longer R105.2, R106.2, R107.2, R108.2, R117.2, R118.2, R119.2, R120.2, R81.2, R82.2, R83.2, R84.2, R93.2, R94.2, R95.2, R96.2
- net OUT1: now also R81.2; no longer R81.1
- net OUT10: now also R106.2; no longer R106.1
- net OUT11: now also R107.2; no longer R107.1
- net OUT12: now also R108.2; no longer R108.1
- net OUT13: now also R117.2; no longer R117.1
- net OUT14: now also R118.2; no longer R118.1
- net OUT15: now also R119.2; no longer R119.1
- net OUT16: now also R120.2; no longer R120.1
- net OUT2: now also R82.2; no longer R82.1
- net OUT3: now also R83.2; no longer R83.1
- net OUT4: now also R84.2; no longer R84.1
- net OUT5: now also R93.2; no longer R93.1
- net OUT6: now also R94.2; no longer R94.1
- net OUT7: now also R95.2; no longer R95.1
- net OUT8: now also R96.2; no longer R96.1
- net OUT9: now also R105.2; no longer R105.1

Commit message: Update esp-24v-16ch-v3-outputs-1.kicad_sch
Parts:
- Q10, Q11, Q12, Q13, Q14, Q15, Q16, Q17, Q18, Q19, Q4, Q5, Q6, Q7, Q8, Q9: footprint Tales:SOT-23 -> Tales:SOT-23-Narrow
Changed lines of the file:
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@@
 			)
 		)
-		(property "Footprint" "Tales:SOT-23"
+		(property "Footprint" "Tales:SOT-23-Narrow"
 			(at 248.92 74.93 0)
 			(effects
@@
 			)
 		)
-		(property "Footprint" "Tales:SOT-23"
+		(property "Footprint" "Tales:SOT-23-Narrow"
 			(at 120.65 74.93 0)
 			(effects
@@
 			)
 		)
-		(property "Footprint" "Tales:SOT-23"
+		(property "Footprint" "Tales:SOT-23-Narrow"
 			(at 55.88 74.93 0)
 			(effects
@@
 			)
 		)
-		(property "Footprint" "Tales:SOT-23"
+		(property "Footprint" "Tales:SOT-23-Narrow"
 			(at 248.92 38.1 0)
 			(effects
@@
 			)
 		)
-		(property "Footprint" "Tales:SOT-23"
+		(property "Footprint" "Tales:SOT-23-Narrow"
 			(at 120.65 111.76 0)
 			(effects
@@
 			)
 		)
-		(property "Footprint" "Tales:SOT-23"
+		(property "Footprint" "Tales:SOT-23-Narrow"
 			(at 55.88 148.59 0)
 			(effects
@@
 			)
 		)
-		(property "Footprint" "Tales:SOT-23"
+		(property "Footprint" "Tales:SOT-23-Narrow"
 			(at 185.42 111.76 0)
 			(effects
@@
 			)
 		)
-		(property "Footprint" "Tales:SOT-23"
+		(property "Footprint" "Tales:SOT-23-Narrow"
 			(at 55.88 111.76 0)
 			(effects
@@
 			)
 		)
-		(property "Footprint" "Tales:SOT-23"
+		(property "Footprint" "Tales:SOT-23-Narrow"
 			(at 185.42 148.59 0)
 			(effects
@@
 			)
 		)
-		(property "Footprint" "Tales:SOT-23"
+		(property "Footprint" "Tales:SOT-23-Narrow"
 			(at 248.92 148.59 0)
 			(effects
@@
 			)
 		)
-		(property "Footprint" "Tales:SOT-23"
+		(property "Footprint" "Tales:SOT-23-Narrow"
 			(at 185.42 38.1 0)
 			(effects
@@
 			)
 		)
-		(property "Footprint" "Tales:SOT-23"
+		(property "Footprint" "Tales:SOT-23-Narrow"
 			(at 248.92 111.76 0)
 			(effects
@@
 			)
 		)
-		(property "Footprint" "Tales:SOT-23"
+		(property "Footprint" "Tales:SOT-23-Narrow"
 			(at 120.65 148.59 0)
 			(effects
@@
 			)
 		)
-		(property "Footprint" "Tales:SOT-23"
+		(property "Footprint" "Tales:SOT-23-Narrow"
 			(at 185.42 74.93 0)
 			(effects
@@
 			)
 		)
-		(property "Footprint" "Tales:SOT-23"
+		(property "Footprint" "Tales:SOT-23-Narrow"
 			(at 120.65 38.1 0)
 			(effects
@@
 			)
 		)
-		(property "Footprint" "Tales:SOT-23"
+		(property "Footprint" "Tales:SOT-23-Narrow"
 			(at 55.88 38.1 0)
 			(effects

Commit message: Final touches to fabrication
Parts:
- D39, D40, D41, D42, D43, D44, D45, D46, D47, D48, D49, D50, D51, D52, D53, D54: Case 0603 -> 0603/1608
Changed lines of the file:
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@@
 			)
 		)
-		(property "Case" "0603"
+		(property "Case" "0603/1608"
 			(at 246.38 67.31 0)
 			(effects
@@
 			)
 		)
-		(property "Case" "0603"
+		(property "Case" "0603/1608"
 			(at 53.34 104.14 0)
 			(effects
@@
 			)
 		)
-		(property "Case" "0603"
+		(property "Case" "0603/1608"
 			(at 246.38 140.97 0)
 			(effects
@@
 			)
 		)
-		(property "Case" "0603"
+		(property "Case" "0603/1608"
 			(at 53.34 30.48 0)
 			(effects
@@
 			)
 		)
-		(property "Case" "0603"
+		(property "Case" "0603/1608"
 			(at 182.88 140.97 0)
 			(effects
@@
 			)
 		)
-		(property "Case" "0603"
+		(property "Case" "0603/1608"
 			(at 118.11 67.31 0)
 			(effects
@@
 			)
 		)
-		(property "Case" "0603"
+		(property "Case" "0603/1608"
 			(at 118.11 104.14 0)
 			(effects
@@
 			)
 		)
-		(property "Case" "0603"
+		(property "Case" "0603/1608"
 			(at 182.88 67.31 0)
 			(effects
@@
 			)
 		)
-		(property "Case" "0603"
+		(property "Case" "0603/1608"
 			(at 118.11 140.97 0)
 			(effects
@@
 			)
 		)
-		(property "Case" "0603"
+		(property "Case" "0603/1608"
 			(at 246.38 104.14 0)
 			(effects
@@
 			)
 		)
-		(property "Case" "0603"
+		(property "Case" "0603/1608"
 			(at 246.38 30.48 0)
 			(effects
@@
 			)
 		)
-		(property "Case" "0603"
+		(property "Case" "0603/1608"
 			(at 182.88 104.14 0)
 			(effects
@@
 			)
 		)
-		(property "Case" "0603"
+		(property "Case" "0603/1608"
 			(at 53.34 140.97 0)
 			(effects
@@
 			)
 		)
-		(property "Case" "0603"
+		(property "Case" "0603/1608"
 			(at 182.88 30.48 0)
 			(effects
@@
 			)
 		)
-		(property "Case" "0603"
+		(property "Case" "0603/1608"
 			(at 53.34 67.31 0)
 			(effects
@@
 			)
 		)
-		(property "Case" "0603"
+		(property "Case" "0603/1608"
 			(at 118.11 30.48 0)
 			(effects

Commit message: Added temperature sensor
Parts:
- R101, R102, R103, R104, R113, R114, R115, R116, R125, R126, R127, R128, R89, R90, R91, R92: value 5,6k/0,1W -> 5,6k/100mW
Changed lines of the file:
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@@
 			)
 		)
-		(property "Value" "5,6k/0,1W"
+		(property "Value" "5,6k/100mW"
 			(at 248.92 22.86 0)
 			(effects
@@
 			)
 		)
-		(property "Value" "5,6k/0,1W"
+		(property "Value" "5,6k/100mW"
 			(at 120.65 59.69 0)
 			(effects
@@
 			)
 		)
-		(property "Value" "5,6k/0,1W"
+		(property "Value" "5,6k/100mW"
 			(at 185.42 59.69 0)
 			(effects
@@
 			)
 		)
-		(property "Value" "5,6k/0,1W"
+		(property "Value" "5,6k/100mW"
 			(at 55.88 96.52 0)
 			(effects
@@
 			)
 		)
-		(property "Value" "5,6k/0,1W"
+		(property "Value" "5,6k/100mW"
 			(at 185.42 22.86 0)
 			(effects
@@
 			)
 		)
-		(property "Value" "5,6k/0,1W"
+		(property "Value" "5,6k/100mW"
 			(at 120.65 22.86 0)
 			(effects
@@
 			)
 		)
-		(property "Value" "5,6k/0,1W"
+		(property "Value" "5,6k/100mW"
 			(at 120.65 133.35 0)
 			(effects
@@
 			)
 		)
-		(property "Value" "5,6k/0,1W"
+		(property "Value" "5,6k/100mW"
 			(at 55.88 133.35 0)
 			(effects
@@
 			)
 		)
-		(property "Value" "5,6k/0,1W"
+		(property "Value" "5,6k/100mW"
 			(at 55.88 59.69 0)
 			(effects
@@
 			)
 		)
-		(property "Value" "5,6k/0,1W"
+		(property "Value" "5,6k/100mW"
 			(at 248.92 133.35 0)
 			(effects
@@
 			)
 		)
-		(property "Value" "5,6k/0,1W"
+		(property "Value" "5,6k/100mW"
 			(at 185.42 96.52 0)
 			(effects
@@
 			)
 		)
-		(property "Value" "5,6k/0,1W"
+		(property "Value" "5,6k/100mW"
 			(at 185.42 133.35 0)
 			(effects
@@
 			)
 		)
-		(property "Value" "5,6k/0,1W"
+		(property "Value" "5,6k/100mW"
 			(at 248.92 59.69 0)
 			(effects
@@
 			)
 		)
-		(property "Value" "5,6k/0,1W"
+		(property "Value" "5,6k/100mW"
 			(at 55.88 22.86 0)
 			(effects
@@
 			)
 		)
-		(property "Value" "5,6k/0,1W"
+		(property "Value" "5,6k/100mW"
 			(at 248.92 96.52 0)
 			(effects
@@
 			)
 		)
-		(property "Value" "5,6k/0,1W"
+		(property "Value" "5,6k/100mW"
 			(at 120.65 96.52 0)
 			(effects

Commit message: Updating component part numbers
Parts:
- D39, D40, D41, D42, D43, D44, D45, D46, D47, D48, D49, D50, D51, D52, D53, D54: value GREEN/0603 -> AMBER/0603; LCSC Part # C72043 -> C165983; Mfr Everlight -> BrtLed(Bright LED Elec); Mfr PN 19-217/GHC-YR1S2/3T -> BL-HJC36G-AV-TRB; Vendor PN C72043 -> C165983

Commit message: Prefab checks
Parts:
- D39, D40, D41, D42, D43, D44, D45, D46, D47, D48, D49, D50, D51, D52, D53, D54: value AMBER/0603 -> EMERALD/0603; LCSC Part # C165983 -> C2984266; Mfr BrtLed(Bright LED Elec) -> Everlight Elec; Mfr PN BL-HJC36G-AV-TRB -> 19-213/GHC-XS1T1N/5T; Vendor PN C165983 -> C2984266

Commit message: Improvements to high speed signals routing
Parts:
- R101, R102, R103, R104, R113, R114, R115, R116, R125, R126, R127, R128, R89, R90, R91, R92: value 5,6k/100mW -> 6,8k/100mW; LCSC Part # C23189 -> C23212; Mfr PN 0603WAF5601T5E -> 0603WAF6801T5E; Vendor PN C23189 -> C23212
Changed lines of the file:
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@@
 			)
 		)
-		(property "Value" "5,6k/100mW"
+		(property "Value" "6,8k/100mW"
 			(at 248.92 22.86 0)
 			(effects
@@
 			)
 		)
-		(property "Mfr PN" "0603WAF5601T5E"
+		(property "Mfr PN" "0603WAF6801T5E"
 			(at 246.38 22.86 0)
 			(effects
@@
 			)
 		)
-		(property "Vendor PN" "C23189"
+		(property "Vendor PN" "C23212 "
 			(at 246.38 22.86 0)
 			(effects
@@
 			)
 		)
-		(property "LCSC Part #" "C23189"
+		(property "LCSC Part #" "C23212"
 			(at 248.92 25.4 0)
 			(effects
@@
 			)
 		)
-		(property "Value" "5,6k/100mW"
+		(property "Value" "6,8k/100mW"
 			(at 120.65 59.69 0)
 			(effects
@@
 			)
 		)
-		(property "Mfr PN" "0603WAF5601T5E"
+		(property "Mfr PN" "0603WAF6801T5E"
 			(at 118.11 59.69 0)
 			(effects
@@
 			)
 		)
-		(property "Vendor PN" "C23189"
+		(property "Vendor PN" "C23212 "
 			(at 118.11 59.69 0)
 			(effects
@@
 			)
 		)
-		(property "LCSC Part #" "C23189"
+		(property "LCSC Part #" "C23212"
 			(at 120.65 62.23 0)
 			(effects
@@
 			)
 		)
-		(property "Value" "5,6k/100mW"
+		(property "Value" "6,8k/100mW"
 			(at 185.42 59.69 0)
 			(effects
@@
 			)
 		)
-		(property "Mfr PN" "0603WAF5601T5E"
+		(property "Mfr PN" "0603WAF6801T5E"
 			(at 182.88 59.69 0)
 			(effects
@@
 			)
 		)
-		(property "Vendor PN" "C23189"
+		(property "Vendor PN" "C23212 "
 			(at 182.88 59.69 0)
 			(effects
@@
 			)
 		)
-		(property "LCSC Part #" "C23189"
+		(property "LCSC Part #" "C23212"
 			(at 185.42 62.23 0)
 			(effects
@@
 			)
 		)
-		(property "Value" "5,6k/100mW"
+		(property "Value" "6,8k/100mW"
 			(at 55.88 96.52 0)
 			(effects
@@
 			)
 		)
-		(property "Mfr PN" "0603WAF5601T5E"
+		(property "Mfr PN" "0603WAF6801T5E"
 			(at 53.34 96.52 0)
 			(effects
@@
 			)
 		)
-		(property "Vendor PN" "C23189"
+		(property "Vendor PN" "C23212 "
 			(at 53.34 96.52 0)
 			(effects
@@
 			)
 		)
-		(property "LCSC Part #" "C23189"
+		(property "LCSC Part #" "C23212"
 			(at 55.88 99.06 0)
 			(effects
@@
 			)
 		)
-		(property "Value" "5,6k/100mW"
+		(property "Value" "6,8k/100mW"
 			(at 185.42 22.86 0)
 			(effects
@@
 			)
 		)
-		(property "Mfr PN" "0603WAF5601T5E"
+		(property "Mfr PN" "0603WAF6801T5E"
 			(at 182.88 22.86 0)
 			(effects
@@
 			)
 		)
-		(property "Vendor PN" "C23189"
+		(property "Vendor PN" "C23212 "
 			(at 182.88 22.86 0)
 			(effects
@@
 			)
 		)
-		(property "LCSC Part #" "C23189"
+		(property "LCSC Part #" "C23212"
 			(at 185.42 25.4 0)
 			(effects
@@
 			)
 		)
-		(property "Value" "5,6k/100mW"
+		(property "Value" "6,8k/100mW"
 			(at 120.65 22.86 0)
 			(effects
@@
 			)
 		)
-		(property "Mfr PN" "0603WAF5601T5E"
+		(property "Mfr PN" "0603WAF6801T5E"
 			(at 118.11 22.86 0)
 			(effects
@@
 			)
 		)
-		(property "Vendor PN" "C23189"
+		(property "Vendor PN" "C23212 "
 			(at 118.11 22.86 0)
 			(effects
@@
 			)
 		)
-		(property "LCSC Part #" "C23189"
+		(property "LCSC Part #" "C23212"
 			(at 120.65 25.4 0)
 			(effects
@@
 			)
 		)
-		(property "Value" "5,6k/100mW"
+		(property "Value" "6,8k/100mW"
 			(at 120.65 133.35 0)
 			(effects
@@
 			)
 		)
-		(property "Mfr PN" "0603WAF5601T5E"
+		(property "Mfr PN" "0603WAF6801T5E"
 			(at 118.11 133.35 0)
 			(effects
@@
 			)
 		)
-		(property "Vendor PN" "C23189"
+		(property "Vendor PN" "C23212 "
 			(at 118.11 133.35 0)
 			(effects
@@
 			)
 		)
-		(property "LCSC Part #" "C23189"
+		(property "LCSC Part #" "C23212"
 			(at 120.65 135.89 0)
 			(effects
@@
 			)
 		)
-		(property "Value" "5,6k/100mW"
+		(property "Value" "6,8k/100mW"
 			(at 55.88 133.35 0)
 			(effects
@@
 			)
 		)
-		(property "Mfr PN" "0603WAF5601T5E"
+		(property "Mfr PN" "0603WAF6801T5E"
 			(at 53.34 133.35 0)
 			(effects
@@
 			)
 		)
-		(property "Vendor PN" "C23189"
+		(property "Vendor PN" "C23212 "
 			(at 53.34 133.35 0)
 			(effects
@@
 			)
 		)
-		(property "LCSC Part #" "C23189"
+		(property "LCSC Part #" "C23212"
 			(at 55.88 135.89 0)
 			(effects
@@
 			)
 		)
-		(property "Value" "5,6k/100mW"
+		(property "Value" "6,8k/100mW"
 			(at 55.88 59.69 0)
 			(effects
@@
 			)
 		)
-		(property "Mfr PN" "0603WAF5601T5E"
+		(property "Mfr PN" "0603WAF6801T5E"
 			(at 53.34 59.69 0)
 			(effects
@@
 			)
 		)
-		(property "Vendor PN" "C23189"
+		(property "Vendor PN" "C23212 "
 			(at 53.34 59.69 0)
 			(effects
@@
 			)
 		)
-		(property "LCSC Part #" "C23189"
+		(property "LCSC Part #" "C23212"
 			(at 55.88 62.23 0)
 			(effects
@@
 			)
 		)
-		(property "Value" "5,6k/100mW"
+		(property "Value" "6,8k/100mW"
 			(at 248.92 133.35 0)
 			(effects
@@
 			)
 		)
-		(property "Mfr PN" "0603WAF5601T5E"
+		(property "Mfr PN" "0603WAF6801T5E"
 			(at 246.38 133.35 0)
 			(effects
@@
 			)
 		)
-		(property "Vendor PN" "C23189"
+		(property "Vendor PN" "C23212 "
 			(at 246.38 133.35 0)
 			(effects
@@
 			)
 		)
-		(property "LCSC Part #" "C23189"
+		(property "LCSC Part #" "C23212"
 			(at 248.92 135.89 0)
 			(effects
@@
 			)
 		)
-		(property "Value" "5,6k/100mW"
+		(property "Value" "6,8k/100mW"
 			(at 185.42 96.52 0)
 			(effects
@@
 			)
 		)
-		(property "Mfr PN" "0603WAF5601T5E"
+		(property "Mfr PN" "0603WAF6801T5E"
 			(at 182.88 96.52 0)
 			(effects
@@
 			)
 		)
-		(property "Vendor PN" "C23189"
+		(property "Vendor PN" "C23212 "
 			(at 182.88 96.52 0)
 			(effects
@@
 			)
 		)
-		(property "LCSC Part #" "C23189"
+		(property "LCSC Part #" "C23212"
 			(at 185.42 99.06 0)
 			(effects
@@
 			)
 		)
-		(property "Value" "5,6k/100mW"
+		(property "Value" "6,8k/100mW"
 			(at 185.42 133.35 0)
 			(effects
@@
 			)
 		)
-		(property "Mfr PN" "0603WAF5601T5E"
+		(property "Mfr PN" "0603WAF6801T5E"
 			(at 182.88 133.35 0)
 			(effects
@@
 			)
 		)
-		(property "Vendor PN" "C23189"
+		(property "Vendor PN" "C23212 "
 			(at 182.88 133.35 0)
 			(effects
@@
 			)
 		)
-		(property "LCSC Part #" "C23189"
+		(property "LCSC Part #" "C23212"
 			(at 185.42 135.89 0)
 			(effects
@@
 			)
 		)
-		(property "Value" "5,6k/100mW"
+		(property "Value" "6,8k/100mW"
 			(at 248.92 59.69 0)
 			(effects
@@
 			)
 		)
-		(property "Mfr PN" "0603WAF5601T5E"
+		(property "Mfr PN" "0603WAF6801T5E"
 			(at 246.38 59.69 0)
 			(effects
@@
 			)
 		)
-		(property "Vendor PN" "C23189"
+		(property "Vendor PN" "C23212 "
 			(at 246.38 59.69 0)
 			(effects
@@
 			)
 		)
-		(property "LCSC Part #" "C23189"
+		(property "LCSC Part #" "C23212"
 			(at 248.92 62.23 0)
 			(effects
@@
 			)
 		)
-		(property "Value" "5,6k/100mW"
+		(property "Value" "6,8k/100mW"
 			(at 55.88 22.86 0)
 			(effects
@@
 			)
 		)
-		(property "Mfr PN" "0603WAF5601T5E"
+		(property "Mfr PN" "0603WAF6801T5E"
 			(at 53.34 22.86 0)
 			(effects
@@
 			)
 		)
-		(property "Vendor PN" "C23189"
+		(property "Vendor PN" "C23212 "
 			(at 53.34 22.86 0)
 			(effects
@@
 			)
 		)
-		(property "LCSC Part #" "C23189"
+		(property "LCSC Part #" "C23212"
 			(at 55.88 25.4 0)
 			(effects
@@
 			)
 		)
-		(property "Value" "5,6k/100mW"
+		(property "Value" "6,8k/100mW"
 			(at 248.92 96.52 0)
 			(effects
@@
 			)
 		)
-		(property "Mfr PN" "0603WAF5601T5E"
+		(property "Mfr PN" "0603WAF6801T5E"
 			(at 246.38 96.52 0)
 			(effects
@@
 			)
 		)
-		(property "Vendor PN" "C23189"
+		(property "Vendor PN" "C23212 "
 			(at 246.38 96.52 0)
 			(effects
@@
 			)
 		)
-		(property "LCSC Part #" "C23189"
+		(property "LCSC Part #" "C23212"
 			(at 248.92 99.06 0)
 			(effects
@@
 			)
 		)
-		(property "Value" "5,6k/100mW"
+		(property "Value" "6,8k/100mW"
 			(at 120.65 96.52 0)
 			(effects
@@
 			)
 		)
-		(property "Mfr PN" "0603WAF5601T5E"
+		(property "Mfr PN" "0603WAF6801T5E"
 			(at 118.11 96.52 0)
 			(effects
@@
 			)
 		)
-		(property "Vendor PN" "C23189"
+		(property "Vendor PN" "C23212 "
 			(at 118.11 96.52 0)
 			(effects
@@
 			)
 		)
-		(property "LCSC Part #" "C23189"
+		(property "LCSC Part #" "C23212"
 			(at 120.65 99.06 0)
 			(effects
