File: V3/esp-24v-16ch-v3-i2c.kicad_sch (KiCad schematic)
At the start: 14 parts, among them J8 NTC, U12 AHT20, U13 ADS1115IDGS, U6 MCP23017_SS, U7 MCP23017_SS

Commit message: Renamed to V3.2
Other:
- title: ESP 16x 24VDC Input 16x 24VDC Output Module -> ESP 24V 16xIn/16xOut/4xNTC Module
Changed lines of the file:
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@@
 	(paper "A4")
 	(title_block
-		(title "ESP 16x 24VDC Input 16x 24VDC Output Module")
-		(date "2023-05-05")
-		(rev "V3")
+		(title "ESP 24V 16xIn/16xOut/4xNTC Module")
+		(date "2025-06-29")
+		(rev "V3.2")
 	)
 	(junction

Commit message: BOM corrected
Parts:
- C42: value 0,1uF/50V -> 100nF/50V; Case (none) -> 0402/1005
Changed lines of the file:
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@@
 			)
 		)
-		(property "Value" "0,1uF/50V"
+		(property "Value" "100nF/50V"
 			(at 96.52 140.3413 0)
 			(effects
@@
 			(at 99.06 140.97 0)
 			(effects
+				(font
+					(size 1.27 1.27)
+				)
+				(hide yes)
+			)
+		)
+		(property "Case" "0402/1005"
+			(at 99.06 140.97 0)
+			(effects
