File: V3/esp-24v-16ch-v3.kicad_pcb (KiCad board)
At the start: 4 copper layers, 108 x 67.8 mm, 270 parts, among them J1 VIN, J2 USB_C_Receptacle_USB2.0, J3 DB141V-2.54-8P, J4 DB141V-2.54-8P, J5 DB141V-2.54-8P, J6 DB141V-2.54-8P, J7 ETHERNET, J8 NTC, Q1 WPM2015-3/TR, Q10 MMBT2222A, Q11 MMBT2222A, Q12 MMBT2222A, Q13 MMBT2222A, Q14 MMBT2222A, Q15 MMBT2222A, Q16 MMBT2222A, Q17 MMBT2222A, Q18 MMBT2222A, Q19 MMBT2222A, Q2 MMUN2211LT3G, Q3 UMH3N, Q4 MMBT2222A, Q5 MMBT2222A, Q6 MMBT2222A, Q7 MMBT2222A, Q8 MMBT2222A, Q9 MMBT2222A, SW1 RESET, U1 SY8089A1AAC, U10 OR-3H4-4, U11 OR-3H4-4, U12 AHT20, U13 ADS1115IDGS, U2 TX4138, U3 CH340C, U4 ESP32-WROOM-32UE-N16, U5 LAN8710A, U6 MCP23017_SS, U7 MCP23017_SS, U8 OR-3H4-4, U9 OR-3H4-4

Commit message: Files for new release
Routing:
- net GND: vias 119 -> 123
Changed lines of the file:
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@@
+	)
+	(via
+		(at 106.27 80.58)
+		(size 0.6)
+		(drill 0.3)
+		(layers "F.Cu" "B.Cu")
+		(free yes)
+		(net 1)
 	)
 	(via
@@
 	)
 	(via
+		(at 109.27 81.58)
+		(size 0.6)
+		(drill 0.3)
+		(layers "F.Cu" "B.Cu")
+		(free yes)
+		(net 1)
+	)
+	(via
 		(at 149.86 77.5198)
 		(size 0.6)
@@
 		(size 1)
 		(drill 0.4)
+		(layers "F.Cu" "B.Cu")
+		(free yes)
+		(net 1)
+	)
+	(via
+		(at 131.642974 96.430574)
+		(size 0.6)
+		(drill 0.3)
 		(layers "F.Cu" "B.Cu")
 		(free yes)
@@
 		(net 1)
 	)
+	(via
+		(at 133.27 97.58)
+		(size 0.6)
+		(drill 0.3)
+		(layers "F.Cu" "B.Cu")
+		(free yes)
+		(net 1)
+	)

Commit message: BOM corrected
Parts:
- C42: value 0,1uF/50V -> 100nF/50V
Changed lines of the file:
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@@
 			)
 		)
-		(property "Value" "0,1uF/50V"
+		(property "Value" "100nF/50V"
 			(at 0 1.16 0)
 			(layer "F.Fab")
@@
 			(at 0 0 0)
 			(unlocked yes)
+			(layer "F.Fab")
+			(hide yes)
+			(effects
+				(font
+					(size 1 1)
+					(thickness 0.15)
+				)
+			)
+		)
+		(property "Case" "0402/1005"
+			(at 0 0 0)
+			(unlocked yes)

Commit message: AD/DC opamp swapped for DC model
Parts:
- U10, U11, U8, U9: value OR-3H4-4 -> OR-3H7-4
Changed lines of the file:
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@@
 			)
 		)
-		(property "Value" "OR-3H4-4"
+		(property "Value" "OR-3H7-4"
 			(at 0 6.1 90)
 			(layer "F.Fab")
@@
 			)
 		)
-		(property "Description" ""
+		(property "Description" "Quad DC Optocoupler, Vce 80V, CTR 100%, SOP16"
 			(at 0 0 90)
 			(layer "F.Fab")
@@
 			)
 		)
-		(property "LCSC Part #" "C2838167"
+		(property "LCSC Part #" "C2838427"
 			(at 191.8 -12.68 0)
 			(layer "F.Fab")
@@
 			)
 		)
-		(property "Mfr PN" "OR-3H4-4GB-TA1-GK"
+		(property "Mfr PN" "OR-3H7-4GB-TA1-G"
 			(at 191.8 -12.68 0)
 			(layer "F.Fab")
@@
 			)
 		)
-		(property "Vendor PN" "C2838167"
+		(property "Vendor PN" "C2838427"
 			(at 191.8 -12.68 0)
 			(layer "F.Fab")
@@
 			)
 		)
-		(property "Value" "OR-3H4-4"
+		(property "Value" "OR-3H7-4"
 			(at 0 6.1 90)
 			(layer "F.Fab")
@@
 			)
 		)
-		(property "Description" ""
+		(property "Description" "Quad DC Optocoupler, Vce 80V, CTR 100%, SOP16"
 			(at 0 0 90)
 			(layer "F.Fab")
@@
 			)
 		)
-		(property "LCSC Part #" "C2838167"
+		(property "LCSC Part #" "C2838427"
 			(at 200.055 -4.425 0)
 			(layer "F.Fab")
@@
 			)
 		)
-		(property "Mfr PN" "OR-3H4-4GB-TA1-GK"
+		(property "Mfr PN" "OR-3H7-4GB-TA1-G"
 			(at 200.055 -4.425 0)
 			(layer "F.Fab")
@@
 			)
 		)
-		(property "Vendor PN" "C2838167"
+		(property "Vendor PN" "C2838427"
 			(at 200.055 -4.425 0)
 			(layer "F.Fab")
@@
 			)
 		)
-		(property "Value" "OR-3H4-4"
+		(property "Value" "OR-3H7-4"
 			(at 0 6.1 90)
 			(layer "F.Fab")
@@
 			)
 		)
-		(property "Description" ""
+		(property "Description" "Quad DC Optocoupler, Vce 80V, CTR 100%, SOP16"
 			(at 0 0 90)
 			(layer "F.Fab")
@@
 			)
 		)
-		(property "LCSC Part #" "C2838167"
+		(property "LCSC Part #" "C2838427"
 			(at 216.565 12.085 0)
 			(layer "F.Fab")
@@
 			)
 		)
-		(property "Mfr PN" "OR-3H4-4GB-TA1-GK"
+		(property "Mfr PN" "OR-3H7-4GB-TA1-G"
 			(at 216.565 12.085 0)
 			(layer "F.Fab")
@@
 			)
 		)
-		(property "Vendor PN" "C2838167"
+		(property "Vendor PN" "C2838427"
 			(at 216.565 12.085 0)
 			(layer "F.Fab")
@@
 			)
 		)
-		(property "Value" "OR-3H4-4"
+		(property "Value" "OR-3H7-4"
 			(at 0 6.1 90)
 			(layer "F.Fab")
@@
 			)
 		)
-		(property "Description" ""
+		(property "Description" "Quad DC Optocoupler, Vce 80V, CTR 100%, SOP16"
 			(at 0 0 90)
 			(layer "F.Fab")
@@
 			)
 		)
-		(property "LCSC Part #" "C2838167"
+		(property "LCSC Part #" "C2838427"
 			(at 208.31 3.83 0)
 			(layer "F.Fab")
@@
 			)
 		)
-		(property "Mfr PN" "OR-3H4-4GB-TA1-GK"
+		(property "Mfr PN" "OR-3H7-4GB-TA1-G"
 			(at 208.31 3.83 0)
 			(layer "F.Fab")
@@
 			)
 		)
-		(property "Vendor PN" "C2838167"
+		(property "Vendor PN" "C2838427"
 			(at 208.31 3.83 0)
 			(layer "F.Fab")
