File: V4/esp-24v-16ch-outputs.kicad_sch (KiCad schematic)
At the start: 5 parts, among them Q5 MMBT2222A

Commit message: Routing V4
Parts:
- renumbered D56 to D60, Q5 to Q9, R77 to R89, R78 to R90, R79 to R91
Changed lines of the file:
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@@
 		(on_board yes)
 		(dnp no)
-		(property "Reference" "#PWR0199"
+		(property "Reference" "#PWR0211"
 			(at 107.95 118.11 0)
 			(effects
@@
 		(on_board yes)
 		(dnp no)
-		(property "Reference" "#PWR0200"
+		(property "Reference" "#PWR0212"
 			(at 144.78 64.77 0)
 			(effects
@@
 		(on_board yes)
 		(dnp no)
-		(property "Reference" "R79"
+		(property "Reference" "R91"
 			(at 147.32 66.04 0)
 			(effects
@@
 		(on_board yes)
 		(dnp no)
-		(property "Reference" "R78"
+		(property "Reference" "R90"
 			(at 125.73 96.52 90)
 			(effects
@@
 		(on_board yes)
 		(dnp no)
-		(property "Reference" "D56"
+		(property "Reference" "D60"
 			(at 142.24 80.01 90)
 			(effects
@@
 		(on_board yes)
 		(dnp no)
-		(property "Reference" "R77"
+		(property "Reference" "R89"
 			(at 110.49 107.95 0)
 			(effects
@@
 		(on_board yes)
 		(dnp no)
-		(property "Reference" "#PWR0201"
+		(property "Reference" "#PWR0213"
 			(at 144.78 119.38 0)
 			(effects
@@
 		(on_board yes)
 		(dnp no)
-		(property "Reference" "Q5"
+		(property "Reference" "Q9"
 			(at 148.59 99.06 0)
 			(effects

Commit message: Routing V4
Parts:
- D60: value EMERALD/0603 -> WHITE/0603; LCSC Part # C2984266 -> C2290; Mfr Everlight Elec -> Hubei KENTO Elec; Mfr PN 19-213/GHC-XS1T1N/5T -> KT-0603W; Vendor PN C2984266 -> C2290
Changed lines of the file:
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@@
 			)
 		)
-		(property "Value" "EMERALD/0603"
+		(property "Value" "WHITE/0603"
 			(at 142.24 82.55 90)
 			(effects
@@
 			)
 		)
-		(property "Mfr" "Everlight Elec"
+		(property "Mfr" "Hubei KENTO Elec"
 			(at 144.78 82.55 0)
 			(effects
@@
 			)
 		)
-		(property "Mfr PN" "19-213/GHC-XS1T1N/5T"
+		(property "Mfr PN" "KT-0603W"
 			(at 144.78 82.55 0)
 			(effects
@@
 			)
 		)
-		(property "Vendor PN" "C2984266"
+		(property "Vendor PN" "C2290"
 			(at 144.78 82.55 0)
 			(effects
@@
 			)
 		)
-		(property "LCSC Part #" "C2984266"
+		(property "LCSC Part #" "C2290"
 			(at 142.24 85.09 90)
 			(effects

Commit message: Upgrade to Kicad 9
Parts:
- renumbered D60 to D7, Q9 to Q4, R89 to R26, R90 to R27, R91 to R28
Changed lines of the file:
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@@
 (kicad_sch
-	(version 20231120)
+	(version 20250114)
 	(generator "eeschema")
-	(generator_version "8.0")
+	(generator_version "9.0")
 	(paper "A4")
 	(title_block
@@
 		(shape input)
 		(at 166.37 95.25 0)
-		(fields_autoplaced yes)
 		(effects
 			(font
@@
 		(shape input)
 		(at 99.06 101.6 180)
-		(fields_autoplaced yes)
 		(effects
 			(font
@@
 		(on_board yes)
 		(dnp no)
-		(property "Reference" "#PWR0211"
+		(property "Reference" "#PWR084"
 			(at 107.95 118.11 0)
 			(effects
@@
 		(on_board yes)
 		(dnp no)
-		(property "Reference" "#PWR0212"
+		(property "Reference" "#PWR085"
 			(at 144.78 64.77 0)
 			(effects
@@
 		(on_board yes)
 		(dnp no)
-		(property "Reference" "R91"
+		(property "Reference" "R28"
 			(at 147.32 66.04 0)
 			(effects
@@
 		(on_board yes)
 		(dnp no)
-		(property "Reference" "R90"
+		(property "Reference" "R27"
 			(at 125.73 96.52 90)
 			(effects
@@
 		(on_board yes)
 		(dnp no)
-		(property "Reference" "D60"
+		(property "Reference" "D7"
 			(at 142.24 80.01 90)
 			(effects
@@
 		(on_board yes)
 		(dnp no)
-		(property "Reference" "R89"
+		(property "Reference" "R26"
 			(at 110.49 107.95 0)
 			(effects
@@
 		(on_board yes)
 		(dnp no)
-		(property "Reference" "#PWR0213"
+		(property "Reference" "#PWR086"
 			(at 144.78 119.38 0)
 			(effects
@@
 		(on_board yes)
 		(dnp no)
-		(property "Reference" "Q9"
+		(property "Reference" "Q4"
 			(at 148.59 99.06 0)
 			(effects

Commit message: Updated to 2 NTCs instead of 4.
Parts:
- Q4: symbol Device:Q_NPN_BEC -> Transistor_BJT:Q_NPN_BEC
- R26: LCSC Part # C60490 -> C25744; Mfr Yageo -> Uniroyal; Mfr PN RC0402FR-0710KL -> 0402WGF1002TCE; Vendor PN C60490 -> C25744
- R27, R28: Technology (none) -> 1%
Changed lines of the file:
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@@
 			)
 		)
-		(property "Technology" "~"
+		(property "Technology" "1%"
 			(at 144.78 68.58 0)
 			(effects
@@
 			)
 		)
-		(property "Technology" "~"
+		(property "Technology" "1%"
 			(at 125.73 101.6 0)
 			(effects
@@
 			)
 		)
-		(property "Description" ""
+		(property "Description" "Light emitting diode, small symbol"
 			(at 144.78 82.55 0)
 			(effects
@@
 		)
 		(property "JLCPCB BOM" "1"
+			(at 144.78 82.55 0)
+			(effects
+				(font
+					(size 1.27 1.27)
+				)
+				(hide yes)
+			)
+		)
+		(property "Sim.Pin" "1=K 2=A"
 			(at 144.78 82.55 0)
 			(effects
@@
 			)
 		)
-		(property "Mfr" "Yageo"
+		(property "Mfr" "Uniroyal"
 			(at 107.95 106.68 0)
 			(effects
@@
 			)
 		)
-		(property "Mfr PN" "RC0402FR-0710KL"
+		(property "Mfr PN" "0402WGF1002TCE"
 			(at 107.95 106.68 0)
 			(effects
@@
 			)
 		)
-		(property "Vendor PN" "C60490"
-			(at 107.95 106.68 0)
-			(effects
-				(font
-					(size 1.27 1.27)
-				)
-				(hide yes)
-			)
-		)
-		(property "LCSC Part #" "C60490"
+		(property "Vendor PN" "C25744"
+			(at 107.95 106.68 0)
+			(effects
+				(font
+					(size 1.27 1.27)
+				)
+				(hide yes)
+			)
+		)
+		(property "LCSC Part #" "C25744"
 			(at 110.49 113.03 0)
 			(effects
@@
 	)
 	(symbol
-		(lib_id "Device:Q_NPN_BEC")
+		(lib_id "Transistor_BJT:Q_NPN_BEC")
 		(at 142.24 101.6 0)
 		(unit 1)
@@
 			)
 		)
-		(property "Description" ""
+		(property "Description" "NPN transistor, base/emitter/collector"
 			(at 142.24 101.6 0)
 			(effects

Commit message: Version 4.1
Other:
- note added: "I_{LED} = (24V - V_{LED}) / 6.8k I_{LED} = (24V - 2.7V) / 6.8k I_{LED} = 3,13 mA"
Changed lines of the file:
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@@
 		(rev "V4")
+	)
+	(text "I_{LED} = (24V - V_{LED}) / 6.8k\nI_{LED} = (24V - 2.7V) / 6.8k\nI_{LED} = 3,13 mA"
+		(exclude_from_sim no)
+		(at 154.94 86.36 0)
+		(effects
+			(font
+				(size 1.5 1.5)
+			)
+			(justify left bottom)
+		)
 	)
 	(junction
