File: V4/esp-24v-16ch-v4.kicad_sch (KiCad schematic)
At the start: 4 parts, among them J1 DB141V-2.54-8P, J2 DB141V-2.54-8P, J3 DB141V-2.54-8P, J4 DB141V-2.54-8P

Commit message: Updating PCB for V4
Connections:
- net Outputs 1-16/J8-OUT1 renamed Output 1/OUTPUT
- net Outputs 1-16/J8-OUT2 renamed Output 2/OUTPUT
- net Outputs 1-16/J8-OUT3 renamed Output 3/OUTPUT
- net Outputs 1-16/J8-OUT4 renamed Output 4/OUTPUT
- net Outputs 1-16/J8-OUT5 renamed Output 5/OUTPUT
- net Outputs 1-16/J8-OUT6 renamed Output 6/OUTPUT
- net Outputs 1-16/J8-OUT7 renamed Output 7/OUTPUT
- net Outputs 1-16/J8-OUT8 renamed Output 8/OUTPUT
- net Outputs 1-16/J9-OUT10 renamed Output 10/OUTPUT
- net Outputs 1-16/J9-OUT11 renamed Output 11/OUTPUT
- net Outputs 1-16/J9-OUT12 renamed Output 12/OUTPUT
- net Outputs 1-16/J9-OUT13 renamed Output 13/OUTPUT
- net Outputs 1-16/J9-OUT14 renamed Output 14/OUTPUT
- net Outputs 1-16/J9-OUT15 renamed Output 15/OUTPUT
- net Outputs 1-16/J9-OUT16 renamed Output 16/OUTPUT
- net Outputs 1-16/J9-OUT9 renamed Output 9/OUTPUT
Other:
- sheet Input1 renamed Input 1
- sheet Input10 renamed Input 10
- sheet Input11 renamed Input 11
- sheet Input12 renamed Input 12
- sheet Input13 renamed Input 13
- sheet Input14 renamed Input 14
- sheet Input15 renamed Input 15
- sheet Input16 renamed Input 16
- sheet Input2 renamed Input 2
- sheet Input3 renamed Input 3
- sheet Input4 renamed Input 4
- sheet Input5 renamed Input 5
- sheet Input6 renamed Input 6
- sheet Input7 renamed Input 7
- sheet Input8 renamed Input 8
- sheet Input9 renamed Input 9
- removed sheet Outputs 1-16
- added sheet Output 1 (esp-24v-16ch-outputs.kicad_sch)
- added sheet Output 10 (esp-24v-16ch-outputs.kicad_sch)
- added sheet Output 11 (esp-24v-16ch-outputs.kicad_sch)
- added sheet Output 12 (esp-24v-16ch-outputs.kicad_sch)
- added sheet Output 13 (esp-24v-16ch-outputs.kicad_sch)
- added sheet Output 14 (esp-24v-16ch-outputs.kicad_sch)
- added sheet Output 15 (esp-24v-16ch-outputs.kicad_sch)
- added sheet Output 16 (esp-24v-16ch-outputs.kicad_sch)
- added sheet Output 2 (esp-24v-16ch-outputs.kicad_sch)
- added sheet Output 3 (esp-24v-16ch-outputs.kicad_sch)
- added sheet Output 4 (esp-24v-16ch-outputs.kicad_sch)
- added sheet Output 5 (esp-24v-16ch-outputs.kicad_sch)
- added sheet Output 6 (esp-24v-16ch-outputs.kicad_sch)
- added sheet Output 7 (esp-24v-16ch-outputs.kicad_sch)
- added sheet Output 8 (esp-24v-16ch-outputs.kicad_sch)
- added sheet Output 9 (esp-24v-16ch-outputs.kicad_sch)
- sheet Input 1: file esp-24v-16ch-v4-input1.kicad_sch -> esp-24v-16ch-v4-inputs.kicad_sch
- sheet Input 10: file esp-24v-16ch-v4-input1.kicad_sch -> esp-24v-16ch-v4-inputs.kicad_sch
- sheet Input 11: file esp-24v-16ch-v4-input1.kicad_sch -> esp-24v-16ch-v4-inputs.kicad_sch
- sheet Input 12: file esp-24v-16ch-v4-input1.kicad_sch -> esp-24v-16ch-v4-inputs.kicad_sch
- sheet Input 13: file esp-24v-16ch-v4-input1.kicad_sch -> esp-24v-16ch-v4-inputs.kicad_sch
- sheet Input 14: file esp-24v-16ch-v4-input1.kicad_sch -> esp-24v-16ch-v4-inputs.kicad_sch
- sheet Input 15: file esp-24v-16ch-v4-input1.kicad_sch -> esp-24v-16ch-v4-inputs.kicad_sch
- sheet Input 16: file esp-24v-16ch-v4-input1.kicad_sch -> esp-24v-16ch-v4-inputs.kicad_sch
- sheet Input 2: file esp-24v-16ch-v4-input1.kicad_sch -> esp-24v-16ch-v4-inputs.kicad_sch
- sheet Input 3: file esp-24v-16ch-v4-input1.kicad_sch -> esp-24v-16ch-v4-inputs.kicad_sch
- sheet Input 4: file esp-24v-16ch-v4-input1.kicad_sch -> esp-24v-16ch-v4-inputs.kicad_sch
- sheet Input 5: file esp-24v-16ch-v4-input1.kicad_sch -> esp-24v-16ch-v4-inputs.kicad_sch
- sheet Input 6: file esp-24v-16ch-v4-input1.kicad_sch -> esp-24v-16ch-v4-inputs.kicad_sch
- sheet Input 7: file esp-24v-16ch-v4-input1.kicad_sch -> esp-24v-16ch-v4-inputs.kicad_sch
- sheet Input 8: file esp-24v-16ch-v4-input1.kicad_sch -> esp-24v-16ch-v4-inputs.kicad_sch
- sheet Input 9: file esp-24v-16ch-v4-input1.kicad_sch -> esp-24v-16ch-v4-inputs.kicad_sch
- moved on the sheet: J1, J2, J3, J4

Commit message: Fabrication updates
Connections:
- net Input 1/INPUT renamed IN1
- net Input 10/INPUT renamed IN10
- net Input 11/INPUT renamed IN11
- net Input 12/INPUT renamed IN12
- net Input 13/INPUT renamed IN13
- net Input 14/INPUT renamed IN14
- net Input 15/INPUT renamed IN15
- net Input 16/INPUT renamed IN16
- net Input 2/INPUT renamed IN2
- net Input 3/INPUT renamed IN3
- net Input 4/INPUT renamed IN4
- net Input 5/INPUT renamed IN5
- net Input 6/INPUT renamed IN6
- net Input 7/INPUT renamed IN7
- net Input 8/INPUT renamed IN8
- net Input 9/INPUT renamed IN9
- net Output 1/OUTPUT renamed OUT1
- net Output 10/OUTPUT renamed OUT10
- net Output 11/OUTPUT renamed OUT11
- net Output 12/OUTPUT renamed OUT12
- net Output 13/OUTPUT renamed OUT13
- net Output 14/OUTPUT renamed OUT14
- net Output 15/OUTPUT renamed OUT15
- net Output 16/OUTPUT renamed OUT16
- net Output 2/OUTPUT renamed OUT2
- net Output 3/OUTPUT renamed OUT3
- net Output 4/OUTPUT renamed OUT4
- net Output 5/OUTPUT renamed OUT5
- net Output 6/OUTPUT renamed OUT6
- net Output 7/OUTPUT renamed OUT7
- net Output 8/OUTPUT renamed OUT8
- net Output 9/OUTPUT renamed OUT9

Commit message: Version 4.1
Parts:
- J2, J4: now not fitted
Other:
- sheet Input 1: file esp-24v-16ch-v4-inputs.kicad_sch -> esp-24v-16ch-v4-inputs1-8.kicad_sch
- sheet Input 10: file esp-24v-16ch-v4-inputs.kicad_sch -> esp-24v-16ch-v4-inputs9-16.kicad_sch
- sheet Input 11: file esp-24v-16ch-v4-inputs.kicad_sch -> esp-24v-16ch-v4-inputs9-16.kicad_sch
- sheet Input 12: file esp-24v-16ch-v4-inputs.kicad_sch -> esp-24v-16ch-v4-inputs9-16.kicad_sch
- sheet Input 13: file esp-24v-16ch-v4-inputs.kicad_sch -> esp-24v-16ch-v4-inputs9-16.kicad_sch
- sheet Input 14: file esp-24v-16ch-v4-inputs.kicad_sch -> esp-24v-16ch-v4-inputs9-16.kicad_sch
- sheet Input 15: file esp-24v-16ch-v4-inputs.kicad_sch -> esp-24v-16ch-v4-inputs9-16.kicad_sch
- sheet Input 16: file esp-24v-16ch-v4-inputs.kicad_sch -> esp-24v-16ch-v4-inputs9-16.kicad_sch
- sheet Input 2: file esp-24v-16ch-v4-inputs.kicad_sch -> esp-24v-16ch-v4-inputs1-8.kicad_sch
- sheet Input 3: file esp-24v-16ch-v4-inputs.kicad_sch -> esp-24v-16ch-v4-inputs1-8.kicad_sch
- sheet Input 4: file esp-24v-16ch-v4-inputs.kicad_sch -> esp-24v-16ch-v4-inputs1-8.kicad_sch
- sheet Input 5: file esp-24v-16ch-v4-inputs.kicad_sch -> esp-24v-16ch-v4-inputs1-8.kicad_sch
- sheet Input 6: file esp-24v-16ch-v4-inputs.kicad_sch -> esp-24v-16ch-v4-inputs1-8.kicad_sch
- sheet Input 7: file esp-24v-16ch-v4-inputs.kicad_sch -> esp-24v-16ch-v4-inputs1-8.kicad_sch
- sheet Input 8: file esp-24v-16ch-v4-inputs.kicad_sch -> esp-24v-16ch-v4-inputs1-8.kicad_sch
- sheet Input 9: file esp-24v-16ch-v4-inputs.kicad_sch -> esp-24v-16ch-v4-inputs9-16.kicad_sch
- sheet Output 1: file esp-24v-16ch-outputs.kicad_sch -> esp-24v-16ch-v4-outputs1-8.kicad_sch
- sheet Output 10: file esp-24v-16ch-outputs.kicad_sch -> esp-24v-16ch-v4-outputs9-16.kicad_sch
- sheet Output 11: file esp-24v-16ch-outputs.kicad_sch -> esp-24v-16ch-v4-outputs9-16.kicad_sch
- sheet Output 12: file esp-24v-16ch-outputs.kicad_sch -> esp-24v-16ch-v4-outputs9-16.kicad_sch
- sheet Output 13: file esp-24v-16ch-outputs.kicad_sch -> esp-24v-16ch-v4-outputs9-16.kicad_sch
- sheet Output 14: file esp-24v-16ch-outputs.kicad_sch -> esp-24v-16ch-v4-outputs9-16.kicad_sch
- sheet Output 15: file esp-24v-16ch-outputs.kicad_sch -> esp-24v-16ch-v4-outputs9-16.kicad_sch
- sheet Output 16: file esp-24v-16ch-outputs.kicad_sch -> esp-24v-16ch-v4-outputs9-16.kicad_sch
- sheet Output 2: file esp-24v-16ch-outputs.kicad_sch -> esp-24v-16ch-v4-outputs1-8.kicad_sch
- sheet Output 3: file esp-24v-16ch-outputs.kicad_sch -> esp-24v-16ch-v4-outputs1-8.kicad_sch
- sheet Output 4: file esp-24v-16ch-outputs.kicad_sch -> esp-24v-16ch-v4-outputs1-8.kicad_sch
- sheet Output 5: file esp-24v-16ch-outputs.kicad_sch -> esp-24v-16ch-v4-outputs1-8.kicad_sch
- sheet Output 6: file esp-24v-16ch-outputs.kicad_sch -> esp-24v-16ch-v4-outputs1-8.kicad_sch
- sheet Output 7: file esp-24v-16ch-outputs.kicad_sch -> esp-24v-16ch-v4-outputs1-8.kicad_sch
- sheet Output 8: file esp-24v-16ch-outputs.kicad_sch -> esp-24v-16ch-v4-outputs1-8.kicad_sch
- sheet Output 9: file esp-24v-16ch-outputs.kicad_sch -> esp-24v-16ch-v4-outputs9-16.kicad_sch
Changed lines of the file:
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@@
 		(title "ESP 24V 16xIn/16xOut/4xNTC Module")
 		(date "2025-07-04")
-		(rev "V4")
+		(rev "V4.1")
 	)
 	(wire
@@
 		(in_bom yes)
 		(on_board yes)
-		(dnp no)
+		(dnp yes)
 		(property "Reference" "J4"
 			(at 396.24 182.88 0)
@@
 		(in_bom yes)
 		(on_board yes)
-		(dnp no)
+		(dnp yes)
 		(property "Reference" "J2"
 			(at 119.38 182.88 0)
@@
 			)
 		)
-		(property "Sheetfile" "esp-24v-16ch-outputs.kicad_sch"
+		(property "Sheetfile" "esp-24v-16ch-v4-outputs1-8.kicad_sch"
 			(at 224.79 212.6746 0)
 			(effects
@@
 			)
 		)
-		(property "Sheetfile" "esp-24v-16ch-outputs.kicad_sch"
+		(property "Sheetfile" "esp-24v-16ch-v4-outputs9-16.kicad_sch"
 			(at 322.58 156.7946 0)
 			(effects
@@
 			)
 		)
-		(property "Sheetfile" "esp-24v-16ch-v4-inputs.kicad_sch"
+		(property "Sheetfile" "esp-24v-16ch-v4-inputs1-8.kicad_sch"
 			(at 57.15 240.6146 0)
 			(effects
@@
 			)
 		)
-		(property "Sheetfile" "esp-24v-16ch-outputs.kicad_sch"
+		(property "Sheetfile" "esp-24v-16ch-v4-outputs9-16.kicad_sch"
 			(at 322.58 240.6146 0)
 			(effects
@@
 			)
 		)
-		(property "Sheetfile" "esp-24v-16ch-outputs.kicad_sch"
+		(property "Sheetfile" "esp-24v-16ch-v4-outputs9-16.kicad_sch"
 			(at 322.58 170.7646 0)
 			(effects
@@
 			)
 		)
-		(property "Sheetfile" "esp-24v-16ch-v4-inputs.kicad_sch"
+		(property "Sheetfile" "esp-24v-16ch-v4-inputs1-8.kicad_sch"
 			(at 57.15 184.7346 0)
 			(effects
@@
 			)
 		)
-		(property "Sheetfile" "esp-24v-16ch-v4-inputs.kicad_sch"
+		(property "Sheetfile" "esp-24v-16ch-v4-inputs9-16.kicad_sch"
 			(at 152.4 170.7646 0)
 			(effects
@@
 			)
 		)
-		(property "Sheetfile" "esp-24v-16ch-outputs.kicad_sch"
+		(property "Sheetfile" "esp-24v-16ch-v4-outputs1-8.kicad_sch"
 			(at 224.79 170.7646 0)
 			(effects
@@
 			)
 		)
-		(property "Sheetfile" "esp-24v-16ch-v4-inputs.kicad_sch"
+		(property "Sheetfile" "esp-24v-16ch-v4-inputs1-8.kicad_sch"
 			(at 57.15 198.7046 0)
 			(effects
@@
 			)
 		)
-		(property "Sheetfile" "esp-24v-16ch-outputs.kicad_sch"
+		(property "Sheetfile" "esp-24v-16ch-v4-outputs1-8.kicad_sch"
 			(at 224.79 184.7346 0)
 			(effects
@@
 			)
 		)
-		(property "Sheetfile" "esp-24v-16ch-v4-inputs.kicad_sch"
+		(property "Sheetfile" "esp-24v-16ch-v4-inputs1-8.kicad_sch"
 			(at 57.15 212.6746 0)
 			(effects
@@
 			)
 		)
-		(property "Sheetfile" "esp-24v-16ch-outputs.kicad_sch"
+		(property "Sheetfile" "esp-24v-16ch-v4-outputs9-16.kicad_sch"
 			(at 322.58 142.8246 0)
 			(effects
@@
 			)
 		)
-		(property "Sheetfile" "esp-24v-16ch-v4-inputs.kicad_sch"
+		(property "Sheetfile" "esp-24v-16ch-v4-inputs9-16.kicad_sch"
 			(at 152.4 142.8246 0)
 			(effects
@@
 			)
 		)
-		(property "Sheetfile" "esp-24v-16ch-outputs.kicad_sch"
+		(property "Sheetfile" "esp-24v-16ch-v4-outputs9-16.kicad_sch"
 			(at 322.58 184.7346 0)
 			(effects
@@
 			)
 		)
-		(property "Sheetfile" "esp-24v-16ch-outputs.kicad_sch"
+		(property "Sheetfile" "esp-24v-16ch-v4-outputs9-16.kicad_sch"
 			(at 322.58 226.6446 0)
 			(effects
@@
 			)
 		)
-		(property "Sheetfile" "esp-24v-16ch-outputs.kicad_sch"
+		(property "Sheetfile" "esp-24v-16ch-v4-outputs1-8.kicad_sch"
 			(at 224.79 156.7946 0)
 			(effects
@@
 			)
 		)
-		(property "Sheetfile" "esp-24v-16ch-v4-inputs.kicad_sch"
+		(property "Sheetfile" "esp-24v-16ch-v4-inputs9-16.kicad_sch"
 			(at 152.4 156.7946 0)
 			(effects
@@
 			)
 		)
-		(property "Sheetfile" "esp-24v-16ch-v4-inputs.kicad_sch"
+		(property "Sheetfile" "esp-24v-16ch-v4-inputs9-16.kicad_sch"
 			(at 152.4 198.7046 0)
 			(effects
@@
 			)
 		)
-		(property "Sheetfile" "esp-24v-16ch-outputs.kicad_sch"
+		(property "Sheetfile" "esp-24v-16ch-v4-outputs1-8.kicad_sch"
 			(at 224.79 198.7046 0)
 			(effects
@@
 			)
 		)
-		(property "Sheetfile" "esp-24v-16ch-outputs.kicad_sch"
+		(property "Sheetfile" "esp-24v-16ch-v4-outputs1-8.kicad_sch"
 			(at 224.79 226.6446 0)
 			(effects
@@
 			)
 		)
-		(property "Sheetfile" "esp-24v-16ch-v4-inputs.kicad_sch"
+		(property "Sheetfile" "esp-24v-16ch-v4-inputs9-16.kicad_sch"
 			(at 152.4 212.6746 0)
 			(effects
@@
 			)
 		)
-		(property "Sheetfile" "esp-24v-16ch-v4-inputs.kicad_sch"
+		(property "Sheetfile" "esp-24v-16ch-v4-inputs1-8.kicad_sch"
 			(at 57.15 156.7946 0)
 			(effects
@@
 			)
 		)
-		(property "Sheetfile" "esp-24v-16ch-v4-inputs.kicad_sch"
+		(property "Sheetfile" "esp-24v-16ch-v4-inputs9-16.kicad_sch"
 			(at 152.4 240.6146 0)
 			(effects
@@
 			)
 		)
-		(property "Sheetfile" "esp-24v-16ch-v4-inputs.kicad_sch"
+		(property "Sheetfile" "esp-24v-16ch-v4-inputs9-16.kicad_sch"
 			(at 152.4 184.7346 0)
 			(effects
@@
 			)
 		)
-		(property "Sheetfile" "esp-24v-16ch-outputs.kicad_sch"
+		(property "Sheetfile" "esp-24v-16ch-v4-outputs9-16.kicad_sch"
 			(at 322.58 198.7046 0)
 			(effects
@@
 			)
 		)
-		(property "Sheetfile" "esp-24v-16ch-v4-inputs.kicad_sch"
+		(property "Sheetfile" "esp-24v-16ch-v4-inputs9-16.kicad_sch"
 			(at 152.4 226.6446 0)
 			(effects
@@
 			)
 		)
-		(property "Sheetfile" "esp-24v-16ch-outputs.kicad_sch"
+		(property "Sheetfile" "esp-24v-16ch-v4-outputs9-16.kicad_sch"
 			(at 322.58 212.6746 0)
 			(effects
@@
 			)
 		)
-		(property "Sheetfile" "esp-24v-16ch-v4-inputs.kicad_sch"
+		(property "Sheetfile" "esp-24v-16ch-v4-inputs1-8.kicad_sch"
 			(at 57.15 226.6446 0)
 			(effects
@@
 			)
 		)
-		(property "Sheetfile" "esp-24v-16ch-outputs.kicad_sch"
+		(property "Sheetfile" "esp-24v-16ch-v4-outputs1-8.kicad_sch"
 			(at 224.79 240.6146 0)
 			(effects
@@
 			)
 		)
-		(property "Sheetfile" "esp-24v-16ch-v4-inputs.kicad_sch"
+		(property "Sheetfile" "esp-24v-16ch-v4-inputs1-8.kicad_sch"
 			(at 57.15 142.8246 0)
 			(effects
@@
 			)
 		)
-		(property "Sheetfile" "esp-24v-16ch-v4-inputs.kicad_sch"
+		(property "Sheetfile" "esp-24v-16ch-v4-inputs1-8.kicad_sch"
 			(at 57.15 170.7646 0)
 			(effects
@@
 			)
 		)
-		(property "Sheetfile" "esp-24v-16ch-outputs.kicad_sch"
+		(property "Sheetfile" "esp-24v-16ch-v4-outputs1-8.kicad_sch"
 			(at 224.79 142.8246 0)
 			(effects

Commit message: Version 4.1
Parts:
- J2, J4: now fitted
Changed lines of the file:
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@@
 		(in_bom yes)
 		(on_board yes)
-		(dnp yes)
+		(dnp no)
 		(property "Reference" "J4"
 			(at 396.24 182.88 0)
@@
 		(in_bom yes)
 		(on_board yes)
-		(dnp yes)
+		(dnp no)
 		(property "Reference" "J2"
 			(at 119.38 182.88 0)

Commit message: Rerouting
Parts:
- added FID1, FID2, FID3: Fiducial, Fiducial:Fiducial_1mm_Mask2mm, symbol Mechanical:Fiducial
Other:
- sheet I2C Devices ports: added I2CSCL, I2CSDA, MCPININTA, MCPININTB; removed I2C_SCL, I2C_SDA, MCP1-INTA, MCP1-INTB
- sheet Input 1 ports: added MUXIN; removed MUX_IN
- sheet Input 10 ports: added MUXIN; removed MUX_IN
- sheet Input 11 ports: added MUXIN; removed MUX_IN
- sheet Input 12 ports: added MUXIN; removed MUX_IN
- sheet Input 13 ports: added MUXIN; removed MUX_IN
- sheet Input 14 ports: added MUXIN; removed MUX_IN
- sheet Input 15 ports: added MUXIN; removed MUX_IN
- sheet Input 16 ports: added MUXIN; removed MUX_IN
- sheet Input 2 ports: added MUXIN; removed MUX_IN
- sheet Input 3 ports: added MUXIN; removed MUX_IN
- sheet Input 4 ports: added MUXIN; removed MUX_IN
- sheet Input 5 ports: added MUXIN; removed MUX_IN
- sheet Input 6 ports: added MUXIN; removed MUX_IN
- sheet Input 7 ports: added MUXIN; removed MUX_IN
- sheet Input 8 ports: added MUXIN; removed MUX_IN
- sheet Input 9 ports: added MUXIN; removed MUX_IN
- sheet LAN ports: added EMACCLK, EMACMDC, EMACMDIO, EMACRX, EMACRXD0, EMACRXD1, EMACTXD0, EMACTXD1, EMACTXEN; removed EMAC_CLK, EMAC_MDC, EMAC_MDIO, EMAC_RX, EMAC_RXD0, EMAC_RXD1, EMAC_TXD0, EMAC_TXD1, EMAC_TXEN
- sheet MCU ports: added EMACCLK, EMACMDC, EMACMDIO, EMACRX, EMACRXD0, EMACRXD1, EMACTXD0, EMACTXD1, EMACTXEN, I2CSCL, I2CSDA, MCPININTA, MCPININTB, USBD+, USBD-; removed EMAC_CLK, EMAC_MDC, EMAC_MDIO, EMAC_RX, EMAC_RXD0, EMAC_RXD1, EMAC_TXD0, EMAC_TXD1, EMAC_TXEN, I2C_SCL, I2C_SDA, MCP1-INTA, MCP1-INTB, USB_D+, USB_D-
- sheet Output 1 ports: added MUXOUT; removed MUX_OUT
- sheet Output 10 ports: added MUXOUT; removed MUX_OUT
- sheet Output 11 ports: added MUXOUT; removed MUX_OUT
- sheet Output 12 ports: added MUXOUT; removed MUX_OUT
- sheet Output 13 ports: added MUXOUT; removed MUX_OUT
- sheet Output 14 ports: added MUXOUT; removed MUX_OUT
- sheet Output 15 ports: added MUXOUT; removed MUX_OUT
- sheet Output 16 ports: added MUXOUT; removed MUX_OUT
- sheet Output 2 ports: added MUXOUT; removed MUX_OUT
- sheet Output 3 ports: added MUXOUT; removed MUX_OUT
- sheet Output 4 ports: added MUXOUT; removed MUX_OUT
- sheet Output 5 ports: added MUXOUT; removed MUX_OUT
- sheet Output 6 ports: added MUXOUT; removed MUX_OUT
- sheet Output 7 ports: added MUXOUT; removed MUX_OUT
- sheet Output 8 ports: added MUXOUT; removed MUX_OUT
- sheet Output 9 ports: added MUXOUT; removed MUX_OUT
- sheet Power ports: added USBD+, USBD-; removed USB_D+, USB_D-

Commit message: Rerouting
Other:
- sheet MCU ports: added PHYPWR; removed PHY_PWR
- sheet Power ports: added PHYPWR; removed PHY_PWR
Changed lines of the file:
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@@
 			)
 		)
-		(pin "PHY_PWR" input
+		(pin "PHYPWR" input
 			(at 146.05 34.29 0)
 			(effects
@@
 			)
 		)
-		(pin "PHY_PWR" output
+		(pin "PHYPWR" output
 			(at 165.1 34.29 180)
 			(effects
