File: V4/esp-24v-16ch-v4-inputs9-16.kicad_sch (KiCad schematic)
At the start: 10 parts, among them U12 OR-3H7-4

Commit message: Version 4.1
Parts:
- C43, C44, D33, D34, FB9, R53, R54, R55, U12: now fitted

Commit message: Revising schematics
Connections:
- net +3.3V renamed +3V3
Changed lines of the file:
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@@
 			)
 		)
-		(property "Value" "+3.3V"
+		(property "Value" "+3V3"
 			(at 194.691 76.8858 0)
 			(effects

Commit message: Revising the schematics
Parts:
- R55: value 2k2/62,5mW -> 2k2
Changed lines of the file:
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@@
 			)
 		)
-		(property "Value" "2k2/62,5mW"
+		(property "Value" "2k2"
 			(at 196.85 82.55 0)
 			(effects

Commit message: Rerouting
Connections:
- net INFILTER: now reaches C44.1, D34.1 (K), R54.1
- net INPRE: now reaches D32.1 (A1), FB9.2, R53.1, R54.2
- net INLED: now reaches D33.2 (A), R53.2
- net INOPTO: now reaches D34.2 (A), U12.1
- net MUX_IN renamed MUXIN
Other:
- moved on the sheet: D33, D34, R55, U12A

Commit message: Rerouting
Parts:
- R64: renamed from R53; value 6,8k/100mW -> 10k/100mW; LCSC Part # C23212 -> C25804; Mfr PN 0603WAF6801T5E -> 0603WAF1002T5E; Vendor PN C23212 -> C25804
- renumbered C43 to C46, C44 to C47, D32 to D33, D33 to D34, D34 to D35, R54 to R65, R55 to R66, U12 to U11
