File: V4/esp-24v-16ch-v4-outputs9-16.kicad_sch (KiCad schematic)
At the start: 5 parts, among them Q4 MMBT2222A

Commit message: Version 4.1
Parts:
- D63: renamed from D7; now not fitted
- Q12: renamed from Q4; now not fitted
- R100: renamed from R28; now not fitted
- R98: renamed from R26; now not fitted
- R99: renamed from R27; now not fitted
Changed lines of the file:
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@@
 		(title "ESP 24V 16xIn/16xOut/4xNTC Module")
 		(date "2025-07-04")
-		(rev "V4")
+		(rev "V4.1")
 	)
 	(text "I_{LED} = (24V - V_{LED}) / 6.8k\nI_{LED} = (24V - 2.7V) / 6.8k\nI_{LED} = 3,13 mA"
@@
 		(on_board yes)
 		(dnp no)
-		(property "Reference" "#PWR084"
+		(property "Reference" "#PWR0220"
 			(at 107.95 118.11 0)
 			(effects
@@
 		(on_board yes)
 		(dnp no)
-		(property "Reference" "#PWR085"
+		(property "Reference" "#PWR0221"
 			(at 144.78 64.77 0)
 			(effects
@@
 		(in_bom yes)
 		(on_board yes)
-		(dnp no)
-		(property "Reference" "R28"
+		(dnp yes)
+		(property "Reference" "R100"
 			(at 147.32 66.04 0)
 			(effects
@@
 		(in_bom yes)
 		(on_board yes)
-		(dnp no)
-		(property "Reference" "R27"
+		(dnp yes)
+		(property "Reference" "R99"
 			(at 125.73 96.52 90)
 			(effects
@@
 		(in_bom yes)
 		(on_board yes)
-		(dnp no)
-		(property "Reference" "D7"
+		(dnp yes)
+		(property "Reference" "D63"
 			(at 142.24 80.01 90)
 			(effects
@@
 		(in_bom yes)
 		(on_board yes)
-		(dnp no)
-		(property "Reference" "R26"
+		(dnp yes)
+		(property "Reference" "R98"
 			(at 110.49 107.95 0)
 			(effects
@@
 		(on_board yes)
 		(dnp no)
-		(property "Reference" "#PWR086"
+		(property "Reference" "#PWR0222"
 			(at 144.78 119.38 0)
 			(effects
@@
 		(in_bom yes)
 		(on_board yes)
-		(dnp no)
-		(property "Reference" "Q4"
+		(dnp yes)
+		(property "Reference" "Q12"
 			(at 148.59 99.06 0)
 			(effects

Commit message: Version 4.1
Parts:
- D63, Q12, R100, R98, R99: now fitted

Commit message: Revising the schematics
Parts:
- R98: value 10k/62,5mW -> 10k
- R99: value 1k/62,5mW -> 1k
Changed lines of the file:
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@@
 			)
 		)
-		(property "Value" "1k/62,5mW"
+		(property "Value" "1k"
 			(at 125.73 99.06 90)
 			(effects
@@
 			)
 		)
-		(property "Value" "10k/62,5mW"
+		(property "Value" "10k"
 			(at 110.49 110.49 0)
 			(effects

Commit message: Rerouting
Connections:
- net OUTLED: now reaches D63.2 (A), R100.2
- net OUTBASE: now reaches Q12.1 (B), R99.1
- net MUX_OUT renamed MUXOUT
Other:
- moved on the sheet: R100, R98, R99

Commit message: Rerouting
Parts:
- removed D63: WHITE/0603, Tales:LED_0603_1608Metric, symbol Device:LED_Small
- removed R100: 6,8k/100mW, Tales:R_0603_1608Metric, symbol Device:R_US
- removed R98: 10k, Tales:R_0402_1005Metric, symbol Device:R_US
- removed R99: 1k, Tales:R_0402_1005Metric, symbol Device:R_US
- added D65: WHITE/0603, Tales:LED_0603_1608Metric, symbol Device:LED_Small
- added R112: 10k, Tales:R_0402_1005Metric, symbol Device:R_US
- added R113: 1k, Tales:R_0402_1005Metric, symbol Device:R_US
- added R114: 10k/100mW, Tales:R_0603_1608Metric, symbol Device:R_US
Connections:
- net +24V: now also R114.1
- net GND: now also R112.1
- net MUXOUT: now also R112.2, R113.2
- net OUTBASE: now also R113.1
- net OUTLED: now also D65.2 (A), R114.2
- net OUTPUT: now also D65.1 (K)
