File: V5/esp-24v-16ch-v5-lan.kicad_sch (KiCad schematic)
At the start: 19 parts, among them J7 ETHERNET, U5 LAN8710A

Commit message: Created V5
Parts:
- removed RN1, RN2: 4x2,2k/62,5mW, Tales:R_Array_Convex_4x0402, symbol Device:R_Pack04
- removed RN3: 4x49,9R/62,5mW, Tales:R_Array_Convex_4x0402, symbol Device:R_Pack04
- added R20, R21, R22, R23, R24, R25, R26, R27: 2k2, Tales:R_0402_1005Metric, symbol Device:R_US
- added R30, R31, R32, R33: 49,9R, Tales:R_0402_1005Metric, symbol Device:R_US
- R28: renamed from R22; value 10k/62,5mW -> 10k
- R29: renamed from R23; value 12,1k/62,5mW -> 12,1k
- R34: renamed from R20; value 330R/62,5mW -> 330R
- R35: renamed from R21; value 330R/62,5mW -> 330R
- renumbered C20 to C19, C21 to C20, C22 to C21, C23 to C22, C24 to C23, C19 to C24, C17 to C25, C16 to C26, D6 to D7, J7 to J3
Connections:
- net GND: now also R25.1, R26.1, R27.1
- net ETHLEDYA: now reaches J3.12, R35.2
- net ETHSH: now reaches C26.1, J3.SH
- net ETHLEDGA: now reaches J3.9, R34.2
- net RXD2: now reaches U5.9 (RXD2/~{RMIISEL})
- net RXD2: now also R24.2
- net VCDDR: now reaches C22.1, C23.1, U5.6 (VDDCR)
- net RXER: now reaches U5.13 (RXER/RXD4/~{PHYAD0})
- net RXER: now also R25.2
- net RBIAS: now reaches R29.1, U5.32 (RBIAS)
- net RXCLK: now reaches U5.7 (RXCLK/~{PHYAD1})
- net RXCLK: now also R26.2
- net RXD3: now reaches U5.8 (RXD3/~{PHYAD2})
- net RXD3: now also R27.2
- net +3.3VA renamed +3V3A
- net +3V3A: now also R30.2, R31.2, R32.2, R33.2
- net +3.3VLAN renamed +3V3LAN
- net +3V3LAN: now also R20.1, R21.1, R22.1, R23.1, R24.1
- net EMAC_CLK renamed EMACCLK
- net EMAC_MDC renamed EMACMDC
- net EMAC_MDIO renamed EMACMDIO
- net EMACMDIO: now also R23.2
- net EMAC_RX renamed EMACRX
- net EMACRX: now also R22.2
- net EMAC_RXD0 renamed EMACRXD0
- net EMACRXD0: now also R20.2
- net EMAC_RXD1 renamed EMACRXD1
- net EMACRXD1: now also R21.2
- net EMAC_TXD0 renamed EMACTXD0
- net EMAC_TXD1 renamed EMACTXD1
- net EMAC_TXEN renamed EMACTXEN
- net LED_G_K renamed ETHLEDGK
- net LED_Y_A renamed ETHLEDY
- net RD+ renamed ETHRXD+
- net ETHRXD+: now also R30.1
- net RD- renamed ETHRXD-
- net ETHRXD-: now also R31.1
- net TD+ renamed ETHTXD+
- net ETHTXD+: now also R32.1
- net TD- renamed ETHTXD-
- net ETHTXD-: now also R33.1
- net /PHY_RST renamed PHYNRST
Other:
- note added: "RESISTORS: 62,5mW WHERE NOT SPECIFIED"
- title: ESP 24V 16xIn/16xOut/4xNTC Module -> ESP 24V 16xIn/16xOut/1-Wire Module
- moved on the sheet: C18, C19, C24, C26, R28, R29, R34, R35

Commit message: Reviewed capacitor sizes and voltages.
Parts:
- C18, C24: value 10uF/10V -> 10uF/25V; footprint Tales:C_0603_1608Metric -> Tales:C_0805_2012Metric; Case 0603/1608 -> 0805/2012; LCSC Part # C19702 -> C15850; Mfr PN CL10A106KP8NNNC -> CL21A106KAYNNNE; Vendor PN C19702 -> C15850
- J3: footprint Tales:RJ45_HanRun_HR911105A -> Tales:RJ45_HanRun_HR915340A; symbol Tales:RJ45_HanRun_HR911105A -> Tales:RJ45_HanRun_HR915340A
- R28: Package 0402/1005 -> (none)
Connections:
- net +3V3A: no longer R34.1
- net +3V3LAN: now also R34.1
- net ETHLEDYA: now also J3.11; no longer J3.12
- net GND: now also J3.12; no longer J3.11

Commit message: Inputs GND separated from main GND.
Parts:
- renumbered C26 to C18, C25 to C19, C24 to C20, C18 to C21, C19 to C22, C20 to C23, C21 to C24, C22 to C25, C23 to C26, J3 to J8, R34 to R20, R20 to R21, R35 to R22, R21 to R23, R22 to R24, R23 to R25, R24 to R26, R25 to R27, R26 to R28, R27 to R29, R28 to R30, R29 to R31, R30 to R32, R32 to R33, R31 to R34, R33 to R35
