File: V5/esp-24v-16ch-v5-mcu.kicad_sch (KiCad schematic)
At the start: 17 parts, among them Q3 UMH3N, SW1 RESET, U3 CH340K, U4 ESP32-WROOM-32UE-N16

Commit message: V5.2
Other:
- note added: "TEMPLATE FOR GPIO ASSIGNMENT {"NAME":"ESP-24V-16CH-V5","GPIO":[0,3200,0,3232,0,0,0,0,5536,10240,10241,0,0, 0,5600,0,0,0,0,5568,0,0,0,0,0,0,0,0,608,640,192,193,0,0,0,0],"FLAG":0,"BASE":1} See https://tasmota.github.io/docs/Templates/"
- note added: "TEMPLATE FOR MCP23017 I/O ASSIGNMENT {"NAME":"MCP23017 expander","BASE":0,"GPIO":[192,193,194,195,196,197,198,0,199,200,201, 202,203,204,205,0,224,225,226,227,228,229,230,231,232,233,234,235,236,237,238,239]} Save as mcp23x.dat and load into tasmota's filesystem. See https://tasmota.github.io/docs/MCP230xx/"
- note removed: "TEMPLATE FOR GPIO ASSIGNMENT {"NAME":"ESP-24V-16CH-V5","GPIO":[0,3200,0,3232,0,0,0,0,5536,10240,10241,0,0, 0,5600,0,0,0,0,5568,0,0,0,0,0,0,0,0,608,640,0,0,0,0,0,0],"FLAG":0,"BASE":1} See https://tasmota.github.io/docs/Templates/"
- note removed: "TEMPLATE FOR MCP23017 I/O ASSIGNMENT {"NAME":"MCP23017 expander","BASE":0,"GPIO":[160,161,162,163,164,165,166,167,168,169,170, 171,172,173,174,175,224,225,226,227,228,229,230,231,232,233,234,235,236,237,238,239]} Save as mcp23x.dat and load into tasmota's filesystem. See https://tasmota.github.io/docs/MCP230xx/"
Changed lines of the file:
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@@
 		)
 	)
-	(text "TEMPLATE FOR GPIO ASSIGNMENT\n\n{\"NAME\":\"ESP-24V-16CH-V5\",\"GPIO\":[0,3200,0,3232,0,0,0,0,5536,10240,10241,0,0,\n0,5600,0,0,0,0,5568,0,0,0,0,0,0,0,0,608,640,0,0,0,0,0,0],\"FLAG\":0,\"BASE\":1}\n\nSee https://tasmota.github.io/docs/Templates/"
+	(text "TEMPLATE FOR GPIO ASSIGNMENT\n\n{\"NAME\":\"ESP-24V-16CH-V5\",\"GPIO\":[0,3200,0,3232,0,0,0,0,5536,10240,10241,0,0,\n0,5600,0,0,0,0,5568,0,0,0,0,0,0,0,0,608,640,192,193,0,0,0,0],\"FLAG\":0,\"BASE\":1}\n\nSee https://tasmota.github.io/docs/Templates/"
 		(exclude_from_sim no)
 		(at 15.24 134.62 0)
@@
 		)
 	)
-	(text "TEMPLATE FOR MCP23017 I/O ASSIGNMENT\n\n{\"NAME\":\"MCP23017 expander\",\"BASE\":0,\"GPIO\":[160,161,162,163,164,165,166,167,168,169,170,\n171,172,173,174,175,224,225,226,227,228,229,230,231,232,233,234,235,236,237,238,239]}\n\nSave as mcp23x.dat and load into tasmota's filesystem.\nSee https://tasmota.github.io/docs/MCP230xx/"
+	(text "TEMPLATE FOR MCP23017 I/O ASSIGNMENT\n\n{\"NAME\":\"MCP23017 expander\",\"BASE\":0,\"GPIO\":[192,193,194,195,196,197,198,0,199,200,201,\n202,203,204,205,0,224,225,226,227,228,229,230,231,232,233,234,235,236,237,238,239]}\n\nSave as mcp23x.dat and load into tasmota's filesystem.\nSee https://tasmota.github.io/docs/MCP230xx/"
 		(exclude_from_sim no)
 		(at 15.24 152.4 0)

Commit message: Reviewed capacitor sizes and voltages.
Parts:
- C13, C16: value 10uF/10V -> 10uF/25V; footprint Tales:C_0603_1608Metric -> Tales:C_0805_2012Metric; Case 0603/1608 -> 0805/2012; LCSC Part # C19702 -> C15850; Mfr PN CL10A106KP8NNNC -> CL21A106KAYNNNE; Vendor PN C19702 -> C15850
- C14, C15, R12, R13, R16: Package 0402/1005 -> (none)

Commit message: Removed INTB connection from inputs MCP23017
Parts:
- removed R15: 2k2, Tales:R_0402_1005Metric, symbol Device:R_US
Connections:
- net MCPININTB: no longer names the net of U4.13 (IO14)
- no-connect marks 13 -> 14
Other:
- note added: "TEMPLATE FOR MCP23017 I/O ASSIGNMENT {"NAME":"MCP23017 expander","BASE":0,"GPIO":[192,193,194,195,196,197,198,0,199,200,201, 202,203,204,205,0,224,225,226,227,228,229,230,231,232,233,234,235,236,237,238,239], "IOCON":0x5C} Save as mcp23x.dat and load into tasmota's filesystem. See https://tasmota.github.io/docs/MCP230xx/"
- note removed: "TEMPLATE FOR MCP23017 I/O ASSIGNMENT {"NAME":"MCP23017 expander","BASE":0,"GPIO":[192,193,194,195,196,197,198,0,199,200,201, 202,203,204,205,0,224,225,226,227,228,229,230,231,232,233,234,235,236,237,238,239]} Save as mcp23x.dat and load into tasmota's filesystem. See https://tasmota.github.io/docs/MCP230xx/"

Commit message: Inputs GND separated from main GND.
Parts:
- added R16: 2k2, Tales:R_0402_1005Metric, symbol Device:R_US
- renumbered R17 to R14, R14 to R15, R18 to R17, R16 to R18
Connections:
- net +3V3: now also R16.1
- net MCPIN2INT: now reaches U4.13 (IO14)
- net MCPIN2INT: now also R16.2
- net INPUT1: no longer names the net of U4.6 (IO34)
- net INPUT2: no longer names the net of U4.7 (IO35)
- net MCPININTA renamed MCPIN1INT
- no-connect marks 14 -> 15
