File: V6/eumesmo-io-24v16ch-v6-inputs1-8.kicad_sch (KiCad schematic)
At the start: 10 parts, among them U12 OR-3H7-4

Commit message: Replaced 0603 10k resistors for 0805.
Parts:
- C35, C36, FB1, U12: FT Rotation Offset (none) -> 0; JLCPCB BOM 1 -> (none)
- D11: renamed from D13; FT Rotation Offset (none) -> 0; JLCPCB BOM 1 -> (none)
- D12: renamed from D11; JLCPCB BOM 1 -> (none)
- D13: renamed from D12; FT Rotation Offset (none) -> 0; JLCPCB BOM 1 -> (none)
- R42: renamed from R44; value 2k2 -> 2,2k; FT Rotation Offset (none) -> 0; JLCPCB BOM 1 -> (none)
- R43: value 1k8/125mW -> 1,8k/125mW; FT Rotation Offset (none) -> 0; JLCPCB BOM 1 -> (none)
- R44: renamed from R42; value 10k/100mW -> 10k/125mW; footprint Tales:R_0603_1608Metric -> Tales:R_0805_2012Metric; Case 0603/1608 -> 0805/2012; FT Rotation Offset (none) -> 0; JLCPCB BOM 1 -> (none); LCSC Part # C25804 -> C17414; Mfr PN 0603WAF1002T5E -> 0805W8F1002T5E; Vendor PN C25804 -> C17414
