File: V6/eumesmo-io-24v16ch-v6-inputs9-16.kicad_sch (KiCad schematic)
At the start: 10 parts, among them U14 OR-3H7-4

Commit message: Replaced 0603 10k resistors for 0805.
Parts:
- C51, C52, FB9, U14: FT Rotation Offset (none) -> 0; JLCPCB BOM 1 -> (none)
- D35: renamed from D37; FT Rotation Offset (none) -> 0; JLCPCB BOM 1 -> (none)
- D36: renamed from D35; JLCPCB BOM 1 -> (none)
- D37: renamed from D36; FT Rotation Offset (none) -> 0; JLCPCB BOM 1 -> (none)
- R66: renamed from R68; value 2k2 -> 2,2k; FT Rotation Offset (none) -> 0; JLCPCB BOM 1 -> (none)
- R67: value 1k8/125mW -> 1,8k/125mW; FT Rotation Offset (none) -> 0; JLCPCB BOM 1 -> (none)
- R68: renamed from R66; value 10k/100mW -> 10k/125mW; footprint Tales:R_0603_1608Metric -> Tales:R_0805_2012Metric; Case 0603/1608 -> 0805/2012; FT Rotation Offset (none) -> 0; JLCPCB BOM 1 -> (none); LCSC Part # C25804 -> C17414; Mfr PN 0603WAF1002T5E -> 0805W8F1002T5E; Vendor PN C25804 -> C17414
