File: V6/eumesmo-io-24v16ch-v6-outputs9-16.kicad_sch (KiCad schematic)
At the start: 5 parts, among them Q12 MMBT2222A

Commit message: Replaced 0603 10k resistors for 0805.
Parts:
- D67, Q12, R115: FT Rotation Offset (none) -> 0; JLCPCB BOM 1 -> (none)
- R114: renamed from R116; value 10k/100mW -> 10k/125mW; footprint Tales:R_0603_1608Metric -> Tales:R_0805_2012Metric; Case 0603/1608 -> 0805/2012; FT Rotation Offset (none) -> 0; JLCPCB BOM 1 -> (none); LCSC Part # C25804 -> C17414; Mfr PN 0603WAF1002T5E -> 0805W8F1002T5E; Vendor PN C25804 -> C17414
- R116: renamed from R114; FT Rotation Offset (none) -> 0; JLCPCB BOM 1 -> (none); LCSC Part # C25744 -> C60490; Mfr Uniroyal -> Yageo; Mfr PN 0402WGF1002TCE -> RC0402FR-0710KL; Vendor PN C25744 -> C60490
Changed lines of the file:
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@@
 		(in_pos_files yes)
 		(dnp no)
-		(property "Reference" "#PWR0239"
+		(property "Reference" "#PWR0238"
 			(at 144.78 58.42 0)
 			(hide yes)
@@
 			(project "eumesmo-io-24v16ch-v6"
 				(path "/2bc5a21a-1d79-419d-a592-6852cc07b00a/118d8d95-c0ce-4d84-8406-4e7809444f6f"
-					(reference "#PWR0242")
+					(reference "#PWR0241")
 					(unit 1)
 				)
 				(path "/2bc5a21a-1d79-419d-a592-6852cc07b00a/18f82f59-0c23-40f7-8b4c-a32f0bda1493"
-					(reference "#PWR0260")
+					(reference "#PWR0259")
 					(unit 1)
 				)
 				(path "/2bc5a21a-1d79-419d-a592-6852cc07b00a/1c051e73-1175-469e-a364-cac197036f64"
-					(reference "#PWR0245")
+					(reference "#PWR0244")
 					(unit 1)
 				)
 				(path "/2bc5a21a-1d79-419d-a592-6852cc07b00a/58d16e81-f114-46b0-87d3-9324f007724a"
-					(reference "#PWR0239")
+					(reference "#PWR0238")
 					(unit 1)
 				)
 				(path "/2bc5a21a-1d79-419d-a592-6852cc07b00a/609d2beb-47a4-466a-8275-c7d831b810a1"
-					(reference "#PWR0248")
+					(reference "#PWR0247")
 					(unit 1)
 				)
 				(path "/2bc5a21a-1d79-419d-a592-6852cc07b00a/7ca24c0f-2468-4efa-8ee6-749df6aa5e15"
-					(reference "#PWR0257")
+					(reference "#PWR0256")
 					(unit 1)
 				)
 				(path "/2bc5a21a-1d79-419d-a592-6852cc07b00a/da3c2bc1-d321-4b0b-8d45-9bd0460c9e5a"
-					(reference "#PWR0251")
+					(reference "#PWR0250")
 					(unit 1)
 				)
 				(path "/2bc5a21a-1d79-419d-a592-6852cc07b00a/dbf038c9-8c09-4484-aee5-b965d923f833"
-					(reference "#PWR0254")
+					(reference "#PWR0253")
 					(unit 1)
 				)
@@
 			)
 		)
-		(property "JLCPCB BOM" "1"
-			(at 142.24 101.6 0)
-			(hide yes)
-			(show_name no)
-			(do_not_autoplace no)
-			(effects
-				(font
-					(size 1.27 1.27)
-				)
-			)
-		)
 		(property "LCSC Part #" "C8512"
 			(at 148.59 104.14 0)
@@
 			)
 		)
-		(property "Sim.Device" "NPN"
-			(at 142.24 101.6 0)
-			(hide yes)
-			(show_name no)
-			(do_not_autoplace no)
-			(effects
-				(font
-					(size 1.27 1.27)
-				)
-			)
-		)
-		(property "Sim.Pins" "1=B 2=E 3=C"
+		(property "FT Rotation Offset" "0"
 			(at 142.24 101.6 0)
 			(hide yes)
@@
 			)
 		)
-		(property "JLCPCB BOM" "1"
-			(at 119.38 101.6 0)
+		(property "FT Rotation Offset" "0"
+			(at 119.38 101.6 90)
 			(hide yes)
 			(show_name no)
@@
 		(in_pos_files yes)
 		(dnp no)
-		(property "Reference" "#PWR0238"
+		(property "Reference" "#PWR0239"
 			(at 101.6 118.11 0)
 			(hide yes)
@@
 			(project "eumesmo-io-24v16ch-v6"
 				(path "/2bc5a21a-1d79-419d-a592-6852cc07b00a/118d8d95-c0ce-4d84-8406-4e7809444f6f"
-					(reference "#PWR0241")
+					(reference "#PWR0242")
 					(unit 1)
 				)
 				(path "/2bc5a21a-1d79-419d-a592-6852cc07b00a/18f82f59-0c23-40f7-8b4c-a32f0bda1493"
-					(reference "#PWR0259")
+					(reference "#PWR0260")
 					(unit 1)
 				)
 				(path "/2bc5a21a-1d79-419d-a592-6852cc07b00a/1c051e73-1175-469e-a364-cac197036f64"
-					(reference "#PWR0244")
+					(reference "#PWR0245")
 					(unit 1)
 				)
 				(path "/2bc5a21a-1d79-419d-a592-6852cc07b00a/58d16e81-f114-46b0-87d3-9324f007724a"
-					(reference "#PWR0238")
+					(reference "#PWR0239")
 					(unit 1)
 				)
 				(path "/2bc5a21a-1d79-419d-a592-6852cc07b00a/609d2beb-47a4-466a-8275-c7d831b810a1"
-					(reference "#PWR0247")
+					(reference "#PWR0248")
 					(unit 1)
 				)
 				(path "/2bc5a21a-1d79-419d-a592-6852cc07b00a/7ca24c0f-2468-4efa-8ee6-749df6aa5e15"
-					(reference "#PWR0256")
+					(reference "#PWR0257")
 					(unit 1)
 				)
 				(path "/2bc5a21a-1d79-419d-a592-6852cc07b00a/da3c2bc1-d321-4b0b-8d45-9bd0460c9e5a"
-					(reference "#PWR0250")
+					(reference "#PWR0251")
 					(unit 1)
 				)
 				(path "/2bc5a21a-1d79-419d-a592-6852cc07b00a/dbf038c9-8c09-4484-aee5-b965d923f833"
-					(reference "#PWR0253")
+					(reference "#PWR0254")
 					(unit 1)
 				)
@@
 		(in_pos_files yes)
 		(dnp no)
-		(property "Reference" "R114"
+		(property "Reference" "R116"
 			(at 104.14 107.95 0)
 			(show_name no)
@@
 			)
 		)
-		(property "Mfr" "Uniroyal"
+		(property "Mfr" "Yageo"
 			(at 101.6 106.68 0)
 			(hide yes)
@@
 			)
 		)
-		(property "Mfr PN" "0402WGF1002TCE"
+		(property "Mfr PN" "RC0402FR-0710KL"
 			(at 101.6 106.68 0)
 			(hide yes)
@@
 			)
 		)
-		(property "Vendor PN" "C25744"
+		(property "Vendor PN" "C60490"
 			(at 101.6 106.68 0)
 			(hide yes)
@@
 			)
 		)
-		(property "LCSC Part #" "C25744"
+		(property "LCSC Part #" "C60490"
 			(at 104.14 113.03 0)
 			(show_name no)
@@
 				)
 				(justify right)
-			)
-		)
-		(property "JLCPCB BOM" "1"
-			(at 101.6 106.68 0)
-			(hide yes)
-			(show_name no)
-			(do_not_autoplace no)
-			(effects
-				(font
-					(size 1.27 1.27)
-				)
 			)
 		)
@@
 		)
 		(property "Case" "0402/1005"
+			(at 101.6 106.68 0)
+			(hide yes)
+			(show_name no)
+			(do_not_autoplace no)
+			(effects
+				(font
+					(size 1.27 1.27)
+				)
+			)
+		)
+		(property "FT Rotation Offset" "0"
 			(at 101.6 106.68 0)
 			(hide yes)
@@
 			(project "eumesmo-io-24v16ch-v6"
 				(path "/2bc5a21a-1d79-419d-a592-6852cc07b00a/118d8d95-c0ce-4d84-8406-4e7809444f6f"
-					(reference "R117")
+					(reference "R119")
 					(unit 1)
 				)
 				(path "/2bc5a21a-1d79-419d-a592-6852cc07b00a/18f82f59-0c23-40f7-8b4c-a32f0bda1493"
-					(reference "R135")
+					(reference "R137")
 					(unit 1)
 				)
 				(path "/2bc5a21a-1d79-419d-a592-6852cc07b00a/1c051e73-1175-469e-a364-cac197036f64"
-					(reference "R120")
+					(reference "R122")
 					(unit 1)
 				)
 				(path "/2bc5a21a-1d79-419d-a592-6852cc07b00a/58d16e81-f114-46b0-87d3-9324f007724a"
-					(reference "R114")
+					(reference "R116")
 					(unit 1)
 				)
 				(path "/2bc5a21a-1d79-419d-a592-6852cc07b00a/609d2beb-47a4-466a-8275-c7d831b810a1"
-					(reference "R123")
+					(reference "R125")
 					(unit 1)
 				)
 				(path "/2bc5a21a-1d79-419d-a592-6852cc07b00a/7ca24c0f-2468-4efa-8ee6-749df6aa5e15"
-					(reference "R132")
+					(reference "R134")
 					(unit 1)
 				)
 				(path "/2bc5a21a-1d79-419d-a592-6852cc07b00a/da3c2bc1-d321-4b0b-8d45-9bd0460c9e5a"
-					(reference "R126")
+					(reference "R128")
 					(unit 1)
 				)
 				(path "/2bc5a21a-1d79-419d-a592-6852cc07b00a/dbf038c9-8c09-4484-aee5-b965d923f833"
-					(reference "R129")
+					(reference "R131")
 					(unit 1)
 				)
@@
 			)
 		)
-		(property "JLCPCB BOM" "1"
-			(at 144.78 82.55 0)
-			(hide yes)
-			(show_name no)
-			(do_not_autoplace no)
-			(effects
-				(font
-					(size 1.27 1.27)
-				)
-			)
-		)
-		(property "Sim.Pin" "1=K 2=A"
-			(at 144.78 82.55 0)
-			(hide yes)
-			(show_name no)
-			(do_not_autoplace no)
-			(effects
-				(font
-					(size 1.27 1.27)
-				)
-			)
-		)
-		(property "Sim.Pins" "1=K 2=A"
-			(at 144.78 82.55 0)
+		(property "FT Rotation Offset" "0"
+			(at 144.78 82.55 90)
 			(hide yes)
 			(show_name no)
@@
 		(in_pos_files yes)
 		(dnp no)
-		(property "Reference" "R116"
+		(property "Reference" "R114"
 			(at 147.32 59.69 0)
 			(show_name no)
@@
 			)
 		)
-		(property "Value" "10k/100mW"
+		(property "Value" "10k/125mW"
 			(at 147.32 62.23 0)
 			(show_name no)
@@
 			)
 		)
-		(property "Footprint" "Tales:R_0603_1608Metric"
+		(property "Footprint" "Tales:R_0805_2012Metric"
 			(at 145.796 62.484 90)
 			(hide yes)
@@
 			)
 		)
-		(property "Case" "0603/1608"
+		(property "Case" "0805/2012"
 			(at 144.78 62.23 0)
 			(hide yes)
@@
 			)
 		)
-		(property "Mfr PN" "0603WAF1002T5E"
+		(property "Mfr PN" "0805W8F1002T5E"
 			(at 144.78 62.23 0)
 			(hide yes)
@@
 			)
 		)
-		(property "Vendor PN" "C25804"
+		(property "Vendor PN" "C17414"
 			(at 144.78 62.23 0)
 			(hide yes)
@@
 			)
 		)
-		(property "LCSC Part #" "C25804"
+		(property "LCSC Part #" "C17414"
 			(at 147.32 64.77 0)
 			(show_name no)
@@
 			)
 		)
-		(property "JLCPCB BOM" "1"
+		(property "FT Rotation Offset" "0"
 			(at 144.78 62.23 0)
 			(hide yes)
@@
 			(project "eumesmo-io-24v16ch-v6"
 				(path "/2bc5a21a-1d79-419d-a592-6852cc07b00a/118d8d95-c0ce-4d84-8406-4e7809444f6f"
-					(reference "R119")
+					(reference "R117")
 					(unit 1)
 				)
 				(path "/2bc5a21a-1d79-419d-a592-6852cc07b00a/18f82f59-0c23-40f7-8b4c-a32f0bda1493"
-					(reference "R137")
+					(reference "R135")
 					(unit 1)
 				)
 				(path "/2bc5a21a-1d79-419d-a592-6852cc07b00a/1c051e73-1175-469e-a364-cac197036f64"
-					(reference "R122")
+					(reference "R120")
 					(unit 1)
 				)
 				(path "/2bc5a21a-1d79-419d-a592-6852cc07b00a/58d16e81-f114-46b0-87d3-9324f007724a"
-					(reference "R116")
+					(reference "R114")
 					(unit 1)
 				)
 				(path "/2bc5a21a-1d79-419d-a592-6852cc07b00a/609d2beb-47a4-466a-8275-c7d831b810a1"
-					(reference "R125")
+					(reference "R123")
 					(unit 1)
 				)
 				(path "/2bc5a21a-1d79-419d-a592-6852cc07b00a/7ca24c0f-2468-4efa-8ee6-749df6aa5e15"
-					(reference "R134")
+					(reference "R132")
 					(unit 1)
 				)
 				(path "/2bc5a21a-1d79-419d-a592-6852cc07b00a/da3c2bc1-d321-4b0b-8d45-9bd0460c9e5a"
-					(reference "R128")
+					(reference "R126")
 					(unit 1)
 				)
 				(path "/2bc5a21a-1d79-419d-a592-6852cc07b00a/dbf038c9-8c09-4484-aee5-b965d923f833"
-					(reference "R131")
-					(unit 1)
-				)
+					(reference "R129")
+					(unit 1)
+				)
