File: V6/eumesmo-io-24v16ch-v6-lan.kicad_sch (KiCad schematic)
At the start: 29 parts, among them J8 ETHERNET, U6 TPS3823-33, U7 LAN8710A

Commit message: Replaced 0603 10k resistors for 0805.
Parts:
- C19: renamed from C21; FT Rotation Offset (none) -> 0; JLCPCB BOM 1 -> (none)
- C20: renamed from C22; FT Rotation Offset (none) -> 0; JLCPCB BOM 1 -> (none)
- C21: renamed from C23; FT Rotation Offset (none) -> 0; JLCPCB BOM 1 -> (none)
- C22: renamed from C24; FT Rotation Offset (none) -> 0; JLCPCB BOM 1 -> (none)
- C23: renamed from C25; FT Rotation Offset (none) -> 0; JLCPCB BOM 1 -> (none)
- C24: renamed from C20; FT Rotation Offset (none) -> 0; JLCPCB BOM 1 -> (none)
- C25: renamed from C19; FT Rotation Offset (none) -> 0; JLCPCB BOM 1 -> (none); LCSC Part # C161353 -> C9196; Mfr Murata Electronics -> FH; Mfr PN GR431BR7LA102KW66L -> 1206B102K202NT; Vendor PN C161353 -> C9196
- D8, R36: FT Rotation Offset (none) -> 0; JLCPCB BOM 1 -> (none)
- J8: FT Rotation Offset (none) -> 0; JLCPCB BOM 1 -> (none); LCSC Part # C2760325 -> C6674467; Mfr PN HR915340A -> HR915340AE; Vendor PN C2760325 -> C6674467
- R22: value 1.5k -> 1,5k; FT Rotation Offset (none) -> 0; JLCPCB BOM 1 -> (none)
- R23: value 2.2k -> 2,2k; FT Rotation Offset (none) -> 0; JLCPCB BOM 1 -> (none)
- R24: renamed from R25; value 2.2k -> 2,2k; FT Rotation Offset (none) -> 0; JLCPCB BOM 1 -> (none)
- R25: renamed from R27; value 2.2k -> 2,2k; FT Rotation Offset (none) -> 0; JLCPCB BOM 1 -> (none)
- R26: renamed from R28; value 2.2k -> 2,2k; FT Rotation Offset (none) -> 0; JLCPCB BOM 1 -> (none)
- R27: renamed from R29; value 2.2k -> 2,2k; FT Rotation Offset (none) -> 0; JLCPCB BOM 1 -> (none)
- R28: renamed from R30; value 2.2k -> 2,2k; FT Rotation Offset (none) -> 0; JLCPCB BOM 1 -> (none)
- R29: renamed from R31; value 2.2k -> 2,2k; FT Rotation Offset (none) -> 0; JLCPCB BOM 1 -> (none)
- R30: renamed from R32; FT Rotation Offset (none) -> 0; JLCPCB BOM 1 -> (none); LCSC Part # C25852 -> C281773; Mfr Uniroyal -> Yageo; Mfr PN 0402WGF1212TCE -> RT0402BRD0712K1L; Vendor PN C25852 -> C281773
- R31: renamed from R33; FT Rotation Offset (none) -> 0; JLCPCB BOM 1 -> (none)
- R32: renamed from R35; FT Rotation Offset (none) -> 0; JLCPCB BOM 1 -> (none)
- R33: renamed from R24; FT Rotation Offset (none) -> 0; JLCPCB BOM 1 -> (none)
- R34: renamed from R26; FT Rotation Offset (none) -> 0; JLCPCB BOM 1 -> (none)
- R35: renamed from R34; FT Rotation Offset (none) -> 0; JLCPCB BOM 1 -> (none)
- TP11: renamed from TP15; JLCPCB BOM 0 -> (none)
- TP12: renamed from TP14; JLCPCB BOM 0 -> (none)
- TP13: value CLK -> TP; JLCPCB BOM 0 -> (none); now not fitted; now left out of the parts list
- U6: renamed from U7; FT Rotation Offset (none) -> 0; JLCPCB BOM 1 -> (none)
- U7: renamed from U6; Case (none) -> SOT-23-5; FT Rotation Offset (none) -> 0; LCSC Part # (none) -> C7719; Mfr (none) -> Texas Instruments; Mfr PN (none) -> TPS3823-33DBVR; Vendor (none) -> JLCPCB; Vendor PN (none) -> C7719
Other:
- note removed: "OPÇÕES RJ45 HANRUN HR911105A JLCPCB C12074 HORIZONTAL MAGNÉTICO HANRUN HY951180A JLCPCB C34677 VERTICAL MAGNÉTICO"

Commit message: Adjusted components according to availability in JLCPCB.
Parts:
- R24, R25, R26, R27, R28, R29: Vendor PN C25744 -> C25879
Changed lines of the file:
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@@
 			)
 		)
-		(property "Vendor PN" "C25744"
+		(property "Vendor PN" "C25879"
 			(at 80.01 45.72 0)
 			(hide yes)
@@
 			)
 		)
-		(property "Vendor PN" "C25744"
+		(property "Vendor PN" "C25879"
 			(at 90.17 45.72 0)
 			(hide yes)
@@
 			)
 		)
-		(property "Vendor PN" "C25744"
+		(property "Vendor PN" "C25879"
 			(at 120.65 45.72 0)
 			(hide yes)
@@
 			)
 		)
-		(property "Vendor PN" "C25744"
+		(property "Vendor PN" "C25879"
 			(at 69.85 45.72 0)
 			(hide yes)
@@
 			)
 		)
-		(property "Vendor PN" "C25744"
+		(property "Vendor PN" "C25879"
 			(at 110.49 45.72 0)
 			(hide yes)
@@
 			)
 		)
-		(property "Vendor PN" "C25744"
+		(property "Vendor PN" "C25879"
 			(at 100.33 45.72 0)
 			(hide yes)

Commit message: Replaced U7 TPS3823-33 (200ms) for a TPS3820-33 (25ms)
Parts:
- U7: value TPS3823-33 -> TPS3820-33; LCSC Part # C7719 -> C130064; Mfr PN TPS3823-33DBVR -> TPS3820-33DBVR; Vendor PN C7719 -> C130064
Other:
- note added: "25ms RESET DELAY"
- note removed: "200ms RESET DELAY"
Changed lines of the file:
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@@
 		(rev "V6.3")
 	)
-	(text "200ms RESET DELAY"
+	(text "25ms RESET DELAY"
 		(exclude_from_sim no)
 		(at 139.7 137.16 0)
@@
 	)
 	(symbol
-		(lib_id "Power_Supervisor:TPS3823-xxDBV")
-		(at 129.54 133.35 0)
-		(unit 1)
-		(body_style 1)
-		(exclude_from_sim no)
-		(in_bom yes)
-		(on_board yes)
-		(in_pos_files yes)
-		(dnp no)
-		(property "Reference" "U7"
-			(at 132.08 140.97 0)
-			(show_name no)
-			(do_not_autoplace no)
-			(effects
-				(font
-					(size 1.27 1.27)
-				)
-				(justify left)
-			)
-		)
-		(property "Value" "TPS3823-33"
-			(at 132.08 143.51 0)
-			(show_name no)
-			(do_not_autoplace no)
-			(effects
-				(font
-					(size 1.27 1.27)
-				)
-				(justify left)
-			)
-		)
-		(property "Footprint" "Package_TO_SOT_SMD:SOT-23-5"
-			(at 127 133.35 0)
-			(hide yes)
-			(show_name no)
-			(do_not_autoplace no)
-			(effects
-				(font
-					(size 1.27 1.27)
-				)
-			)
-		)
-		(property "Datasheet" "https://www.ti.com/lit/ds/symlink/tps3823.pdf"
-			(at 127 133.35 0)
-			(hide yes)
-			(show_name no)
-			(do_not_autoplace no)
-			(effects
-				(font
-					(size 1.27 1.27)
-				)
-			)
-		)
-		(property "Description" "Supervisory Circuit with watchdog & manual reset, push-pull ~{RESET} output, SOT-23-6"
-			(at 129.54 133.35 0)
-			(hide yes)
-			(show_name no)
-			(do_not_autoplace no)
-			(effects
-				(font
-					(size 1.27 1.27)
-				)
-			)
-		)
-		(property "Case" "SOT-23-5"
-			(at 129.54 133.35 0)
-			(hide yes)
-			(show_name no)
-			(do_not_autoplace no)
-			(effects
-				(font
-					(size 1.27 1.27)
-				)
-			)
-		)
-		(property "LCSC Part #" "C7719"
-			(at 129.54 133.35 0)
-			(hide yes)
-			(show_name no)
-			(do_not_autoplace no)
-			(effects
-				(font
-					(size 1.27 1.27)
-				)
-			)
-		)
-		(property "Mfr" "Texas Instruments"
-			(at 129.54 133.35 0)
-			(hide yes)
-			(show_name no)
-			(do_not_autoplace no)
-			(effects
-				(font
-					(size 1.27 1.27)
-				)
-			)
-		)
-		(property "Mfr PN" "TPS3823-33DBVR"
-			(at 129.54 133.35 0)
-			(hide yes)
-			(show_name no)
-			(do_not_autoplace no)
-			(effects
-				(font
-					(size 1.27 1.27)
-				)
-			)
-		)
-		(property "Vendor" "JLCPCB"
-			(at 129.54 133.35 0)
-			(hide yes)
-			(show_name no)
-			(do_not_autoplace no)
-			(effects
-				(font
-					(size 1.27 1.27)
-				)
-			)
-		)
-		(property "Vendor PN" "C7719"
-			(at 129.54 133.35 0)
-			(hide yes)
-			(show_name no)
-			(do_not_autoplace no)
-			(effects
-				(font
-					(size 1.27 1.27)
-				)
-			)
-		)
-		(property "FT Rotation Offset" "0"
-			(at 129.54 133.35 0)
-			(hide yes)
-			(show_name no)
-			(do_not_autoplace no)
-			(effects
-				(font
-					(size 1.27 1.27)
-				)
-			)
-		)
-		(pin "3"
-		)
-		(pin "1"
-		)
-		(pin "5"
-		)
-		(pin "2"
-		)
-		(pin "4"
-		)
-		(instances
-			(project "eumesmo-io-24v16ch-v6"
-				(path "/2bc5a21a-1d79-419d-a592-6852cc07b00a/c76fc600-a423-4f14-bc69-e86c7c986b21"
-					(reference "U7")
-					(unit 1)
-				)
-			)
-		)
-	)
-	(symbol
 		(lib_id "Device:R_US")
 		(at 80.01 45.72 0)
@@
 					(unit 1)
 				)
+			)
+		)
+	)
+	(symbol
+		(lib_id "Power_Supervisor:TPS3823-xxDBV")
+		(at 129.54 133.35 0)
+		(unit 1)
+		(body_style 1)
+		(exclude_from_sim no)
+		(in_bom yes)
+		(on_board yes)
+		(in_pos_files yes)
+		(dnp no)
+		(property "Reference" "U7"
+			(at 132.08 140.97 0)
+			(show_name no)
+			(do_not_autoplace no)
+			(effects
+				(font
+					(size 1.27 1.27)
+				)
+				(justify left)
+			)
+		)
+		(property "Value" "TPS3820-33"
+			(at 132.08 143.51 0)
+			(show_name no)
+			(do_not_autoplace no)
+			(effects
+				(font
+					(size 1.27 1.27)
+				)
+				(justify left)
+			)
+		)
+		(property "Footprint" "Package_TO_SOT_SMD:SOT-23-5"
+			(at 127 133.35 0)
+			(hide yes)
+			(show_name no)
+			(do_not_autoplace no)
+			(effects
+				(font
+					(size 1.27 1.27)
+				)
+			)
+		)
+		(property "Datasheet" "https://www.ti.com/lit/ds/symlink/tps3823.pdf"
+			(at 127 133.35 0)
+			(hide yes)
+			(show_name no)
+			(do_not_autoplace no)
+			(effects
+				(font
+					(size 1.27 1.27)
+				)
+			)
+		)
+		(property "Description" "Supervisory Circuit with watchdog & manual reset, push-pull ~{RESET} output, SOT-23-6"
+			(at 129.54 133.35 0)
+			(hide yes)
+			(show_name no)
+			(do_not_autoplace no)
+			(effects
+				(font
+					(size 1.27 1.27)
+				)
+			)
+		)
+		(property "Case" "SOT-23-5"
+			(at 129.54 133.35 0)
+			(hide yes)
+			(show_name no)
+			(do_not_autoplace no)
+			(effects
+				(font
+					(size 1.27 1.27)
+				)
+			)
+		)
+		(property "LCSC Part #" "C130064"
+			(at 132.08 146.05 0)
+			(show_name no)
+			(do_not_autoplace no)
+			(effects
+				(font
+					(size 1.27 1.27)
+				)
+				(justify left)
+			)
+		)
+		(property "Mfr" "Texas Instruments"
+			(at 129.54 133.35 0)
+			(hide yes)
+			(show_name no)
+			(do_not_autoplace no)
+			(effects
+				(font
+					(size 1.27 1.27)
+				)
+			)
+		)
+		(property "Mfr PN" "TPS3820-33DBVR"
+			(at 129.54 133.35 0)
+			(hide yes)
+			(show_name no)
+			(do_not_autoplace no)
+			(effects
+				(font
+					(size 1.27 1.27)
+				)
+			)
+		)
+		(property "Vendor" "JLCPCB"
+			(at 129.54 133.35 0)
+			(hide yes)
+			(show_name no)
+			(do_not_autoplace no)
+			(effects
+				(font
+					(size 1.27 1.27)
+				)
+			)
+		)
+		(property "Vendor PN" "C130064"
+			(at 129.54 133.35 0)
+			(hide yes)
+			(show_name no)
+			(do_not_autoplace no)
+			(effects
+				(font
+					(size 1.27 1.27)
+				)
+			)
+		)
+		(property "FT Rotation Offset" "0"
+			(at 129.54 133.35 0)
+			(hide yes)
+			(show_name no)
+			(do_not_autoplace no)
+			(effects
+				(font
+					(size 1.27 1.27)
+				)
+			)
+		)
+		(pin "3"
+		)
+		(pin "1"
+		)
+		(pin "2"
+		)
+		(pin "4"
+		)
+		(pin "5"
+		)
+		(instances
+			(project "eumesmo-io-24v16ch-v6"
+				(path "/2bc5a21a-1d79-419d-a592-6852cc07b00a/c76fc600-a423-4f14-bc69-e86c7c986b21"
+					(reference "U7")
+					(unit 1)
+				)
