File: V6/eumesmo-io-24v16ch-v6-power.kicad_sch (KiCad schematic)
At the start: 51 parts, among them J6 250-202, J7 USB_C_Receptacle_USB2.0, Q1 WPM2015-3/TR, Q2 MMUN2211LT3G, U1 SY8089A1AAC, U2 TX4138

Commit message: Replaced 0603 10k resistors for 0805.
Parts:
- removed TP2, TP3: GND, Tales:TestPoint_Keystone_5019_Miniature, symbol Connector:TestPoint
- C1: renamed from C8; FT Rotation Offset (none) -> 0; JLCPCB BOM 1 -> (none)
- C10: renamed from C13; FT Rotation Offset (none) -> 0; JLCPCB BOM 1 -> (none)
- C11: renamed from C14; FT Rotation Offset (none) -> 0; JLCPCB BOM 1 -> (none)
- C12: renamed from C3; FT Rotation Offset (none) -> 0; JLCPCB BOM 1 -> (none)
- C13: renamed from C7; FT Rotation Offset (none) -> 0; JLCPCB BOM 1 -> (none)
- C14: renamed from C1; FT Rotation Offset (none) -> 0; JLCPCB BOM 1 -> (none)
- C2, D1, D4, J6, Q1, Q2: FT Rotation Offset (none) -> 0; JLCPCB BOM 1 -> (none)
- C3: renamed from C4; FT Rotation Offset (none) -> 0; JLCPCB BOM 1 -> (none)
- C4: renamed from C10; FT Rotation Offset (none) -> 0; JLCPCB BOM 1 -> (none)
- C5: renamed from C11; FT Rotation Offset (none) -> 0; JLCPCB BOM 1 -> (none)
- C6: renamed from C5; FT Rotation Offset (none) -> 0; JLCPCB BOM 1 -> (none)
- C7: renamed from C6; FT Rotation Offset (none) -> 0; JLCPCB BOM 1 -> (none)
- C8: renamed from C9; FT Rotation Offset (none) -> 0; JLCPCB BOM 1 -> (none)
- C9: renamed from C12; FT Rotation Offset (none) -> 0; JLCPCB BOM 1 -> (none)
- D2: renamed from D6; FT Rotation Offset (none) -> 0; JLCPCB BOM 1 -> (none)
- D3: renamed from D5; FT Rotation Offset (none) -> 0; JLCPCB BOM 1 -> (none)
- D5: renamed from D2; FT Rotation Offset (none) -> -90; JLCPCB BOM 1 -> (none)
- D6: renamed from D3; FT Rotation Offset (none) -> 0; JLCPCB BOM 1 -> (none)
- J7: FT Rotation Offset (none) -> 180; JLCPCB BOM 1 -> (none)
- L1: renamed from L2; FT Rotation Offset (none) -> 0; JLCPCB BOM 1 -> (none); LCSC Part # C169386 -> C3000382; Mfr Sunlord -> SXN; Mfr PN SWRB1205S-330MT -> SMDRI125-330MT; Vendor PN C169386 -> C3000382
- L2: renamed from L3; FT Rotation Offset (none) -> 0; JLCPCB BOM 1 -> (none)
- L3: renamed from L1; FT Rotation Offset (none) -> 0; JLCPCB BOM 1 -> (none)
- R1: renamed from R7; FT Rotation Offset (none) -> 0; JLCPCB BOM 1 -> (none)
- R10: renamed from R3; FT Rotation Offset (none) -> 0; JLCPCB BOM 1 -> (none)
- R11: renamed from R6; FT Rotation Offset (none) -> 0; JLCPCB BOM 1 -> (none)
- R12: renamed from R4; FT Rotation Offset (none) -> 0; JLCPCB BOM 1 -> (none)
- R2: renamed from R5; FT Rotation Offset (none) -> 0; JLCPCB BOM 1 -> (none)
- R3: renamed from R12; FT Rotation Offset (none) -> 0; JLCPCB BOM 1 -> (none)
- R4: renamed from R9; FT Rotation Offset (none) -> 0; JLCPCB BOM 1 -> (none)
- R5: renamed from R10; FT Rotation Offset (none) -> 0; JLCPCB BOM 1 -> (none)
- R6: renamed from R1; FT Rotation Offset (none) -> 0; JLCPCB BOM 1 -> (none); Mfr YAGEO -> Yageo
- R7: renamed from R2; FT Rotation Offset (none) -> 0; JLCPCB BOM 1 -> (none); Mfr YAGEO -> Yageo
- R8: FT Rotation Offset (none) -> 0; JLCPCB BOM 1 -> (none); LCSC Part # C25744 -> C60490; Mfr Uniroyal -> Yageo; Mfr PN 0402WGF1002TCE -> RC0402FR-0710KL; Vendor PN C25744 -> C60490
- R9: renamed from R11; FT Rotation Offset (none) -> 0; JLCPCB BOM 1 -> (none)
- TP1: renamed from TP7; value 5VSH -> TP5019; FT Rotation Offset (none) -> 0; JLCPCB BOM 0 -> (none); LCSC Part # (none) -> C238131; Mfr (none) -> Keystone; Mfr PN (none) -> 5019; Vendor (none) -> JLCPCB; Vendor PN (none) -> C238131
- TP2: renamed from TP9; value 5V -> TP5019; FT Rotation Offset (none) -> 0; JLCPCB BOM 0 -> (none); LCSC Part # (none) -> C238131; Mfr (none) -> Keystone; Mfr PN (none) -> 5019; Vendor (none) -> JLCPCB; Vendor PN (none) -> C238131
- TP3: renamed from TP1; value GND -> TP5019; FT Rotation Offset (none) -> 0; JLCPCB BOM 0 -> (none); LCSC Part # (none) -> C238131; Mfr (none) -> Keystone; Mfr PN (none) -> 5019; Vendor (none) -> JLCPCB; Vendor PN (none) -> C238131
- TP4: renamed from TP10; value 3V3A -> TP; JLCPCB BOM 0 -> (none); now not fitted; now left out of the parts list
- TP5: renamed from TP6; value 3V3LAN -> TP; JLCPCB BOM 0 -> (none); now not fitted; now left out of the parts list
- TP6: renamed from TP5; JLCPCB BOM 0 -> (none)
- TP7: renamed from TP4; value 3V3 -> TP5019; FT Rotation Offset (none) -> 0; JLCPCB BOM 0 -> (none); LCSC Part # (none) -> C238131; Mfr (none) -> Keystone; Mfr PN (none) -> 5019; Vendor (none) -> JLCPCB; Vendor PN (none) -> C238131
- TP8: JLCPCB BOM 0 -> (none)
- U1: renamed from U2; FT Rotation Offset (none) -> 0; JLCPCB BOM 1 -> (none)
- U2: renamed from U1; FT Rotation Offset (none) -> 0; JLCPCB BOM 1 -> (none)

Commit message: Adjusted components according to availability in JLCPCB.
Parts:
- R11: value 300R -> 330R; LCSC Part # C25102 -> C25104; Mfr PN 0402WGF3000TCE -> 0402WGF3300TCE; Vendor PN C25102 -> C25104
Changed lines of the file:
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@@
 			)
 		)
-		(property "Value" "300R"
+		(property "Value" "330R"
 			(at 124.46 139.7 0)
 			(show_name no)
@@
 			)
 		)
-		(property "Mfr PN" "0402WGF3000TCE"
+		(property "Mfr PN" "0402WGF3300TCE"
 			(at 121.92 138.43 0)
 			(hide yes)
@@
 			)
 		)
-		(property "Vendor PN" "C25102"
+		(property "Vendor PN" "C25104"
 			(at 121.92 138.43 0)
 			(hide yes)
@@
 			)
 		)
-		(property "LCSC Part #" "C25102"
+		(property "LCSC Part #" "C25104"
 			(at 124.46 142.24 0)
 			(show_name no)

Commit message: ETH connector repositioned.
Parts:
- TP1: now not fitted; now left out of the parts list
Changed lines of the file:
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@@
 		(body_style 1)
 		(exclude_from_sim no)
-		(in_bom yes)
+		(in_bom no)
 		(on_board yes)
 		(in_pos_files yes)
-		(dnp no)
+		(dnp yes)
 		(property "Reference" "TP1"
 			(at 245.11 29.21 0)

Commit message: Removed R3 shunt from the PCB, added a closed copper jumper in place.
Parts:
- added JP2: SHUNT, Jumper:SolderJumper-2_P1.3mm_Bridged_RoundedPad1.0x1.5mm, symbol Jumper:Jumper_2_Small_Bridged
- R3: now not fitted; now left out of the parts list
Connections:
- net +5V: now also JP2.2 (B)
- net 5VSH: now also JP2.1 (A)
Other:
- note added: "SHUNT R3 USED FOR CURRENT SENSING DURING DEVELOPMENT. CAN BE REMOVED FROM PRODUCTION BATCHES."
- note removed: "SHUNT USED FOR CURRENT SENSING DURING DEVELOPMENT. CAN BE REMOVED FROM PRODUCTION BATCHES."
Changed lines of the file:
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@@
 		)
 	)
-	(text "SHUNT USED FOR CURRENT SENSING\nDURING DEVELOPMENT. CAN BE\nREMOVED FROM PRODUCTION BATCHES."
+	(text "SHUNT R3 USED FOR CURRENT SENSING\nDURING DEVELOPMENT. CAN BE\nREMOVED FROM PRODUCTION BATCHES."
 		(exclude_from_sim no)
-		(at 260.35 45.72 0)
+		(at 251.46 21.59 0)
 		(effects
 			(font
@@
 	(wire
 		(pts
+			(xy 267.97 49.53) (xy 267.97 39.37)
+		)
+		(stroke
+			(width 0)
+			(type default)
+		)
+	)
+	(wire
+		(pts
 			(xy 156.21 39.37) (xy 156.21 46.99)
 		)
@@
 	(wire
 		(pts
+			(xy 260.35 49.53) (xy 267.97 49.53)
+		)
+		(stroke
+			(width 0)
+			(type default)
+		)
+	)
+	(wire
+		(pts
 			(xy 156.21 53.34) (xy 156.21 52.07)
 		)
@@
 	(wire
 		(pts
+			(xy 255.27 49.53) (xy 246.38 49.53)
+		)
+		(stroke
+			(width 0)
+			(type default)
+		)
+	)
+	(wire
+		(pts
 			(xy 198.12 110.49) (xy 210.82 110.49)
 		)
@@
 	(wire
 		(pts
+			(xy 246.38 49.53) (xy 246.38 39.37)
+		)
+		(stroke
+			(width 0)
+			(type default)
+		)
+	)
+	(wire
+		(pts
 			(xy 203.2 39.37) (xy 185.42 39.37)
 		)
@@
 	)
 	(symbol
+		(lib_id "Jumper:Jumper_2_Small_Bridged")
+		(at 257.81 49.53 0)
+		(unit 1)
+		(body_style 1)
+		(exclude_from_sim no)
+		(in_bom yes)
+		(on_board yes)
+		(in_pos_files yes)
+		(dnp no)
+		(fields_autoplaced yes)
+		(property "Reference" "JP2"
+			(at 257.81 44.45 0)
+			(show_name no)
+			(do_not_autoplace no)
+			(effects
+				(font
+					(size 1.27 1.27)
+				)
+			)
+		)
+		(property "Value" "SHUNT"
+			(at 257.81 46.99 0)
+			(show_name no)
+			(do_not_autoplace no)
+			(effects
+				(font
+					(size 1.27 1.27)
+				)
+			)
+		)
+		(property "Footprint" "Jumper:SolderJumper-2_P1.3mm_Bridged_RoundedPad1.0x1.5mm"
+			(at 257.81 49.53 0)
+			(hide yes)
+			(show_name no)
+			(do_not_autoplace no)
+			(effects
+				(font
+					(size 1.27 1.27)
+				)
+			)
+		)
+		(property "Datasheet" ""
+			(at 257.81 49.53 0)
+			(hide yes)
+			(show_name no)
+			(do_not_autoplace no)
+			(effects
+				(font
+					(size 1.27 1.27)
+				)
+			)
+		)
+		(property "Description" "Jumper, 2-pole, small symbol, bridged"
+			(at 257.81 49.53 0)
+			(hide yes)
+			(show_name no)
+			(do_not_autoplace no)
+			(effects
+				(font
+					(size 1.27 1.27)
+				)
+			)
+		)
+		(pin "1"
+		)
+		(pin "2"
+		)
+		(instances
+			(project "eumesmo-io-24v16ch-v6"
+				(path "/2bc5a21a-1d79-419d-a592-6852cc07b00a/7b388c9c-6faf-4681-b727-510de2ea001e"
+					(reference "JP2")
+					(unit 1)
+				)
+			)
+		)
+	)
+	(symbol
 		(lib_id "power:GND")
 		(at 138.43 45.72 0)
@@
 		(body_style 1)
 		(exclude_from_sim no)
-		(in_bom yes)
-		(on_board yes)
+		(in_bom no)
+		(on_board no)
 		(in_pos_files yes)
-		(dnp no)
+		(dnp yes)
 		(fields_autoplaced yes)
 		(property "Reference" "R3"
